File: kicad/Row_A.sch (KiCad schematic (older format))
At the start: 18 parts, among them U1 APA102, U10 APA102, U11 APA102, U12 APA102, U13 APA102, U14 APA102, U15 APA102, U16 APA102, U2 APA102, U3 APA102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

Commit message: added Gerbers
Connections:
- wire segments 118 -> 152
Changed lines of the file:
@@
 $EndComp
 Wire Wire Line
-	1150 1800 1150 2400
+	1150 1800 1150 2350
 Connection ~ 1800 2850
 Wire Wire Line
@@
 Connection ~ 1800 2350
 Wire Wire Line
-	950  2350 9550 2350
+	950  2350 1150 2350
 Wire Wire Line
 	10800 3100 10800 1600
@@
 	1800 2350 1800 2450
 Wire Wire Line
-	950  2850 10650 2850
+	950  2850 1800 2850
 Connection ~ 1150 2350
 Text HLabel 950  2850 0    60   Input ~ 12
@@
 $EndComp
 Wire Wire Line
-	1150 4150 1150 4750
+	1150 4150 1150 4700
 Connection ~ 1800 5200
 Wire Wire Line
@@
 Connection ~ 1800 4700
 Wire Wire Line
-	950  4700 9550 4700
+	950  4700 1150 4700
 Wire Wire Line
 	10800 5450 10800 3950
@@
 	1800 4700 1800 4800
 Wire Wire Line
-	950  5200 10650 5200
+	950  5200 1800 5200
 Connection ~ 1150 4700
 $Comp
@@
 Wire Wire Line
 	750  3950 1300 3950
+Wire Wire Line
+	1800 2850 2250 2850
+Wire Wire Line
+	1800 2350 2350 2350
+Wire Wire Line
+	1150 2350 1150 2400
+Wire Wire Line
+	1150 2350 1800 2350
+Wire Wire Line
+	2350 2350 3550 2350
+Wire Wire Line
+	2250 2850 3450 2850
+Wire Wire Line
+	3450 2850 4650 2850
+Wire Wire Line
+	3550 2350 4750 2350
+Wire Wire Line
+	4650 2850 5850 2850
+Wire Wire Line
+	4750 2350 5950 2350
+Wire Wire Line
+	5850 2850 7050 2850
+Wire Wire Line
+	5950 2350 7150 2350
+Wire Wire Line
+	7050 2850 8250 2850
+Wire Wire Line
+	7150 2350 8350 2350
+Wire Wire Line
+	8250 2850 9450 2850
+Wire Wire Line
+	8350 2350 9550 2350
+Wire Wire Line
+	9450 2850 10650 2850
+Wire Wire Line
+	1800 5200 2250 5200
+Wire Wire Line
+	1800 4700 2350 4700
+Wire Wire Line
+	1150 4700 1150 4750
+Wire Wire Line
+	1150 4700 1800 4700
+Wire Wire Line
+	2350 4700 3550 4700
+Wire Wire Line
+	2250 5200 3450 5200
+Wire Wire Line
+	3450 5200 4650 5200
+Wire Wire Line
+	3550 4700 4750 4700
+Wire Wire Line
+	4650 5200 5850 5200
+Wire Wire Line
+	4750 4700 5950 4700
+Wire Wire Line
+	5850 5200 7050 5200
+Wire Wire Line
+	5950 4700 7150 4700
+Wire Wire Line
+	7050 5200 8250 5200
+Wire Wire Line
+	7150 4700 8350 4700
+Wire Wire Line
+	8250 5200 9450 5200
+Wire Wire Line
+	8350 4700 9550 4700
+Wire Wire Line
+	9450 5200 10650 5200
 $EndSCHEMATC

Commit message: renamed all files, fresh Gerbers
Parts:
- C1, C2: footprint chromogram_libs:c_0805 -> KlokTHREEjr_libs:c_0805; symbol chromogram:C_NP -> KlokTHREEjr:C_NP
- U1, U10, U11, U12, U13, U14, U15, U16, U2, U3, U4, U5, U6, U7, U8, U9: footprint chromogram_libs:APA102 -> KlokTHREEjr_libs:APA102; symbol chromogram:APA102 -> KlokTHREEjr:APA102
Changed lines of the file:
@@
 EESchema Schematic File Version 4
-LIBS:chromogram
-LIBS:chromogram-cache
+LIBS:KlokTHREEjr
+LIBS:KlokTHREEjr-cache
 EELAYER 26 0
 EELAYER END
@@
 encoding utf-8
 Sheet 2 12
-Title "Chromogram"
+Title "KlokTHREEjr"
 Date "2017-12-26"
 Rev "rev 1"
-Comp "WyoLum"
-Comment1 "www.wyolum.com"
+Comp "www.wyolum.com"
+Comment1 "https://github.com/wyolum/KlokTHREEjr"
 Comment2 ""
 Comment3 ""
@@
 $EndDescr
 $Comp
-L chromogram:C_NP C1
+L KlokTHREEjr:C_NP C1
 U 1 1 5118AB57
 P 1800 2600
 F 0 "C1" H 1825 2700 40  0000 L CNB
 F 1 "100nF" H 1825 2500 40  0000 L CNN
-F 2 "chromogram_libs:c_0805" H 1800 2600 50  0001 C CNN
+F 2 "KlokTHREEjr_libs:c_0805" H 1800 2600 50  0001 C CNN
 F 3 "" H 1800 2600 60  0001 C CNN
 F 4 "Value" H 1800 2600 60  0001 C CNN "manf#"
@@
 GND
 $Comp
-L chromogram:APA102 U1
+L KlokTHREEjr:APA102 U1
 U 1 1 56C2E1C1
 P 1700 1600
@@
 F 0 "U1" H 1700 1900 40  0000 C CNB
 F 1 "APA102" H 1700 1275 40  0000 C CNN
-F 2 "chromogram_libs:APA102" H 1600 2000 60  0001 C CNN
+F 2 "KlokTHREEjr_libs:APA102" H 1600 2000 60  0001 C CNN
 F 3 "" H 1700 1600 60  0001 C CNN
 F 4 "mfr_pn" H 1700 1600 60  0001 C CNN "manf#"
@@
 5V
 $Comp
-L chromogram:GND #PWR01
+L KlokTHREEjr:GND #PWR01
 U 1 1 56C2E1DA
 P 1150 2400
@@
 5V
 $Comp
-L chromogram:APA102 U2
+L KlokTHREEjr:APA102 U2
 U 1 1 56C2E1EC
 P 2900 1600
@@
 F 0 "U2" H 2900 1900 40  0000 C CNB
 F 1 "APA102" H 2900 1275 40  0000 C CNN
-F 2 "chromogram_libs:APA102" H 2800 2000 60  0001 C CNN
+F 2 "KlokTHREEjr_libs:APA102" H 2800 2000 60  0001 C CNN
 F 3 "" H 2900 1600 60  0001 C CNN
 F 4 "mfr_pn" H 2900 1600 60  0001 C CNN "manf#"
@@
 $EndComp
 $Comp
-L chromogram:APA102 U3
+L KlokTHREEjr:APA102 U3
 U 1 1 56C2E1F4
 P 4100 1600
@@
 F 0 "U3" H 4100 1900 40  0000 C CNB
 F 1 "APA102" H 4100 1275 40  0000 C CNN
-F 2 "chromogram_libs:APA102" H 4000 2000 60  0001 C CNN
+F 2 "KlokTHREEjr_libs:APA102" H 4000 2000 60  0001 C CNN
 F 3 "" H 4100 1600 60  0001 C CNN
 F 4 "mfr_pn" H 4100 1600 60  0001 C CNN "manf#"
@@
 $EndComp
 $Comp
-L chromogram:APA102 U4
+L KlokTHREEjr:APA102 U4
 U 1 1 56C2E1FC
 P 5300 1600
@@
 F 0 "U4" H 5300 1900 40  0000 C CNB
 F 1 "APA102" H 5300 1275 40  0000 C CNN
-F 2 "chromogram_libs:APA102" H 5200 2000 60  0001 C CNN
+F 2 "KlokTHREEjr_libs:APA102" H 5200 2000 60  0001 C CNN
 F 3 "" H 5300 1600 60  0001 C CNN
 F 4 "mfr_pn" H 5300 1600 60  0001 C CNN "manf#"
@@
 $EndComp
 $Comp
-L chromogram:APA102 U5
+L KlokTHREEjr:APA102 U5
 U 1 1 56C2E204
 P 6500 1600
@@
 F 0 "U5" H 6500 1900 40  0000 C CNB
 F 1 "APA102" H 6500 1275 40  0000 C CNN
-F 2 "chromogram_libs:APA102" H 6400 2000 60  0001 C CNN
+F 2 "KlokTHREEjr_libs:APA102" H 6400 2000 60  0001 C CNN
 F 3 "" H 6500 1600 60  0001 C CNN
 F 4 "mfr_pn" H 6500 1600 60  0001 C CNN "manf#"
@@
 $EndComp
 $Comp
-L chromogram:APA102 U6
+L KlokTHREEjr:APA102 U6
 U 1 1 56C2E20C
 P 7700 1600
@@
 F 0 "U6" H 7700 1900 40  0000 C CNB
 F 1 "APA102" H 7700 1275 40  0000 C CNN
-F 2 "chromogram_libs:APA102" H 7600 2000 60  0001 C CNN
+F 2 "KlokTHREEjr_libs:APA102" H 7600 2000 60  0001 C CNN
 F 3 "" H 7700 1600 60  0001 C CNN
 F 4 "mfr_pn" H 7700 1600 60  0001 C CNN "manf#"
@@
 $EndComp
 $Comp
-L chromogram:APA102 U7
+L KlokTHREEjr:APA102 U7
 U 1 1 56C2E214
 P 8900 1600
@@
 F 0 "U7" H 8900 1900 40  0000 C CNB
 F 1 "APA102" H 8900 1275 40  0000 C CNN
-F 2 "chromogram_libs:APA102" H 8800 2000 60  0001 C CNN
+F 2 "KlokTHREEjr_libs:APA102" H 8800 2000 60  0001 C CNN
 F 3 "" H 8900 1600 60  0001 C CNN
 F 4 "mfr_pn" H 8900 1600 60  0001 C CNN "manf#"
@@
 $EndComp
 $Comp
-L chromogram:APA102 U8
+L KlokTHREEjr:APA102 U8
 U 1 1 56C2E21C
 P 10100 1600
@@
 F 0 "U8" H 10100 1900 40  0000 C CNB
 F 1 "APA102" H 10100 1275 40  0000 C CNN
-F 2 "chromogram_libs:APA102" H 10000 2000 60  0001 C CNN
+F 2 "KlokTHREEjr_libs:APA102" H 10000 2000 60  0001 C CNN
 F 3 "" H 10100 1600 60  0001 C CNN
 F 4 "mfr_pn" H 10100 1600 60  0001 C CNN "manf#"
@@
 CI_A
 $Comp
-L chromogram:C_NP C2
+L KlokTHREEjr:C_NP C2
 U 1 1 5A48F6EA
 P 1800 4950
 F 0 "C2" H 1825 5050 40  0000 L CNB
 F 1 "100nF" H 1825 4850 40  0000 L CNN
-F 2 "chromogram_libs:c_0805" H 1800 4950 50  0001 C CNN
+F 2 "KlokTHREEjr_libs:c_0805" H 1800 4950 50  0001 C CNN
 F 3 "" H 1800 4950 60  0001 C CNN
 F 4 "Value" H 1800 4950 60  0001 C CNN "manf#"
@@
 CI_B
 $Comp
-L chromogram:APA102 U9
+L KlokTHREEjr:APA102 U9
 U 1 1 5A48F6F4
 P 1700 3950
@@
 F 0 "U9" H 1700 4250 40  0000 C CNB
 F 1 "APA102" H 1700 3625 40  0000 C CNN
-F 2 "chromogram_libs:APA102" H 1600 4350 60  0001 C CNN
+F 2 "KlokTHREEjr_libs:APA102" H 1600 4350 60  0001 C CNN
 F 3 "" H 1700 3950 60  0001 C CNN
 F 4 "mfr_pn" H 1700 3950 60  0001 C CNN "manf#"
@@
 CI_B
 $Comp
-L chromogram:GND #PWR02
+L KlokTHREEjr:GND #PWR02
 U 1 1 5A48F6FE
 P 1150 4750
@@
 Connection ~ 1150 4700
 $Comp
-L chromogram:APA102 U10
+L KlokTHREEjr:APA102 U10
 U 1 1 5A48F710
 P 2900 3950
@@
 F 0 "U10" H 2900 4250 40  0000 C CNB
 F 1 "APA102" H 2900 3625 40  0000 C CNN
-F 2 "chromogram_libs:APA102" H 2800 4350 60  0001 C CNN
+F 2 "KlokTHREEjr_libs:APA102" H 2800 4350 60  0001 C CNN
 F 3 "" H 2900 3950 60  0001 C CNN
 F 4 "mfr_pn" H 2900 3950 60  0001 C CNN "manf#"
@@
 $EndComp
 $Comp
-L chromogram:APA102 U11
+L KlokTHREEjr:APA102 U11
 U 1 1 5A48F717
 P 4100 3950
@@
 F 0 "U11" H 4100 4250 40  0000 C CNB
 F 1 "APA102" H 4100 3625 40  0000 C CNN
-F 2 "chromogram_libs:APA102" H 4000 4350 60  0001 C CNN
+F 2 "KlokTHREEjr_libs:APA102" H 4000 4350 60  0001 C CNN
 F 3 "" H 4100 3950 60  0001 C CNN
 F 4 "mfr_pn" H 4100 3950 60  0001 C CNN "manf#"
@@
 $EndComp
 $Comp
-L chromogram:APA102 U12
+L KlokTHREEjr:APA102 U12
 U 1 1 5A48F71E
 P 5300 3950
@@
 F 0 "U12" H 5300 4250 40  0000 C CNB
 F 1 "APA102" H 5300 3625 40  0000 C CNN
-F 2 "chromogram_libs:APA102" H 5200 4350 60  0001 C CNN
+F 2 "KlokTHREEjr_libs:APA102" H 5200 4350 60  0001 C CNN
 F 3 "" H 5300 3950 60  0001 C CNN
 F 4 "mfr_pn" H 5300 3950 60  0001 C CNN "manf#"
@@
 $EndComp
 $Comp
-L chromogram:APA102 U13
+L KlokTHREEjr:APA102 U13
 U 1 1 5A48F725
 P 6500 3950
@@
 F 0 "U13" H 6500 4250 40  0000 C CNB
 F 1 "APA102" H 6500 3625 40  0000 C CNN
-F 2 "chromogram_libs:APA102" H 6400 4350 60  0001 C CNN
+F 2 "KlokTHREEjr_libs:APA102" H 6400 4350 60  0001 C CNN
 F 3 "" H 6500 3950 60  0001 C CNN
 F 4 "mfr_pn" H 6500 3950 60  0001 C CNN "manf#"
@@
 $EndComp
 $Comp
-L chromogram:APA102 U14
+L KlokTHREEjr:APA102 U14
 U 1 1 5A48F72C
 P 7700 3950
@@
 F 0 "U14" H 7700 4250 40  0000 C CNB
 F 1 "APA102" H 7700 3625 40  0000 C CNN
-F 2 "chromogram_libs:APA102" H 7600 4350 60  0001 C CNN
+F 2 "KlokTHREEjr_libs:APA102" H 7600 4350 60  0001 C CNN
 F 3 "" H 7700 3950 60  0001 C CNN
 F 4 "mfr_pn" H 7700 3950 60  0001 C CNN "manf#"
@@
 $EndComp
 $Comp
-L chromogram:APA102 U15
+L KlokTHREEjr:APA102 U15
 U 1 1 5A48F733
 P 8900 3950
@@
 F 0 "U15" H 8900 4250 40  0000 C CNB
 F 1 "APA102" H 8900 3625 40  0000 C CNN
-F 2 "chromogram_libs:APA102" H 8800 4350 60  0001 C CNN
+F 2 "KlokTHREEjr_libs:APA102" H 8800 4350 60  0001 C CNN
 F 3 "" H 8900 3950 60  0001 C CNN
 F 4 "mfr_pn" H 8900 3950 60  0001 C CNN "manf#"
@@
 $EndComp
 $Comp
-L chromogram:APA102 U16
+L KlokTHREEjr:APA102 U16
 U 1 1 5A48F73A
 P 10100 3950
@@
 F 0 "U16" H 10100 4250 40  0000 C CNB
 F 1 "APA102" H 10100 3625 40  0000 C CNN
-F 2 "chromogram_libs:APA102" H 10000 4350 60  0001 C CNN
+F 2 "KlokTHREEjr_libs:APA102" H 10000 4350 60  0001 C CNN
 F 3 "" H 10100 3950 60  0001 C CNN
 F 4 "mfr_pn" H 10100 3950 60  0001 C CNN "manf#"
