File: kicad/Row_C.sch (KiCad schematic (older format))
At the start: 28 parts

Commit message: schematic WIP
Parts:
- removed C40, C41, C42, C43, C44, C45, C46, C47, C48, C49, C50, C51, C52, C53: 100n, C4_Pretty:c_0805_led, symbol C2
- removed LED29, LED30, LED31, LED32, LED33, LED34, LED35, LED36, LED37, LED38, LED39, LED40, LED41, LED42: WS2812B, C4_Pretty:RGB_WS2811B, symbol WS2812B
- added C5, C6: 100nF, symbol ultim8x8_sym:C2
- added U33, U34, U35, U36, U37, U38, U39, U40, U41, U42, U43, U44, U45, U46, U47, U48: APA102, ultim8x8_libs:APA102, symbol ultim8x8_sym:APA102
Connections:
- net labels added: CI_C, CI_D, DI_D
- net labels removed: DO_C
- wire segments 82 -> 152

Commit message: schematic WIP
Parts:
- C5, C6: footprint (none) -> chromogram_libs:c_0805; symbol ultim8x8_sym:C2 -> chromogram:C2
- U33, U34, U35, U36, U37, U38, U39, U40, U41, U42, U43, U44, U45, U46, U47, U48: footprint ultim8x8_libs:APA102 -> chromogram_libs:APA102; symbol ultim8x8_sym:APA102 -> chromogram:APA102
Changed lines of the file:
@@
 $Descr A4 11693 8268
 encoding utf-8
-Sheet 4 9
+Sheet 4 10
 Title "Chromogram"
 Date "2017-12-26"
@@
 GND
 $Comp
-L ultim8x8_sym:APA102 U33
+L chromogram:APA102 U33
 U 1 1 56C296A0
 P 1700 1600
 F 0 "U33" H 1700 1900 40  0000 C CNB
 F 1 "APA102" H 1700 1275 40  0000 C CNN
-F 2 "ultim8x8_libs:APA102" H 1600 2000 60  0001 C CNN
+F 2 "chromogram_libs:APA102" H 1600 2000 60  0001 C CNN
 F 3 "" H 1700 1600 60  0001 C CNN
 F 4 "mfr_pn" H 1700 1600 60  0001 C CNN "manf#"
@@
 5V
 $Comp
-L ultim8x8_sym:APA102 U34
+L chromogram:APA102 U34
 U 1 1 56C296CB
 P 2900 1600
 F 0 "U34" H 2900 1900 40  0000 C CNB
 F 1 "APA102" H 2900 1275 40  0000 C CNN
-F 2 "ultim8x8_libs:APA102" H 2800 2000 60  0001 C CNN
+F 2 "chromogram_libs:APA102" H 2800 2000 60  0001 C CNN
 F 3 "" H 2900 1600 60  0001 C CNN
 F 4 "mfr_pn" H 2900 1600 60  0001 C CNN "manf#"
@@
 $EndComp
 $Comp
-L ultim8x8_sym:APA102 U35
+L chromogram:APA102 U35
 U 1 1 56C296D3
 P 4100 1600
 F 0 "U35" H 4100 1900 40  0000 C CNB
 F 1 "APA102" H 4100 1275 40  0000 C CNN
-F 2 "ultim8x8_libs:APA102" H 4000 2000 60  0001 C CNN
+F 2 "chromogram_libs:APA102" H 4000 2000 60  0001 C CNN
 F 3 "" H 4100 1600 60  0001 C CNN
 F 4 "mfr_pn" H 4100 1600 60  0001 C CNN "manf#"
@@
 $EndComp
 $Comp
-L ultim8x8_sym:APA102 U36
+L chromogram:APA102 U36
 U 1 1 56C296DB
 P 5300 1600
 F 0 "U36" H 5300 1900 40  0000 C CNB
 F 1 "APA102" H 5300 1275 40  0000 C CNN
-F 2 "ultim8x8_libs:APA102" H 5200 2000 60  0001 C CNN
+F 2 "chromogram_libs:APA102" H 5200 2000 60  0001 C CNN
 F 3 "" H 5300 1600 60  0001 C CNN
 F 4 "mfr_pn" H 5300 1600 60  0001 C CNN "manf#"
@@
 $EndComp
 $Comp
-L ultim8x8_sym:APA102 U37
+L chromogram:APA102 U37
 U 1 1 56C296E3
 P 6500 1600
 F 0 "U37" H 6500 1900 40  0000 C CNB
 F 1 "APA102" H 6500 1275 40  0000 C CNN
-F 2 "ultim8x8_libs:APA102" H 6400 2000 60  0001 C CNN
+F 2 "chromogram_libs:APA102" H 6400 2000 60  0001 C CNN
 F 3 "" H 6500 1600 60  0001 C CNN
 F 4 "mfr_pn" H 6500 1600 60  0001 C CNN "manf#"
@@
 $EndComp
 $Comp
-L ultim8x8_sym:APA102 U38
+L chromogram:APA102 U38
 U 1 1 56C296EB
 P 7700 1600
 F 0 "U38" H 7700 1900 40  0000 C CNB
 F 1 "APA102" H 7700 1275 40  0000 C CNN
-F 2 "ultim8x8_libs:APA102" H 7600 2000 60  0001 C CNN
+F 2 "chromogram_libs:APA102" H 7600 2000 60  0001 C CNN
 F 3 "" H 7700 1600 60  0001 C CNN
 F 4 "mfr_pn" H 7700 1600 60  0001 C CNN "manf#"
@@
 $EndComp
 $Comp
-L ultim8x8_sym:APA102 U39
+L chromogram:APA102 U39
 U 1 1 56C296F3
 P 8900 1600
 F 0 "U39" H 8900 1900 40  0000 C CNB
 F 1 "APA102" H 8900 1275 40  0000 C CNN
-F 2 "ultim8x8_libs:APA102" H 8800 2000 60  0001 C CNN
+F 2 "chromogram_libs:APA102" H 8800 2000 60  0001 C CNN
 F 3 "" H 8900 1600 60  0001 C CNN
 F 4 "mfr_pn" H 8900 1600 60  0001 C CNN "manf#"
@@
 $EndComp
 $Comp
-L ultim8x8_sym:APA102 U40
+L chromogram:APA102 U40
 U 1 1 56C296FB
 P 10100 1600
 F 0 "U40" H 10100 1900 40  0000 C CNB
 F 1 "APA102" H 10100 1275 40  0000 C CNN
-F 2 "ultim8x8_libs:APA102" H 10000 2000 60  0001 C CNN
+F 2 "chromogram_libs:APA102" H 10000 2000 60  0001 C CNN
 F 3 "" H 10100 1600 60  0001 C CNN
 F 4 "mfr_pn" H 10100 1600 60  0001 C CNN "manf#"
@@
 CI_D
 $Comp
-L ultim8x8_sym:APA102 U41
+L chromogram:APA102 U41
 U 1 1 5A4DEB9E
 P 1700 3950
 F 0 "U41" H 1700 4250 40  0000 C CNB
 F 1 "APA102" H 1700 3625 40  0000 C CNN
-F 2 "ultim8x8_libs:APA102" H 1600 4350 60  0001 C CNN
+F 2 "chromogram_libs:APA102" H 1600 4350 60  0001 C CNN
 F 3 "" H 1700 3950 60  0001 C CNN
 F 4 "mfr_pn" H 1700 3950 60  0001 C CNN "manf#"
@@
 CI_D
 $Comp
-L chromogram:GND #PWR?
+L chromogram:GND #PWR014
 U 1 1 5A4DEBA8
 P 1150 4750
-F 0 "#PWR?" H 1150 4750 30  0001 C CNN
+F 0 "#PWR014" H 1150 4750 30  0001 C CNN
 F 1 "GND" H 1150 4680 30  0001 C CNN
 F 2 "" H 1150 4750 60  0001 C CNN
@@
 Connection ~ 1150 4700
 $Comp
-L ultim8x8_sym:APA102 U42
+L chromogram:APA102 U42
 U 1 1 5A4DEBB6
 P 2900 3950
 F 0 "U42" H 2900 4250 40  0000 C CNB
 F 1 "APA102" H 2900 3625 40  0000 C CNN
-F 2 "ultim8x8_libs:APA102" H 2800 4350 60  0001 C CNN
+F 2 "chromogram_libs:APA102" H 2800 4350 60  0001 C CNN
 F 3 "" H 2900 3950 60  0001 C CNN
 F 4 "mfr_pn" H 2900 3950 60  0001 C CNN "manf#"
@@
 $EndComp
 $Comp
-L ultim8x8_sym:APA102 U43
+L chromogram:APA102 U43
 U 1 1 5A4DEBBD
 P 4100 3950
 F 0 "U43" H 4100 4250 40  0000 C CNB
 F 1 "APA102" H 4100 3625 40  0000 C CNN
-F 2 "ultim8x8_libs:APA102" H 4000 4350 60  0001 C CNN
+F 2 "chromogram_libs:APA102" H 4000 4350 60  0001 C CNN
 F 3 "" H 4100 3950 60  0001 C CNN
 F 4 "mfr_pn" H 4100 3950 60  0001 C CNN "manf#"
@@
 $EndComp
 $Comp
-L ultim8x8_sym:APA102 U44
+L chromogram:APA102 U44
 U 1 1 5A4DEBC4
 P 5300 3950
 F 0 "U44" H 5300 4250 40  0000 C CNB
 F 1 "APA102" H 5300 3625 40  0000 C CNN
-F 2 "ultim8x8_libs:APA102" H 5200 4350 60  0001 C CNN
+F 2 "chromogram_libs:APA102" H 5200 4350 60  0001 C CNN
 F 3 "" H 5300 3950 60  0001 C CNN
 F 4 "mfr_pn" H 5300 3950 60  0001 C CNN "manf#"
@@
 $EndComp
 $Comp
-L ultim8x8_sym:APA102 U45
+L chromogram:APA102 U45
 U 1 1 5A4DEBCB
 P 6500 3950
 F 0 "U45" H 6500 4250 40  0000 C CNB
 F 1 "APA102" H 6500 3625 40  0000 C CNN
-F 2 "ultim8x8_libs:APA102" H 6400 4350 60  0001 C CNN
+F 2 "chromogram_libs:APA102" H 6400 4350 60  0001 C CNN
 F 3 "" H 6500 3950 60  0001 C CNN
 F 4 "mfr_pn" H 6500 3950 60  0001 C CNN "manf#"
@@
 $EndComp
 $Comp
-L ultim8x8_sym:APA102 U46
+L chromogram:APA102 U46
 U 1 1 5A4DEBD2
 P 7700 3950
 F 0 "U46" H 7700 4250 40  0000 C CNB
 F 1 "APA102" H 7700 3625 40  0000 C CNN
-F 2 "ultim8x8_libs:APA102" H 7600 4350 60  0001 C CNN
+F 2 "chromogram_libs:APA102" H 7600 4350 60  0001 C CNN
 F 3 "" H 7700 3950 60  0001 C CNN
 F 4 "mfr_pn" H 7700 3950 60  0001 C CNN "manf#"
@@
 $EndComp
 $Comp
-L ultim8x8_sym:APA102 U47
+L chromogram:APA102 U47
 U 1 1 5A4DEBD9
 P 8900 3950
 F 0 "U47" H 8900 4250 40  0000 C CNB
 F 1 "APA102" H 8900 3625 40  0000 C CNN
-F 2 "ultim8x8_libs:APA102" H 8800 4350 60  0001 C CNN
+F 2 "chromogram_libs:APA102" H 8800 4350 60  0001 C CNN
 F 3 "" H 8900 3950 60  0001 C CNN
 F 4 "mfr_pn" H 8900 3950 60  0001 C CNN "manf#"
@@
 $EndComp
 $Comp
-L ultim8x8_sym:APA102 U48
+L chromogram:APA102 U48
 U 1 1 5A4DEBE0
 P 10100 3950
 F 0 "U48" H 10100 4250 40  0000 C CNB
 F 1 "APA102" H 10100 3625 40  0000 C CNN
-F 2 "ultim8x8_libs:APA102" H 10000 4350 60  0001 C CNN
+F 2 "chromogram_libs:APA102" H 10000 4350 60  0001 C CNN
 F 3 "" H 10100 3950 60  0001 C CNN
 F 4 "mfr_pn" H 10100 3950 60  0001 C CNN "manf#"
@@
 	750  3950 1300 3950
 $Comp
-L ultim8x8_sym:C2 C5
+L chromogram:C2 C5
 U 1 1 5A8CE0F0
 P 1800 2600
 F 0 "C5" H 1893 2645 50  0000 L CNN
 F 1 "100nF" H 1893 2555 50  0000 L CNN
-F 2 "" H 1800 2600 60  0000 C CNN
+F 2 "chromogram_libs:c_0805" H 1800 2600 60  0001 C CNN
 F 3 "" H 1800 2600 60  0000 C CNN
 F 4 "Value" H 1800 2600 50  0001 C CNN "manf#"
@@
 $EndComp
 $Comp
-L ultim8x8_sym:C2 C6
+L chromogram:C2 C6
 U 1 1 5A8CE18F
 P 1800 4950
 F 0 "C6" H 1893 4995 50  0000 L CNN
 F 1 "100nF" H 1893 4905 50  0000 L CNN
-F 2 "" H 1800 4950 60  0000 C CNN
+F 2 "chromogram_libs:c_0805" H 1800 4950 60  0001 C CNN
 F 3 "" H 1800 4950 60  0000 C CNN
 	1    1800 4950

Commit message: schematic dev in progress
Connections:
- wire segments 152 -> 118
Changed lines of the file:
@@
-EESchema Schematic File Version 4
+EESchema Schematic File Version 2
+LIBS:power
 LIBS:chromogram-cache
-EELAYER 26 0
+EELAYER 25 0
 EELAYER END
 $Descr A4 11693 8268
 encoding utf-8
-Sheet 4 10
+Sheet 4 11
 Title "Chromogram"
 Date "2017-12-26"
@@
 5V
 $Comp
-L chromogram:GND #PWR09
+L chromogram:GND #PWR05
 U 1 1 56C296B9
 P 1150 2400
-F 0 "#PWR09" H 1150 2400 30  0001 C CNN
+F 0 "#PWR05" H 1150 2400 30  0001 C CNN
 F 1 "GND" H 1150 2330 30  0001 C CNN
 F 2 "" H 1150 2400 60  0001 C CNN
@@
 $EndComp
 Wire Wire Line
-	1150 1800 1150 2350
-Wire Wire Line
-	950  2350 1150 2350
+	1150 1800 1150 2400
+Wire Wire Line
+	950  2350 9550 2350
 Wire Wire Line
 	10800 3100 10800 1600
 Wire Wire Line
-	950  2850 1800 2850
+	950  2850 10650 2850
 Connection ~ 1150 2350
 Text HLabel 950  2850 0    60   Input ~ 12
@@
 Text Label 1075 1600 0    60   ~ 0
 CI_C
-Wire Wire Line
-	1150 2350 1150 2400
-Wire Wire Line
-	1150 2350 1800 2350
-Wire Wire Line
-	2350 2350 3550 2350
-Wire Wire Line
-	2250 2850 3450 2850
-Wire Wire Line
-	3450 2850 4650 2850
-Wire Wire Line
-	3550 2350 4750 2350
-Wire Wire Line
-	4650 2850 5850 2850
-Wire Wire Line
-	4750 2350 5950 2350
-Wire Wire Line
-	5850 2850 7050 2850
-Wire Wire Line
-	5950 2350 7150 2350
-Wire Wire Line
-	7050 2850 8250 2850
-Wire Wire Line
-	7150 2350 8350 2350
-Wire Wire Line
-	8250 2850 9450 2850
-Wire Wire Line
-	8350 2350 9550 2350
-Wire Wire Line
-	9450 2850 10650 2850
 Text HLabel 950  5450 0    60   Output ~ 12
 CI_D
@@
 CI_D
 $Comp
-L chromogram:GND #PWR014
+L chromogram:GND #PWR06
 U 1 1 5A4DEBA8
 P 1150 4750
-F 0 "#PWR014" H 1150 4750 30  0001 C CNN
+F 0 "#PWR06" H 1150 4750 30  0001 C CNN
 F 1 "GND" H 1150 4680 30  0001 C CNN
 F 2 "" H 1150 4750 60  0001 C CNN
@@
 $EndComp
 Wire Wire Line
-	1150 4150 1150 4700
+	1150 4150 1150 4750
 Wire Wire Line
 	950  5450 10800 5450
 Wire Wire Line
-	950  4700 1150 4700
+	950  4700 9550 4700
 Wire Wire Line
 	10800 5450 10800 3950
 Wire Wire Line
-	950  5200 1800 5200
+	950  5200 10650 5200
 Connection ~ 1150 4700
 $Comp
@@
 DI_D
 Wire Wire Line
-	1150 4700 1150 4750
-Wire Wire Line
-	1150 4700 1800 4700
-Wire Wire Line
-	2350 4700 3550 4700
-Wire Wire Line
-	2250 5200 3450 5200
-Wire Wire Line
-	3450 5200 4650 5200
-Wire Wire Line
-	3550 4700 4750 4700
-Wire Wire Line
-	4650 5200 5850 5200
-Wire Wire Line
-	4750 4700 5950 4700
-Wire Wire Line
-	5850 5200 7050 5200
-Wire Wire Line
-	5950 4700 7150 4700
-Wire Wire Line
-	7050 5200 8250 5200
-Wire Wire Line
-	7150 4700 8350 4700
-Wire Wire Line
-	8250 5200 9450 5200
-Wire Wire Line
-	8350 4700 9550 4700
-Wire Wire Line
-	9450 5200 10650 5200
-Wire Wire Line
-	950  3350 950  3750
+	950  3750 950  3350
 Wire Wire Line
 	750  3100 750  3950
@@
 $EndComp
 Wire Wire Line
-	1800 4750 1800 4700
+	1800 4700 1800 4750
 Connection ~ 1800 4700
 Wire Wire Line
-	1800 4700 2350 4700
-Wire Wire Line
-	1800 5150 1800 5200
+	1800 5200 1800 5150
 Connection ~ 1800 5200
 Wire Wire Line
-	1800 5200 2250 5200
-Wire Wire Line
-	1800 2400 1800 2350
+	1800 2350 1800 2400
 Connection ~ 1800 2350
 Wire Wire Line
-	1800 2350 2350 2350
-Wire Wire Line
-	1800 2800 1800 2850
+	1800 2850 1800 2800
 Connection ~ 1800 2850
-Wire Wire Line
-	1800 2850 2250 2850
 $EndSCHEMATC

Commit message: WIP schematic
Parts:
- C5: symbol chromogram:C2 -> chromogram:C_NP
- C6: symbol chromogram:C2 -> chromogram:C_NP; manf# (none) -> Value
Connections:
- wire segments 118 -> 152
Changed lines of the file:
@@
-EESchema Schematic File Version 2
+EESchema Schematic File Version 4
 LIBS:chromogram
-LIBS:wyolum_kicad_symbols
 LIBS:chromogram-cache
-EELAYER 25 0
+EELAYER 26 0
 EELAYER END
 $Descr A4 11693 8268
@@
 $EndComp
 Wire Wire Line
-	1150 1800 1150 2400
-Wire Wire Line
-	950  2350 9550 2350
+	1150 1800 1150 2350
+Wire Wire Line
+	950  2350 1150 2350
 Wire Wire Line
 	10800 3100 10800 1600
 Wire Wire Line
-	950  2850 10650 2850
+	950  2850 1800 2850
 Connection ~ 1150 2350
 Text HLabel 950  2850 0    60   Input ~ 12
@@
 $EndComp
 Wire Wire Line
-	1150 4150 1150 4750
+	1150 4150 1150 4700
 Wire Wire Line
 	950  5450 10800 5450
 Wire Wire Line
-	950  4700 9550 4700
+	950  4700 1150 4700
 Wire Wire Line
 	10800 5450 10800 3950
 Wire Wire Line
-	950  5200 10650 5200
+	950  5200 1800 5200
 Connection ~ 1150 4700
 $Comp
@@
 	750  3950 1300 3950
 $Comp
-L chromogram:C2 C5
+L chromogram:C_NP C5
 U 1 1 5A8CE0F0
 P 1800 2600
@@
 $EndComp
 $Comp
-L chromogram:C2 C6
+L chromogram:C_NP C6
 U 1 1 5A8CE18F
 P 1800 4950
@@
 F 2 "chromogram_libs:c_0805" H 1800 4950 60  0001 C CNN
 F 3 "" H 1800 4950 60  0000 C CNN
+F 4 "Value" H 1800 4950 50  0001 C CNN "manf#"
 	1    1800 4950
 	1    0    0    -1
 $EndComp
 Wire Wire Line
-	1800 4700 1800 4750
+	1800 4700 1800 4800
 Connection ~ 1800 4700
 Wire Wire Line
-	1800 5200 1800 5150
+	1800 5200 1800 5100
 Connection ~ 1800 5200
 Wire Wire Line
-	1800 2350 1800 2400
+	1800 2350 1800 2450
 Connection ~ 1800 2350
 Wire Wire Line
-	1800 2850 1800 2800
+	1800 2850 1800 2750
 Connection ~ 1800 2850
+Wire Wire Line
+	1150 2350 1150 2400
+Wire Wire Line
+	1150 2350 1800 2350
+Wire Wire Line
+	2350 2350 3550 2350
+Wire Wire Line
+	2250 2850 3450 2850
+Wire Wire Line
+	3450 2850 4650 2850
+Wire Wire Line
+	3550 2350 4750 2350
+Wire Wire Line
+	4650 2850 5850 2850
+Wire Wire Line
+	4750 2350 5950 2350
+Wire Wire Line
+	5850 2850 7050 2850
+Wire Wire Line
+	5950 2350 7150 2350
+Wire Wire Line
+	7050 2850 8250 2850
+Wire Wire Line
+	7150 2350 8350 2350
+Wire Wire Line
+	8250 2850 9450 2850
+Wire Wire Line
+	8350 2350 9550 2350
+Wire Wire Line
+	9450 2850 10650 2850
+Wire Wire Line
+	1150 4700 1150 4750
+Wire Wire Line
+	1150 4700 1800 4700
+Wire Wire Line
+	2350 4700 3550 4700
+Wire Wire Line
+	2250 5200 3450 5200
+Wire Wire Line
+	3450 5200 4650 5200
+Wire Wire Line
+	3550 4700 4750 4700
+Wire Wire Line
+	4650 5200 5850 5200
+Wire Wire Line
+	4750 4700 5950 4700
+Wire Wire Line
+	5850 5200 7050 5200
+Wire Wire Line
+	5950 4700 7150 4700
+Wire Wire Line
+	7050 5200 8250 5200
+Wire Wire Line
+	7150 4700 8350 4700
+Wire Wire Line
+	8250 5200 9450 5200
+Wire Wire Line
+	8350 4700 9550 4700
+Wire Wire Line
+	9450 5200 10650 5200
+Wire Wire Line
+	1800 4700 2350 4700
+Wire Wire Line
+	1800 5200 2250 5200
+Wire Wire Line
+	1800 2350 2350 2350
+Wire Wire Line
+	1800 2850 2250 2850
 $EndSCHEMATC

Commit message: making progress on PCB
Connections:
- wire segments 152 -> 118
Changed lines of the file:
@@
-EESchema Schematic File Version 4
+EESchema Schematic File Version 2
 LIBS:chromogram
+LIBS:wyolum_kicad_symbols
 LIBS:chromogram-cache
-EELAYER 26 0
+EELAYER 25 0
 EELAYER END
 $Descr A4 11693 8268
@@
 $EndComp
 Wire Wire Line
-	1150 1800 1150 2350
-Wire Wire Line
-	950  2350 1150 2350
+	1150 1800 1150 2400
+Wire Wire Line
+	950  2350 9550 2350
 Wire Wire Line
 	10800 3100 10800 1600
 Wire Wire Line
-	950  2850 1800 2850
+	950  2850 10650 2850
 Connection ~ 1150 2350
 Text HLabel 950  2850 0    60   Input ~ 12
@@
 $EndComp
 Wire Wire Line
-	1150 4150 1150 4700
+	1150 4150 1150 4750
 Wire Wire Line
 	950  5450 10800 5450
 Wire Wire Line
-	950  4700 1150 4700
+	950  4700 9550 4700
 Wire Wire Line
 	10800 5450 10800 3950
 Wire Wire Line
-	950  5200 1800 5200
+	950  5200 10650 5200
 Connection ~ 1150 4700
 $Comp
@@
 	1800 2850 1800 2750
 Connection ~ 1800 2850
-Wire Wire Line
-	1150 2350 1150 2400
-Wire Wire Line
-	1150 2350 1800 2350
-Wire Wire Line
-	2350 2350 3550 2350
-Wire Wire Line
-	2250 2850 3450 2850
-Wire Wire Line
-	3450 2850 4650 2850
-Wire Wire Line
-	3550 2350 4750 2350
-Wire Wire Line
-	4650 2850 5850 2850
-Wire Wire Line
-	4750 2350 5950 2350
-Wire Wire Line
-	5850 2850 7050 2850
-Wire Wire Line
-	5950 2350 7150 2350
-Wire Wire Line
-	7050 2850 8250 2850
-Wire Wire Line
-	7150 2350 8350 2350
-Wire Wire Line
-	8250 2850 9450 2850
-Wire Wire Line
-	8350 2350 9550 2350
-Wire Wire Line
-	9450 2850 10650 2850
-Wire Wire Line
-	1150 4700 1150 4750
-Wire Wire Line
-	1150 4700 1800 4700
-Wire Wire Line
-	2350 4700 3550 4700
-Wire Wire Line
-	2250 5200 3450 5200
-Wire Wire Line
-	3450 5200 4650 5200
-Wire Wire Line
-	3550 4700 4750 4700
-Wire Wire Line
-	4650 5200 5850 5200
-Wire Wire Line
-	4750 4700 5950 4700
-Wire Wire Line
-	5850 5200 7050 5200
-Wire Wire Line
-	5950 4700 7150 4700
-Wire Wire Line
-	7050 5200 8250 5200
-Wire Wire Line
-	7150 4700 8350 4700
-Wire Wire Line
-	8250 5200 9450 5200
-Wire Wire Line
-	8350 4700 9550 4700
-Wire Wire Line
-	9450 5200 10650 5200
-Wire Wire Line
-	1800 4700 2350 4700
-Wire Wire Line
-	1800 5200 2250 5200
-Wire Wire Line
-	1800 2350 2350 2350
-Wire Wire Line
-	1800 2850 2250 2850
 $EndSCHEMATC
