File: kicad/Row_F.sch (KiCad schematic (older format))
At the start: 18 parts, among them U81 APA102, U82 APA102, U83 APA102, U84 APA102, U85 APA102, U86 APA102, U87 APA102, U88 APA102, U89 APA102, U90 APA102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

Commit message: renamed all files, fresh Gerbers
Parts:
- C11, C12: footprint chromogram_libs:c_0805 -> KlokTHREEjr_libs:c_0805; symbol chromogram:C_NP -> KlokTHREEjr:C_NP
- U81, U82, U83, U84, U85, U86, U87, U88, U89, U90, U91, U92, U93, U94, U95, U96: footprint chromogram_libs:APA102 -> KlokTHREEjr_libs:APA102; symbol chromogram:APA102 -> KlokTHREEjr:APA102
Changed lines of the file:
@@
 EESchema Schematic File Version 4
-LIBS:chromogram
-LIBS:chromogram-cache
+LIBS:KlokTHREEjr
+LIBS:KlokTHREEjr-cache
 EELAYER 26 0
 EELAYER END
@@
 encoding utf-8
 Sheet 7 12
-Title "Chromogram"
+Title "KlokTHREEjr"
 Date "2017-12-26"
 Rev "rev 1"
-Comp "WyoLum"
-Comment1 "www.wyolum.com"
+Comp "www.wyolum.com"
+Comment1 "https://github.com/wyolum/KlokTHREEjr"
 Comment2 ""
 Comment3 ""
@@
 GND
 $Comp
-L chromogram:APA102 U81
+L KlokTHREEjr:APA102 U81
 U 1 1 56C21E5C
 P 1700 1600
@@
 F 0 "U81" H 1700 1900 40  0000 C CNB
 F 1 "APA102" H 1700 1275 40  0000 C CNN
-F 2 "chromogram_libs:APA102" H 1600 2000 60  0001 C CNN
+F 2 "KlokTHREEjr_libs:APA102" H 1600 2000 60  0001 C CNN
 F 3 "" H 1700 1600 60  0001 C CNN
 F 4 "mfr_pn" H 1700 1600 60  0001 C CNN "manf#"
@@
 5V
 $Comp
-L chromogram:GND #PWR011
+L KlokTHREEjr:GND #PWR011
 U 1 1 56C21E75
 P 1150 2400
@@
 5V
 $Comp
-L chromogram:APA102 U82
+L KlokTHREEjr:APA102 U82
 U 1 1 56C21E87
 P 2900 1600
@@
 F 0 "U82" H 2900 1900 40  0000 C CNB
 F 1 "APA102" H 2900 1275 40  0000 C CNN
-F 2 "chromogram_libs:APA102" H 2800 2000 60  0001 C CNN
+F 2 "KlokTHREEjr_libs:APA102" H 2800 2000 60  0001 C CNN
 F 3 "" H 2900 1600 60  0001 C CNN
 F 4 "mfr_pn" H 2900 1600 60  0001 C CNN "manf#"
@@
 $EndComp
 $Comp
-L chromogram:APA102 U83
+L KlokTHREEjr:APA102 U83
 U 1 1 56C21E8F
 P 4100 1600
@@
 F 0 "U83" H 4100 1900 40  0000 C CNB
 F 1 "APA102" H 4100 1275 40  0000 C CNN
-F 2 "chromogram_libs:APA102" H 4000 2000 60  0001 C CNN
+F 2 "KlokTHREEjr_libs:APA102" H 4000 2000 60  0001 C CNN
 F 3 "" H 4100 1600 60  0001 C CNN
 F 4 "mfr_pn" H 4100 1600 60  0001 C CNN "manf#"
@@
 $EndComp
 $Comp
-L chromogram:APA102 U84
+L KlokTHREEjr:APA102 U84
 U 1 1 56C21E97
 P 5300 1600
@@
 F 0 "U84" H 5300 1900 40  0000 C CNB
 F 1 "APA102" H 5300 1275 40  0000 C CNN
-F 2 "chromogram_libs:APA102" H 5200 2000 60  0001 C CNN
+F 2 "KlokTHREEjr_libs:APA102" H 5200 2000 60  0001 C CNN
 F 3 "" H 5300 1600 60  0001 C CNN
 F 4 "mfr_pn" H 5300 1600 60  0001 C CNN "manf#"
@@
 $EndComp
 $Comp
-L chromogram:APA102 U85
+L KlokTHREEjr:APA102 U85
 U 1 1 56C21E9F
 P 6500 1600
@@
 F 0 "U85" H 6500 1900 40  0000 C CNB
 F 1 "APA102" H 6500 1275 40  0000 C CNN
-F 2 "chromogram_libs:APA102" H 6400 2000 60  0001 C CNN
+F 2 "KlokTHREEjr_libs:APA102" H 6400 2000 60  0001 C CNN
 F 3 "" H 6500 1600 60  0001 C CNN
 F 4 "mfr_pn" H 6500 1600 60  0001 C CNN "manf#"
@@
 $EndComp
 $Comp
-L chromogram:APA102 U86
+L KlokTHREEjr:APA102 U86
 U 1 1 56C21EA7
 P 7700 1600
@@
 F 0 "U86" H 7700 1900 40  0000 C CNB
 F 1 "APA102" H 7700 1275 40  0000 C CNN
-F 2 "chromogram_libs:APA102" H 7600 2000 60  0001 C CNN
+F 2 "KlokTHREEjr_libs:APA102" H 7600 2000 60  0001 C CNN
 F 3 "" H 7700 1600 60  0001 C CNN
 F 4 "mfr_pn" H 7700 1600 60  0001 C CNN "manf#"
@@
 $EndComp
 $Comp
-L chromogram:APA102 U87
+L KlokTHREEjr:APA102 U87
 U 1 1 56C21EAF
 P 8900 1600
@@
 F 0 "U87" H 8900 1900 40  0000 C CNB
 F 1 "APA102" H 8900 1275 40  0000 C CNN
-F 2 "chromogram_libs:APA102" H 8800 2000 60  0001 C CNN
+F 2 "KlokTHREEjr_libs:APA102" H 8800 2000 60  0001 C CNN
 F 3 "" H 8900 1600 60  0001 C CNN
 F 4 "mfr_pn" H 8900 1600 60  0001 C CNN "manf#"
@@
 $EndComp
 $Comp
-L chromogram:APA102 U88
+L KlokTHREEjr:APA102 U88
 U 1 1 56C21EB7
 P 10100 1600
@@
 F 0 "U88" H 10100 1900 40  0000 C CNB
 F 1 "APA102" H 10100 1275 40  0000 C CNN
-F 2 "chromogram_libs:APA102" H 10000 2000 60  0001 C CNN
+F 2 "KlokTHREEjr_libs:APA102" H 10000 2000 60  0001 C CNN
 F 3 "" H 10100 1600 60  0001 C CNN
 F 4 "mfr_pn" H 10100 1600 60  0001 C CNN "manf#"
@@
 CI_G
 $Comp
-L chromogram:APA102 U89
+L KlokTHREEjr:APA102 U89
 U 1 1 5A520EF3
 P 1700 3950
@@
 F 0 "U89" H 1700 4250 40  0000 C CNB
 F 1 "APA102" H 1700 3625 40  0000 C CNN
-F 2 "chromogram_libs:APA102" H 1600 4350 60  0001 C CNN
+F 2 "KlokTHREEjr_libs:APA102" H 1600 4350 60  0001 C CNN
 F 3 "" H 1700 3950 60  0001 C CNN
 F 4 "mfr_pn" H 1700 3950 60  0001 C CNN "manf#"
@@
 CI_G
 $Comp
-L chromogram:GND #PWR012
+L KlokTHREEjr:GND #PWR012
 U 1 1 5A520EFD
 P 1150 4750
@@
 Connection ~ 1150 4700
 $Comp
-L chromogram:APA102 U90
+L KlokTHREEjr:APA102 U90
 U 1 1 5A520F0B
 P 2900 3950
@@
 F 0 "U90" H 2900 4250 40  0000 C CNB
 F 1 "APA102" H 2900 3625 40  0000 C CNN
-F 2 "chromogram_libs:APA102" H 2800 4350 60  0001 C CNN
+F 2 "KlokTHREEjr_libs:APA102" H 2800 4350 60  0001 C CNN
 F 3 "" H 2900 3950 60  0001 C CNN
 F 4 "mfr_pn" H 2900 3950 60  0001 C CNN "manf#"
@@
 $EndComp
 $Comp
-L chromogram:APA102 U91
+L KlokTHREEjr:APA102 U91
 U 1 1 5A520F12
 P 4100 3950
@@
 F 0 "U91" H 4100 4250 40  0000 C CNB
 F 1 "APA102" H 4100 3625 40  0000 C CNN
-F 2 "chromogram_libs:APA102" H 4000 4350 60  0001 C CNN
+F 2 "KlokTHREEjr_libs:APA102" H 4000 4350 60  0001 C CNN
 F 3 "" H 4100 3950 60  0001 C CNN
 F 4 "mfr_pn" H 4100 3950 60  0001 C CNN "manf#"
@@
 $EndComp
 $Comp
-L chromogram:APA102 U92
+L KlokTHREEjr:APA102 U92
 U 1 1 5A520F19
 P 5300 3950
@@
 F 0 "U92" H 5300 4250 40  0000 C CNB
 F 1 "APA102" H 5300 3625 40  0000 C CNN
-F 2 "chromogram_libs:APA102" H 5200 4350 60  0001 C CNN
+F 2 "KlokTHREEjr_libs:APA102" H 5200 4350 60  0001 C CNN
 F 3 "" H 5300 3950 60  0001 C CNN
 F 4 "mfr_pn" H 5300 3950 60  0001 C CNN "manf#"
@@
 $EndComp
 $Comp
-L chromogram:APA102 U93
+L KlokTHREEjr:APA102 U93
 U 1 1 5A520F20
 P 6500 3950
@@
 F 0 "U93" H 6500 4250 40  0000 C CNB
 F 1 "APA102" H 6500 3625 40  0000 C CNN
-F 2 "chromogram_libs:APA102" H 6400 4350 60  0001 C CNN
+F 2 "KlokTHREEjr_libs:APA102" H 6400 4350 60  0001 C CNN
 F 3 "" H 6500 3950 60  0001 C CNN
 F 4 "mfr_pn" H 6500 3950 60  0001 C CNN "manf#"
@@
 $EndComp
 $Comp
-L chromogram:APA102 U94
+L KlokTHREEjr:APA102 U94
 U 1 1 5A520F27
 P 7700 3950
@@
 F 0 "U94" H 7700 4250 40  0000 C CNB
 F 1 "APA102" H 7700 3625 40  0000 C CNN
-F 2 "chromogram_libs:APA102" H 7600 4350 60  0001 C CNN
+F 2 "KlokTHREEjr_libs:APA102" H 7600 4350 60  0001 C CNN
 F 3 "" H 7700 3950 60  0001 C CNN
 F 4 "mfr_pn" H 7700 3950 60  0001 C CNN "manf#"
@@
 $EndComp
 $Comp
-L chromogram:APA102 U95
+L KlokTHREEjr:APA102 U95
 U 1 1 5A520F2E
 P 8900 3950
@@
 F 0 "U95" H 8900 4250 40  0000 C CNB
 F 1 "APA102" H 8900 3625 40  0000 C CNN
-F 2 "chromogram_libs:APA102" H 8800 4350 60  0001 C CNN
+F 2 "KlokTHREEjr_libs:APA102" H 8800 4350 60  0001 C CNN
 F 3 "" H 8900 3950 60  0001 C CNN
 F 4 "mfr_pn" H 8900 3950 60  0001 C CNN "manf#"
@@
 $EndComp
 $Comp
-L chromogram:APA102 U96
+L KlokTHREEjr:APA102 U96
 U 1 1 5A520F35
 P 10100 3950
@@
 F 0 "U96" H 10100 4250 40  0000 C CNB
 F 1 "APA102" H 10100 3625 40  0000 C CNN
-F 2 "chromogram_libs:APA102" H 10000 4350 60  0001 C CNN
+F 2 "KlokTHREEjr_libs:APA102" H 10000 4350 60  0001 C CNN
 F 3 "" H 10100 3950 60  0001 C CNN
 F 4 "mfr_pn" H 10100 3950 60  0001 C CNN "manf#"
@@
 	750  3950 1300 3950
 $Comp
-L chromogram:C_NP C11
+L KlokTHREEjr:C_NP C11
 U 1 1 5A935E60
 P 1800 2600
 F 0 "C11" H 1893 2645 50  0000 L CNN
 F 1 "100nF" H 1893 2555 50  0000 L CNN
-F 2 "chromogram_libs:c_0805" H 1800 2600 60  0001 C CNN
+F 2 "KlokTHREEjr_libs:c_0805" H 1800 2600 60  0001 C CNN
 F 3 "" H 1800 2600 60  0000 C CNN
 F 4 "Value" H 1800 2600 50  0001 C CNN "manf#"
@@
 $EndComp
 $Comp
-L chromogram:C_NP C12
+L KlokTHREEjr:C_NP C12
 U 1 1 5A935F10
 P 1800 4950
 F 0 "C12" H 1893 4995 50  0000 L CNN
 F 1 "100nF" H 1893 4905 50  0000 L CNN
-F 2 "chromogram_libs:c_0805" H 1800 4950 60  0001 C CNN
+F 2 "KlokTHREEjr_libs:c_0805" H 1800 4950 60  0001 C CNN
 F 3 "" H 1800 4950 60  0000 C CNN
 F 4 "Value" H 1800 4950 50  0001 C CNN "manf#"

Commit message: KlokTHREEjr final. Kontroller pending
Changed lines of the file:
@@
 $EndComp
 Wire Wire Line
-	1150 1800 1150 2400
-Wire Wire Line
-	950  2350 9550 2350
+	1150 1800 1150 2350
+Wire Wire Line
+	950  2350 1150 2350
 Wire Wire Line
 	10800 3100 10800 1600
 Wire Wire Line
-	950  2850 10650 2850
+	950  2850 1800 2850
 Connection ~ 1150 2350
 Text HLabel 950  2850 0    60   Input ~ 12
@@
 $EndComp
 Wire Wire Line
-	1150 4150 1150 4750
+	1150 4150 1150 4700
 Wire Wire Line
 	950  5450 10800 5450
 Wire Wire Line
-	950  4700 9550 4700
+	950  4700 1150 4700
 Wire Wire Line
 	10800 5450 10800 3950
 Wire Wire Line
-	950  5200 10650 5200
+	950  5200 1800 5200
 Connection ~ 1150 4700
 $Comp
@@
 	1800 2350 1800 2450
 Connection ~ 1800 2350
+Wire Wire Line
+	1150 2350 1150 2400
+Wire Wire Line
+	1150 2350 1800 2350
+Wire Wire Line
+	2350 2350 3550 2350
+Wire Wire Line
+	2250 2850 3450 2850
+Wire Wire Line
+	3450 2850 4650 2850
+Wire Wire Line
+	3550 2350 4750 2350
+Wire Wire Line
+	4650 2850 5850 2850
+Wire Wire Line
+	4750 2350 5950 2350
+Wire Wire Line
+	5850 2850 7050 2850
+Wire Wire Line
+	5950 2350 7150 2350
+Wire Wire Line
+	7050 2850 8250 2850
+Wire Wire Line
+	7150 2350 8350 2350
+Wire Wire Line
+	8250 2850 9450 2850
+Wire Wire Line
+	8350 2350 9550 2350
+Wire Wire Line
+	9450 2850 10650 2850
+Wire Wire Line
+	1150 4700 1150 4750
+Wire Wire Line
+	1150 4700 1800 4700
+Wire Wire Line
+	2350 4700 3550 4700
+Wire Wire Line
+	2250 5200 3450 5200
+Wire Wire Line
+	3450 5200 4650 5200
+Wire Wire Line
+	3550 4700 4750 4700
+Wire Wire Line
+	4650 5200 5850 5200
+Wire Wire Line
+	4750 4700 5950 4700
+Wire Wire Line
+	5850 5200 7050 5200
+Wire Wire Line
+	5950 4700 7150 4700
+Wire Wire Line
+	7050 5200 8250 5200
+Wire Wire Line
+	7150 4700 8350 4700
+Wire Wire Line
+	8250 5200 9450 5200
+Wire Wire Line
+	8350 4700 9550 4700
+Wire Wire Line
+	9450 5200 10650 5200
+Wire Wire Line
+	1800 4700 2350 4700
+Wire Wire Line
+	1800 5200 2250 5200
+Wire Wire Line
+	1800 2850 2250 2850
+Wire Wire Line
+	1800 2350 2350 2350
 $EndSCHEMATC
