File: kicad/Row_G.sch (KiCad schematic (older format))
At the start: 28 parts

Commit message: schematic WIP
Parts:
- removed C100, C101, C102, C103, C104, C105, C106, C107, C108, C109, C96, C97, C98, C99: 100n, C4_Pretty:c_0805_led, symbol C2
- removed LED85, LED86, LED87, LED88, LED89, LED90, LED91, LED92, LED93, LED94, LED95, LED96, LED97, LED98: WS2812B, C4_Pretty:RGB_WS2811B, symbol WS2812B
- added C13: C2, symbol ultim8x8_sym:C2
- added C14: 100nF, symbol ultim8x8_sym:C2
- added U100, U101, U102, U103, U104, U105, U106, U107, U108, U109, U110, U111, U112, U97, U98, U99: APA102, ultim8x8_libs:APA102, symbol ultim8x8_sym:APA102
Connections:
- net labels added: CI_G, CI_H, DI_H
- net labels removed: DO_G
- wire segments 82 -> 152

Commit message: schematic WIP
Parts:
- C13, C14: footprint (none) -> chromogram_libs:c_0805; symbol ultim8x8_sym:C2 -> chromogram:C2
- U100, U101, U102, U103, U104, U105, U106, U107, U108, U109, U110, U111, U112, U97, U98, U99: footprint ultim8x8_libs:APA102 -> chromogram_libs:APA102; symbol ultim8x8_sym:APA102 -> chromogram:APA102
Changed lines of the file:
@@
 $Descr A4 11693 8268
 encoding utf-8
-Sheet 8 9
+Sheet 8 10
 Title "Chromogram"
 Date "2017-12-26"
@@
 GND
 $Comp
-L ultim8x8_sym:APA102 U97
+L chromogram:APA102 U97
 U 1 1 56C1D372
 P 1700 1600
 F 0 "U97" H 1700 1900 40  0000 C CNB
 F 1 "APA102" H 1700 1275 40  0000 C CNN
-F 2 "ultim8x8_libs:APA102" H 1600 2000 60  0001 C CNN
+F 2 "chromogram_libs:APA102" H 1600 2000 60  0001 C CNN
 F 3 "" H 1700 1600 60  0001 C CNN
 F 4 "mfr_pn" H 1700 1600 60  0001 C CNN "manf#"
@@
 5V
 $Comp
-L ultim8x8_sym:APA102 U98
+L chromogram:APA102 U98
 U 1 1 56C1D39D
 P 2900 1600
 F 0 "U98" H 2900 1900 40  0000 C CNB
 F 1 "APA102" H 2900 1275 40  0000 C CNN
-F 2 "ultim8x8_libs:APA102" H 2800 2000 60  0001 C CNN
+F 2 "chromogram_libs:APA102" H 2800 2000 60  0001 C CNN
 F 3 "" H 2900 1600 60  0001 C CNN
 F 4 "mfr_pn" H 2900 1600 60  0001 C CNN "manf#"
@@
 $EndComp
 $Comp
-L ultim8x8_sym:APA102 U99
+L chromogram:APA102 U99
 U 1 1 56C1D3A5
 P 4100 1600
 F 0 "U99" H 4100 1900 40  0000 C CNB
 F 1 "APA102" H 4100 1275 40  0000 C CNN
-F 2 "ultim8x8_libs:APA102" H 4000 2000 60  0001 C CNN
+F 2 "chromogram_libs:APA102" H 4000 2000 60  0001 C CNN
 F 3 "" H 4100 1600 60  0001 C CNN
 F 4 "mfr_pn" H 4100 1600 60  0001 C CNN "manf#"
@@
 $EndComp
 $Comp
-L ultim8x8_sym:APA102 U100
+L chromogram:APA102 U100
 U 1 1 56C1D3AD
 P 5300 1600
 F 0 "U100" H 5300 1900 40  0000 C CNB
 F 1 "APA102" H 5300 1275 40  0000 C CNN
-F 2 "ultim8x8_libs:APA102" H 5200 2000 60  0001 C CNN
+F 2 "chromogram_libs:APA102" H 5200 2000 60  0001 C CNN
 F 3 "" H 5300 1600 60  0001 C CNN
 F 4 "mfr_pn" H 5300 1600 60  0001 C CNN "manf#"
@@
 $EndComp
 $Comp
-L ultim8x8_sym:APA102 U101
+L chromogram:APA102 U101
 U 1 1 56C1D3B5
 P 6500 1600
 F 0 "U101" H 6500 1900 40  0000 C CNB
 F 1 "APA102" H 6500 1275 40  0000 C CNN
-F 2 "ultim8x8_libs:APA102" H 6400 2000 60  0001 C CNN
+F 2 "chromogram_libs:APA102" H 6400 2000 60  0001 C CNN
 F 3 "" H 6500 1600 60  0001 C CNN
 F 4 "mfr_pn" H 6500 1600 60  0001 C CNN "manf#"
@@
 $EndComp
 $Comp
-L ultim8x8_sym:APA102 U102
+L chromogram:APA102 U102
 U 1 1 56C1D3BD
 P 7700 1600
 F 0 "U102" H 7700 1900 40  0000 C CNB
 F 1 "APA102" H 7700 1275 40  0000 C CNN
-F 2 "ultim8x8_libs:APA102" H 7600 2000 60  0001 C CNN
+F 2 "chromogram_libs:APA102" H 7600 2000 60  0001 C CNN
 F 3 "" H 7700 1600 60  0001 C CNN
 F 4 "mfr_pn" H 7700 1600 60  0001 C CNN "manf#"
@@
 $EndComp
 $Comp
-L ultim8x8_sym:APA102 U103
+L chromogram:APA102 U103
 U 1 1 56C1D3C5
 P 8900 1600
 F 0 "U103" H 8900 1900 40  0000 C CNB
 F 1 "APA102" H 8900 1275 40  0000 C CNN
-F 2 "ultim8x8_libs:APA102" H 8800 2000 60  0001 C CNN
+F 2 "chromogram_libs:APA102" H 8800 2000 60  0001 C CNN
 F 3 "" H 8900 1600 60  0001 C CNN
 F 4 "mfr_pn" H 8900 1600 60  0001 C CNN "manf#"
@@
 $EndComp
 $Comp
-L ultim8x8_sym:APA102 U104
+L chromogram:APA102 U104
 U 1 1 56C1D3CD
 P 10100 1600
 F 0 "U104" H 10100 1900 40  0000 C CNB
 F 1 "APA102" H 10100 1275 40  0000 C CNN
-F 2 "ultim8x8_libs:APA102" H 10000 2000 60  0001 C CNN
+F 2 "chromogram_libs:APA102" H 10000 2000 60  0001 C CNN
 F 3 "" H 10100 1600 60  0001 C CNN
 F 4 "mfr_pn" H 10100 1600 60  0001 C CNN "manf#"
@@
 CI_H
 $Comp
-L ultim8x8_sym:APA102 U105
+L chromogram:APA102 U105
 U 1 1 5A536E6F
 P 1700 3950
 F 0 "U105" H 1700 4250 40  0000 C CNB
 F 1 "APA102" H 1700 3625 40  0000 C CNN
-F 2 "ultim8x8_libs:APA102" H 1600 4350 60  0001 C CNN
+F 2 "chromogram_libs:APA102" H 1600 4350 60  0001 C CNN
 F 3 "" H 1700 3950 60  0001 C CNN
 F 4 "mfr_pn" H 1700 3950 60  0001 C CNN "manf#"
@@
 CI_H
 $Comp
-L chromogram:GND #PWR?
+L chromogram:GND #PWR018
 U 1 1 5A536E79
 P 1150 4750
-F 0 "#PWR?" H 1150 4750 30  0001 C CNN
+F 0 "#PWR018" H 1150 4750 30  0001 C CNN
 F 1 "GND" H 1150 4680 30  0001 C CNN
 F 2 "" H 1150 4750 60  0001 C CNN
@@
 Connection ~ 1150 4700
 $Comp
-L ultim8x8_sym:APA102 U106
+L chromogram:APA102 U106
 U 1 1 5A536E87
 P 2900 3950
 F 0 "U106" H 2900 4250 40  0000 C CNB
 F 1 "APA102" H 2900 3625 40  0000 C CNN
-F 2 "ultim8x8_libs:APA102" H 2800 4350 60  0001 C CNN
+F 2 "chromogram_libs:APA102" H 2800 4350 60  0001 C CNN
 F 3 "" H 2900 3950 60  0001 C CNN
 F 4 "mfr_pn" H 2900 3950 60  0001 C CNN "manf#"
@@
 $EndComp
 $Comp
-L ultim8x8_sym:APA102 U107
+L chromogram:APA102 U107
 U 1 1 5A536E8E
 P 4100 3950
 F 0 "U107" H 4100 4250 40  0000 C CNB
 F 1 "APA102" H 4100 3625 40  0000 C CNN
-F 2 "ultim8x8_libs:APA102" H 4000 4350 60  0001 C CNN
+F 2 "chromogram_libs:APA102" H 4000 4350 60  0001 C CNN
 F 3 "" H 4100 3950 60  0001 C CNN
 F 4 "mfr_pn" H 4100 3950 60  0001 C CNN "manf#"
@@
 $EndComp
 $Comp
-L ultim8x8_sym:APA102 U108
+L chromogram:APA102 U108
 U 1 1 5A536E95
 P 5300 3950
 F 0 "U108" H 5300 4250 40  0000 C CNB
 F 1 "APA102" H 5300 3625 40  0000 C CNN
-F 2 "ultim8x8_libs:APA102" H 5200 4350 60  0001 C CNN
+F 2 "chromogram_libs:APA102" H 5200 4350 60  0001 C CNN
 F 3 "" H 5300 3950 60  0001 C CNN
 F 4 "mfr_pn" H 5300 3950 60  0001 C CNN "manf#"
@@
 $EndComp
 $Comp
-L ultim8x8_sym:APA102 U109
+L chromogram:APA102 U109
 U 1 1 5A536E9C
 P 6500 3950
 F 0 "U109" H 6500 4250 40  0000 C CNB
 F 1 "APA102" H 6500 3625 40  0000 C CNN
-F 2 "ultim8x8_libs:APA102" H 6400 4350 60  0001 C CNN
+F 2 "chromogram_libs:APA102" H 6400 4350 60  0001 C CNN
 F 3 "" H 6500 3950 60  0001 C CNN
 F 4 "mfr_pn" H 6500 3950 60  0001 C CNN "manf#"
@@
 $EndComp
 $Comp
-L ultim8x8_sym:APA102 U110
+L chromogram:APA102 U110
 U 1 1 5A536EA3
 P 7700 3950
 F 0 "U110" H 7700 4250 40  0000 C CNB
 F 1 "APA102" H 7700 3625 40  0000 C CNN
-F 2 "ultim8x8_libs:APA102" H 7600 4350 60  0001 C CNN
+F 2 "chromogram_libs:APA102" H 7600 4350 60  0001 C CNN
 F 3 "" H 7700 3950 60  0001 C CNN
 F 4 "mfr_pn" H 7700 3950 60  0001 C CNN "manf#"
@@
 $EndComp
 $Comp
-L ultim8x8_sym:APA102 U111
+L chromogram:APA102 U111
 U 1 1 5A536EAA
 P 8900 3950
 F 0 "U111" H 8900 4250 40  0000 C CNB
 F 1 "APA102" H 8900 3625 40  0000 C CNN
-F 2 "ultim8x8_libs:APA102" H 8800 4350 60  0001 C CNN
+F 2 "chromogram_libs:APA102" H 8800 4350 60  0001 C CNN
 F 3 "" H 8900 3950 60  0001 C CNN
 F 4 "mfr_pn" H 8900 3950 60  0001 C CNN "manf#"
@@
 $EndComp
 $Comp
-L ultim8x8_sym:APA102 U112
+L chromogram:APA102 U112
 U 1 1 5A536EB1
 P 10100 3950
 F 0 "U112" H 10100 4250 40  0000 C CNB
 F 1 "APA102" H 10100 3625 40  0000 C CNN
-F 2 "ultim8x8_libs:APA102" H 10000 4350 60  0001 C CNN
+F 2 "chromogram_libs:APA102" H 10000 4350 60  0001 C CNN
 F 3 "" H 10100 3950 60  0001 C CNN
 F 4 "mfr_pn" H 10100 3950 60  0001 C CNN "manf#"
@@
 	750  3950 1300 3950
 $Comp
-L ultim8x8_sym:C2 C13
+L chromogram:C2 C13
 U 1 1 5A9521F9
 P 1800 2600
 F 0 "C13" H 1893 2645 50  0000 L CNN
 F 1 "C2" H 1893 2555 50  0000 L CNN
-F 2 "" H 1800 2600 60  0000 C CNN
+F 2 "chromogram_libs:c_0805" H 1800 2600 60  0001 C CNN
 F 3 "" H 1800 2600 60  0000 C CNN
 	1    1800 2600
@@
 $EndComp
 $Comp
-L ultim8x8_sym:C2 C14
+L chromogram:C2 C14
 U 1 1 5A9522A9
 P 1800 4950
 F 0 "C14" H 1893 4995 50  0000 L CNN
 F 1 "100nF" H 1893 4905 50  0000 L CNN
-F 2 "" H 1800 4950 60  0000 C CNN
+F 2 "chromogram_libs:c_0805" H 1800 4950 60  0001 C CNN
 F 3 "" H 1800 4950 60  0000 C CNN
 	1    1800 4950

Commit message: schematic dev in progress
Connections:
- wire segments 152 -> 118
Changed lines of the file:
@@
-EESchema Schematic File Version 4
+EESchema Schematic File Version 2
+LIBS:power
 LIBS:chromogram-cache
-EELAYER 26 0
+EELAYER 25 0
 EELAYER END
 $Descr A4 11693 8268
 encoding utf-8
-Sheet 8 10
+Sheet 8 11
 Title "Chromogram"
 Date "2017-12-26"
@@
 5V
 $Comp
-L chromogram:GND #PWR05
+L chromogram:GND #PWR013
 U 1 1 56C1D38B
 P 1150 2400
-F 0 "#PWR05" H 1150 2400 30  0001 C CNN
+F 0 "#PWR013" H 1150 2400 30  0001 C CNN
 F 1 "GND" H 1150 2330 30  0001 C CNN
 F 2 "" H 1150 2400 60  0001 C CNN
@@
 $EndComp
 Wire Wire Line
-	1150 1800 1150 2350
-Wire Wire Line
-	950  2350 1150 2350
+	1150 1800 1150 2400
+Wire Wire Line
+	950  2350 9550 2350
 Wire Wire Line
 	10800 3100 10800 1600
 Wire Wire Line
-	950  2850 1800 2850
+	950  2850 10650 2850
 Connection ~ 1150 2350
 Text HLabel 950  2850 0    60   Input ~ 12
@@
 Text Label 1075 1600 0    60   ~ 0
 CI_G
-Wire Wire Line
-	1150 2350 1150 2400
-Wire Wire Line
-	1150 2350 1800 2350
-Wire Wire Line
-	2350 2350 3550 2350
-Wire Wire Line
-	2250 2850 3450 2850
-Wire Wire Line
-	3450 2850 4650 2850
-Wire Wire Line
-	3550 2350 4750 2350
-Wire Wire Line
-	4650 2850 5850 2850
-Wire Wire Line
-	4750 2350 5950 2350
-Wire Wire Line
-	5850 2850 7050 2850
-Wire Wire Line
-	5950 2350 7150 2350
-Wire Wire Line
-	7050 2850 8250 2850
-Wire Wire Line
-	7150 2350 8350 2350
-Wire Wire Line
-	8250 2850 9450 2850
-Wire Wire Line
-	8350 2350 9550 2350
-Wire Wire Line
-	9450 2850 10650 2850
 Text HLabel 950  5450 0    60   Output ~ 12
 CI_H
@@
 CI_H
 $Comp
-L chromogram:GND #PWR018
+L chromogram:GND #PWR014
 U 1 1 5A536E79
 P 1150 4750
-F 0 "#PWR018" H 1150 4750 30  0001 C CNN
+F 0 "#PWR014" H 1150 4750 30  0001 C CNN
 F 1 "GND" H 1150 4680 30  0001 C CNN
 F 2 "" H 1150 4750 60  0001 C CNN
@@
 $EndComp
 Wire Wire Line
-	1150 4150 1150 4700
+	1150 4150 1150 4750
 Wire Wire Line
 	950  5450 10800 5450
 Wire Wire Line
-	950  4700 1150 4700
+	950  4700 9550 4700
 Wire Wire Line
 	10800 5450 10800 3950
 Wire Wire Line
-	950  5200 1800 5200
+	950  5200 10650 5200
 Connection ~ 1150 4700
 $Comp
@@
 DI_H
 Wire Wire Line
-	1150 4700 1150 4750
-Wire Wire Line
-	1150 4700 1800 4700
-Wire Wire Line
-	2350 4700 3550 4700
-Wire Wire Line
-	2250 5200 3450 5200
-Wire Wire Line
-	3450 5200 4650 5200
-Wire Wire Line
-	3550 4700 4750 4700
-Wire Wire Line
-	4650 5200 5850 5200
-Wire Wire Line
-	4750 4700 5950 4700
-Wire Wire Line
-	5850 5200 7050 5200
-Wire Wire Line
-	5950 4700 7150 4700
-Wire Wire Line
-	7050 5200 8250 5200
-Wire Wire Line
-	7150 4700 8350 4700
-Wire Wire Line
-	8250 5200 9450 5200
-Wire Wire Line
-	8350 4700 9550 4700
-Wire Wire Line
-	9450 5200 10650 5200
-Wire Wire Line
-	950  3350 950  3750
+	950  3750 950  3350
 Wire Wire Line
 	750  3100 750  3950
@@
 $EndComp
 Wire Wire Line
-	1800 4750 1800 4700
+	1800 4700 1800 4750
 Connection ~ 1800 4700
 Wire Wire Line
-	1800 4700 2350 4700
-Wire Wire Line
-	1800 5150 1800 5200
+	1800 5200 1800 5150
 Connection ~ 1800 5200
 Wire Wire Line
-	1800 5200 2250 5200
-Wire Wire Line
-	1800 2800 1800 2850
+	1800 2850 1800 2800
 Connection ~ 1800 2850
 Wire Wire Line
-	1800 2850 2250 2850
-Wire Wire Line
-	1800 2400 1800 2350
+	1800 2350 1800 2400
 Connection ~ 1800 2350
-Wire Wire Line
-	1800 2350 2350 2350
 $EndSCHEMATC

Commit message: WIP schematic
Parts:
- removed C13: C2, chromogram_libs:c_0805, symbol chromogram:C2
- added C13: 100nF, chromogram_libs:c_0805, symbol chromogram:C_NP
- C14: symbol chromogram:C2 -> chromogram:C_NP; manf# (none) -> Value
Connections:
- wire segments 118 -> 152
Changed lines of the file:
@@
-EESchema Schematic File Version 2
+EESchema Schematic File Version 4
 LIBS:chromogram
-LIBS:wyolum_kicad_symbols
 LIBS:chromogram-cache
-EELAYER 25 0
+EELAYER 26 0
 EELAYER END
 $Descr A4 11693 8268
@@
 $EndComp
 Wire Wire Line
-	1150 1800 1150 2400
-Wire Wire Line
-	950  2350 9550 2350
+	1150 1800 1150 2350
+Wire Wire Line
+	950  2350 1150 2350
 Wire Wire Line
 	10800 3100 10800 1600
 Wire Wire Line
-	950  2850 10650 2850
+	950  2850 1800 2850
 Connection ~ 1150 2350
 Text HLabel 950  2850 0    60   Input ~ 12
@@
 $EndComp
 Wire Wire Line
-	1150 4150 1150 4750
+	1150 4150 1150 4700
 Wire Wire Line
 	950  5450 10800 5450
 Wire Wire Line
-	950  4700 9550 4700
+	950  4700 1150 4700
 Wire Wire Line
 	10800 5450 10800 3950
 Wire Wire Line
-	950  5200 10650 5200
+	950  5200 1800 5200
 Connection ~ 1150 4700
 $Comp
@@
 	750  3950 1300 3950
 $Comp
-L chromogram:C2 C13
-U 1 1 5A9521F9
-P 1800 2600
-F 0 "C13" H 1893 2645 50  0000 L CNN
-F 1 "C2" H 1893 2555 50  0000 L CNN
-F 2 "chromogram_libs:c_0805" H 1800 2600 60  0001 C CNN
-F 3 "" H 1800 2600 60  0000 C CNN
-	1    1800 2600
-	1    0    0    -1
-$EndComp
-$Comp
-L chromogram:C2 C14
+L chromogram:C_NP C14
 U 1 1 5A9522A9
 P 1800 4950
@@
 F 2 "chromogram_libs:c_0805" H 1800 4950 60  0001 C CNN
 F 3 "" H 1800 4950 60  0000 C CNN
+F 4 "Value" H 1800 4950 50  0001 C CNN "manf#"
 	1    1800 4950
 	1    0    0    -1
 $EndComp
 Wire Wire Line
-	1800 4700 1800 4750
+	1800 4700 1800 4800
 Connection ~ 1800 4700
 Wire Wire Line
-	1800 5200 1800 5150
+	1800 5200 1800 5100
 Connection ~ 1800 5200
 Wire Wire Line
-	1800 2850 1800 2800
+	1800 2850 1800 2750
 Connection ~ 1800 2850
 Wire Wire Line
-	1800 2350 1800 2400
+	1800 2350 1800 2450
 Connection ~ 1800 2350
+Wire Wire Line
+	1150 2350 1150 2400
+Wire Wire Line
+	1150 2350 1800 2350
+Wire Wire Line
+	2350 2350 3550 2350
+Wire Wire Line
+	2250 2850 3450 2850
+Wire Wire Line
+	3450 2850 4650 2850
+Wire Wire Line
+	3550 2350 4750 2350
+Wire Wire Line
+	4650 2850 5850 2850
+Wire Wire Line
+	4750 2350 5950 2350
+Wire Wire Line
+	5850 2850 7050 2850
+Wire Wire Line
+	5950 2350 7150 2350
+Wire Wire Line
+	7050 2850 8250 2850
+Wire Wire Line
+	7150 2350 8350 2350
+Wire Wire Line
+	8250 2850 9450 2850
+Wire Wire Line
+	8350 2350 9550 2350
+Wire Wire Line
+	9450 2850 10650 2850
+Wire Wire Line
+	1150 4700 1150 4750
+Wire Wire Line
+	1150 4700 1800 4700
+Wire Wire Line
+	2350 4700 3550 4700
+Wire Wire Line
+	2250 5200 3450 5200
+Wire Wire Line
+	3450 5200 4650 5200
+Wire Wire Line
+	3550 4700 4750 4700
+Wire Wire Line
+	4650 5200 5850 5200
+Wire Wire Line
+	4750 4700 5950 4700
+Wire Wire Line
+	5850 5200 7050 5200
+Wire Wire Line
+	5950 4700 7150 4700
+Wire Wire Line
+	7050 5200 8250 5200
+Wire Wire Line
+	7150 4700 8350 4700
+Wire Wire Line
+	8250 5200 9450 5200
+Wire Wire Line
+	8350 4700 9550 4700
+Wire Wire Line
+	9450 5200 10650 5200
+Wire Wire Line
+	1800 4700 2350 4700
+Wire Wire Line
+	1800 5200 2250 5200
+Wire Wire Line
+	1800 2850 2250 2850
+Wire Wire Line
+	1800 2350 2350 2350
+$Comp
+L chromogram:C_NP C13
+U 1 1 5A96AC0D
+P 1800 2600
+F 0 "C13" H 1893 2645 50  0000 L CNN
+F 1 "100nF" H 1893 2555 50  0000 L CNN
+F 2 "chromogram_libs:c_0805" H 1800 2600 60  0001 C CNN
+F 3 "" H 1800 2600 60  0000 C CNN
+F 4 "Value" H 1800 2600 50  0001 C CNN "manf#"
+	1    1800 2600
+	1    0    0    -1
+$EndComp
 $EndSCHEMATC

Commit message: making progress on PCB
Connections:
- wire segments 152 -> 118
Changed lines of the file:
@@
-EESchema Schematic File Version 4
+EESchema Schematic File Version 2
 LIBS:chromogram
+LIBS:wyolum_kicad_symbols
 LIBS:chromogram-cache
-EELAYER 26 0
+EELAYER 25 0
 EELAYER END
 $Descr A4 11693 8268
@@
 $EndComp
 Wire Wire Line
-	1150 1800 1150 2350
-Wire Wire Line
-	950  2350 1150 2350
+	1150 1800 1150 2400
+Wire Wire Line
+	950  2350 9550 2350
 Wire Wire Line
 	10800 3100 10800 1600
 Wire Wire Line
-	950  2850 1800 2850
+	950  2850 10650 2850
 Connection ~ 1150 2350
 Text HLabel 950  2850 0    60   Input ~ 12
@@
 $EndComp
 Wire Wire Line
-	1150 4150 1150 4700
+	1150 4150 1150 4750
 Wire Wire Line
 	950  5450 10800 5450
 Wire Wire Line
-	950  4700 1150 4700
+	950  4700 9550 4700
 Wire Wire Line
 	10800 5450 10800 3950
 Wire Wire Line
-	950  5200 1800 5200
+	950  5200 10650 5200
 Connection ~ 1150 4700
 $Comp
@@
 	1800 2350 1800 2450
 Connection ~ 1800 2350
-Wire Wire Line
-	1150 2350 1150 2400
-Wire Wire Line
-	1150 2350 1800 2350
-Wire Wire Line
-	2350 2350 3550 2350
-Wire Wire Line
-	2250 2850 3450 2850
-Wire Wire Line
-	3450 2850 4650 2850
-Wire Wire Line
-	3550 2350 4750 2350
-Wire Wire Line
-	4650 2850 5850 2850
-Wire Wire Line
-	4750 2350 5950 2350
-Wire Wire Line
-	5850 2850 7050 2850
-Wire Wire Line
-	5950 2350 7150 2350
-Wire Wire Line
-	7050 2850 8250 2850
-Wire Wire Line
-	7150 2350 8350 2350
-Wire Wire Line
-	8250 2850 9450 2850
-Wire Wire Line
-	8350 2350 9550 2350
-Wire Wire Line
-	9450 2850 10650 2850
-Wire Wire Line
-	1150 4700 1150 4750
-Wire Wire Line
-	1150 4700 1800 4700
-Wire Wire Line
-	2350 4700 3550 4700
-Wire Wire Line
-	2250 5200 3450 5200
-Wire Wire Line
-	3450 5200 4650 5200
-Wire Wire Line
-	3550 4700 4750 4700
-Wire Wire Line
-	4650 5200 5850 5200
-Wire Wire Line
-	4750 4700 5950 4700
-Wire Wire Line
-	5850 5200 7050 5200
-Wire Wire Line
-	5950 4700 7150 4700
-Wire Wire Line
-	7050 5200 8250 5200
-Wire Wire Line
-	7150 4700 8350 4700
-Wire Wire Line
-	8250 5200 9450 5200
-Wire Wire Line
-	8350 4700 9550 4700
-Wire Wire Line
-	9450 5200 10650 5200
-Wire Wire Line
-	1800 4700 2350 4700
-Wire Wire Line
-	1800 5200 2250 5200
-Wire Wire Line
-	1800 2850 2250 2850
-Wire Wire Line
-	1800 2350 2350 2350
 $Comp
 L chromogram:C_NP C13
