File: kicad/Row_H.sch (KiCad schematic (older format))
At the start: 28 parts

Commit message: schematic WIP
Parts:
- removed C110, C111, C112, C113, C114, C115, C116, C117, C118, C119, C120, C121, C122, C123: 100n, C4_Pretty:c_0805_led, symbol C2
- removed LED100, LED101, LED102, LED103, LED104, LED105, LED106, LED107, LED108, LED109, LED110, LED111, LED112, LED99: WS2812B, C4_Pretty:RGB_WS2811B, symbol WS2812B
- added C15, C16: 100nF, ultim8x8_libs:c_0805, symbol ultim8x8_sym:C2
- added U113, U114, U115, U116, U117, U118, U119, U120, U121, U122, U123, U124, U125, U126, U127, U128: APA102, ultim8x8_libs:APA102, symbol ultim8x8_sym:APA102
Connections:
- net labels added: CI_H, CO_H
- wire segments 82 -> 152

Commit message: schematic WIP
Parts:
- C15, C16: footprint ultim8x8_libs:c_0805 -> chromogram_libs:c_0805; symbol ultim8x8_sym:C2 -> chromogram:C2
- U113, U114, U115, U116, U117, U118, U119, U120, U121, U122, U123, U124, U125, U126, U127, U128: footprint ultim8x8_libs:APA102 -> chromogram_libs:APA102; symbol ultim8x8_sym:APA102 -> chromogram:APA102
Changed lines of the file:
@@
 $Descr A4 11693 8268
 encoding utf-8
-Sheet 9 9
+Sheet 9 10
 Title "Chromogram"
 Date "2017-12-26"
@@
 GND
 $Comp
-L ultim8x8_sym:APA102 U113
+L chromogram:APA102 U113
 U 1 1 5118ABBB
 P 1700 1600
 F 0 "U113" H 1700 1900 40  0000 C CNB
 F 1 "APA102" H 1700 1275 40  0000 C CNN
-F 2 "ultim8x8_libs:APA102" H 1600 2000 60  0001 C CNN
+F 2 "chromogram_libs:APA102" H 1600 2000 60  0001 C CNN
 F 3 "" H 1700 1600 60  0001 C CNN
 F 4 "mfr_pn" H 1700 1600 60  0001 C CNN "manf#"
@@
 5V
 $Comp
-L ultim8x8_sym:C2 C15
+L chromogram:C2 C15
 U 1 1 51168961
 P 1800 2600
 F 0 "C15" H 1825 2700 50  0000 L CNN
 F 1 "100nF" H 1825 2500 50  0000 L CNN
-F 2 "ultim8x8_libs:c_0805" H 1800 2600 50  0001 C CNN
+F 2 "chromogram_libs:c_0805" H 1800 2600 50  0001 C CNN
 F 3 "" H 1800 2600 60  0001 C CNN
 F 4 "Value" H 1800 2600 60  0001 C CNN "manf#"
@@
 5V
 $Comp
-L ultim8x8_sym:APA102 U114
+L chromogram:APA102 U114
 U 1 1 56C06E0E
 P 2900 1600
 F 0 "U114" H 2900 1900 40  0000 C CNB
 F 1 "APA102" H 2900 1275 40  0000 C CNN
-F 2 "ultim8x8_libs:APA102" H 2800 2000 60  0001 C CNN
+F 2 "chromogram_libs:APA102" H 2800 2000 60  0001 C CNN
 F 3 "" H 2900 1600 60  0001 C CNN
 F 4 "mfr_pn" H 2900 1600 60  0001 C CNN "manf#"
@@
 $EndComp
 $Comp
-L ultim8x8_sym:APA102 U115
+L chromogram:APA102 U115
 U 1 1 56C06E52
 P 4100 1600
 F 0 "U115" H 4100 1900 40  0000 C CNB
 F 1 "APA102" H 4100 1275 40  0000 C CNN
-F 2 "ultim8x8_libs:APA102" H 4000 2000 60  0001 C CNN
+F 2 "chromogram_libs:APA102" H 4000 2000 60  0001 C CNN
 F 3 "" H 4100 1600 60  0001 C CNN
 F 4 "mfr_pn" H 4100 1600 60  0001 C CNN "manf#"
@@
 $EndComp
 $Comp
-L ultim8x8_sym:APA102 U116
+L chromogram:APA102 U116
 U 1 1 56C06F1D
 P 5300 1600
 F 0 "U116" H 5300 1900 40  0000 C CNB
 F 1 "APA102" H 5300 1275 40  0000 C CNN
-F 2 "ultim8x8_libs:APA102" H 5200 2000 60  0001 C CNN
+F 2 "chromogram_libs:APA102" H 5200 2000 60  0001 C CNN
 F 3 "" H 5300 1600 60  0001 C CNN
 F 4 "mfr_pn" H 5300 1600 60  0001 C CNN "manf#"
@@
 $EndComp
 $Comp
-L ultim8x8_sym:APA102 U117
+L chromogram:APA102 U117
 U 1 1 56C06FBB
 P 6500 1600
 F 0 "U117" H 6500 1900 40  0000 C CNB
 F 1 "APA102" H 6500 1275 40  0000 C CNN
-F 2 "ultim8x8_libs:APA102" H 6400 2000 60  0001 C CNN
+F 2 "chromogram_libs:APA102" H 6400 2000 60  0001 C CNN
 F 3 "" H 6500 1600 60  0001 C CNN
 F 4 "mfr_pn" H 6500 1600 60  0001 C CNN "manf#"
@@
 $EndComp
 $Comp
-L ultim8x8_sym:APA102 U118
+L chromogram:APA102 U118
 U 1 1 56C07772
 P 7700 1600
 F 0 "U118" H 7700 1900 40  0000 C CNB
 F 1 "APA102" H 7700 1275 40  0000 C CNN
-F 2 "ultim8x8_libs:APA102" H 7600 2000 60  0001 C CNN
+F 2 "chromogram_libs:APA102" H 7600 2000 60  0001 C CNN
 F 3 "" H 7700 1600 60  0001 C CNN
 F 4 "mfr_pn" H 7700 1600 60  0001 C CNN "manf#"
@@
 $EndComp
 $Comp
-L ultim8x8_sym:APA102 U119
+L chromogram:APA102 U119
 U 1 1 56C077C2
 P 8900 1600
 F 0 "U119" H 8900 1900 40  0000 C CNB
 F 1 "APA102" H 8900 1275 40  0000 C CNN
-F 2 "ultim8x8_libs:APA102" H 8800 2000 60  0001 C CNN
+F 2 "chromogram_libs:APA102" H 8800 2000 60  0001 C CNN
 F 3 "" H 8900 1600 60  0001 C CNN
 F 4 "mfr_pn" H 8900 1600 60  0001 C CNN "manf#"
@@
 $EndComp
 $Comp
-L ultim8x8_sym:APA102 U120
+L chromogram:APA102 U120
 U 1 1 56C07914
 P 10100 1600
 F 0 "U120" H 10100 1900 40  0000 C CNB
 F 1 "APA102" H 10100 1275 40  0000 C CNN
-F 2 "ultim8x8_libs:APA102" H 10000 2000 60  0001 C CNN
+F 2 "chromogram_libs:APA102" H 10000 2000 60  0001 C CNN
 F 3 "" H 10100 1600 60  0001 C CNN
 F 4 "mfr_pn" H 10100 1600 60  0001 C CNN "manf#"
@@
 CO_H
 $Comp
-L ultim8x8_sym:APA102 U121
+L chromogram:APA102 U121
 U 1 1 5A470142
 P 1700 3950
 F 0 "U121" H 1700 4250 40  0000 C CNB
 F 1 "APA102" H 1700 3625 40  0000 C CNN
-F 2 "ultim8x8_libs:APA102" H 1600 4350 60  0001 C CNN
+F 2 "chromogram_libs:APA102" H 1600 4350 60  0001 C CNN
 F 3 "" H 1700 3950 60  0001 C CNN
 F 4 "mfr_pn" H 1700 3950 60  0001 C CNN "manf#"
@@
 CO_H
 $Comp
-L ultim8x8_sym:C2 C16
+L chromogram:C2 C16
 U 1 1 5A47014C
 P 1800 4950
 F 0 "C16" H 1825 5050 50  0000 L CNN
 F 1 "100nF" H 1825 4850 50  0000 L CNN
-F 2 "ultim8x8_libs:c_0805" H 1800 4950 50  0001 C CNN
+F 2 "chromogram_libs:c_0805" H 1800 4950 50  0001 C CNN
 F 3 "" H 1800 4950 60  0001 C CNN
 F 4 "Value" H 1800 4950 60  0001 C CNN "manf#"
@@
 $EndComp
 $Comp
-L chromogram:GND #PWR?
+L chromogram:GND #PWR019
 U 1 1 5A470153
 P 1150 4750
-F 0 "#PWR?" H 1150 4750 30  0001 C CNN
+F 0 "#PWR019" H 1150 4750 30  0001 C CNN
 F 1 "GND" H 1150 4680 30  0001 C CNN
 F 2 "" H 1150 4750 60  0001 C CNN
@@
 Connection ~ 1150 4700
 $Comp
-L ultim8x8_sym:APA102 U122
+L chromogram:APA102 U122
 U 1 1 5A470165
 P 2900 3950
 F 0 "U122" H 2900 4250 40  0000 C CNB
 F 1 "APA102" H 2900 3625 40  0000 C CNN
-F 2 "ultim8x8_libs:APA102" H 2800 4350 60  0001 C CNN
+F 2 "chromogram_libs:APA102" H 2800 4350 60  0001 C CNN
 F 3 "" H 2900 3950 60  0001 C CNN
 F 4 "mfr_pn" H 2900 3950 60  0001 C CNN "manf#"
@@
 $EndComp
 $Comp
-L ultim8x8_sym:APA102 U123
+L chromogram:APA102 U123
 U 1 1 5A47016C
 P 4100 3950
 F 0 "U123" H 4100 4250 40  0000 C CNB
 F 1 "APA102" H 4100 3625 40  0000 C CNN
-F 2 "ultim8x8_libs:APA102" H 4000 4350 60  0001 C CNN
+F 2 "chromogram_libs:APA102" H 4000 4350 60  0001 C CNN
 F 3 "" H 4100 3950 60  0001 C CNN
 F 4 "mfr_pn" H 4100 3950 60  0001 C CNN "manf#"
@@
 $EndComp
 $Comp
-L ultim8x8_sym:APA102 U124
+L chromogram:APA102 U124
 U 1 1 5A470173
 P 5300 3950
 F 0 "U124" H 5300 4250 40  0000 C CNB
 F 1 "APA102" H 5300 3625 40  0000 C CNN
-F 2 "ultim8x8_libs:APA102" H 5200 4350 60  0001 C CNN
+F 2 "chromogram_libs:APA102" H 5200 4350 60  0001 C CNN
 F 3 "" H 5300 3950 60  0001 C CNN
 F 4 "mfr_pn" H 5300 3950 60  0001 C CNN "manf#"
@@
 $EndComp
 $Comp
-L ultim8x8_sym:APA102 U125
+L chromogram:APA102 U125
 U 1 1 5A47017A
 P 6500 3950
 F 0 "U125" H 6500 4250 40  0000 C CNB
 F 1 "APA102" H 6500 3625 40  0000 C CNN
-F 2 "ultim8x8_libs:APA102" H 6400 4350 60  0001 C CNN
+F 2 "chromogram_libs:APA102" H 6400 4350 60  0001 C CNN
 F 3 "" H 6500 3950 60  0001 C CNN
 F 4 "mfr_pn" H 6500 3950 60  0001 C CNN "manf#"
@@
 $EndComp
 $Comp
-L ultim8x8_sym:APA102 U126
+L chromogram:APA102 U126
 U 1 1 5A470181
 P 7700 3950
 F 0 "U126" H 7700 4250 40  0000 C CNB
 F 1 "APA102" H 7700 3625 40  0000 C CNN
-F 2 "ultim8x8_libs:APA102" H 7600 4350 60  0001 C CNN
+F 2 "chromogram_libs:APA102" H 7600 4350 60  0001 C CNN
 F 3 "" H 7700 3950 60  0001 C CNN
 F 4 "mfr_pn" H 7700 3950 60  0001 C CNN "manf#"
@@
 $EndComp
 $Comp
-L ultim8x8_sym:APA102 U127
+L chromogram:APA102 U127
 U 1 1 5A470188
 P 8900 3950
 F 0 "U127" H 8900 4250 40  0000 C CNB
 F 1 "APA102" H 8900 3625 40  0000 C CNN
-F 2 "ultim8x8_libs:APA102" H 8800 4350 60  0001 C CNN
+F 2 "chromogram_libs:APA102" H 8800 4350 60  0001 C CNN
 F 3 "" H 8900 3950 60  0001 C CNN
 F 4 "mfr_pn" H 8900 3950 60  0001 C CNN "manf#"
@@
 $EndComp
 $Comp
-L ultim8x8_sym:APA102 U128
+L chromogram:APA102 U128
 U 1 1 5A47018F
 P 10100 3950
 F 0 "U128" H 10100 4250 40  0000 C CNB
 F 1 "APA102" H 10100 3625 40  0000 C CNN
-F 2 "ultim8x8_libs:APA102" H 10000 4350 60  0001 C CNN
+F 2 "chromogram_libs:APA102" H 10000 4350 60  0001 C CNN
 F 3 "" H 10100 3950 60  0001 C CNN
 F 4 "mfr_pn" H 10100 3950 60  0001 C CNN "manf#"

Commit message: schematic dev in progress
Connections:
- wire segments 152 -> 118
Changed lines of the file:
@@
-EESchema Schematic File Version 4
+EESchema Schematic File Version 2
+LIBS:power
 LIBS:chromogram-cache
-EELAYER 26 0
+EELAYER 25 0
 EELAYER END
 $Descr A4 11693 8268
 encoding utf-8
-Sheet 9 10
+Sheet 9 11
 Title "Chromogram"
 Date "2017-12-26"
@@
 $EndComp
 $Comp
-L chromogram:GND #PWR04
+L chromogram:GND #PWR015
 U 1 1 5118AAB4
 P 1150 2400
-F 0 "#PWR04" H 1150 2400 30  0001 C CNN
+F 0 "#PWR015" H 1150 2400 30  0001 C CNN
 F 1 "GND" H 1150 2330 30  0001 C CNN
 F 2 "" H 1150 2400 60  0001 C CNN
@@
 $EndComp
 Wire Wire Line
-	1150 1800 1150 2350
+	1150 1800 1150 2400
 Connection ~ 1800 2850
 Wire Wire Line
@@
 Connection ~ 1800 2350
 Wire Wire Line
-	950  2350 1150 2350
+	950  2350 9550 2350
 Wire Wire Line
 	10800 3100 10800 1600
@@
 	1800 2350 1800 2400
 Wire Wire Line
-	950  2850 1800 2850
+	950  2850 10650 2850
 Connection ~ 1150 2350
 Text HLabel 950  2850 0    60   Input ~ 12
@@
 Text Label 1075 1600 0    60   ~ 0
 CI_H
-Wire Wire Line
-	1800 2850 2250 2850
-Wire Wire Line
-	1800 2350 2350 2350
-Wire Wire Line
-	1150 2350 1150 2400
-Wire Wire Line
-	1150 2350 1800 2350
-Wire Wire Line
-	2350 2350 3550 2350
-Wire Wire Line
-	2250 2850 3450 2850
-Wire Wire Line
-	3450 2850 4650 2850
-Wire Wire Line
-	3550 2350 4750 2350
-Wire Wire Line
-	4650 2850 5850 2850
-Wire Wire Line
-	4750 2350 5950 2350
-Wire Wire Line
-	5850 2850 7050 2850
-Wire Wire Line
-	5950 2350 7150 2350
-Wire Wire Line
-	7050 2850 8250 2850
-Wire Wire Line
-	7150 2350 8350 2350
-Wire Wire Line
-	8250 2850 9450 2850
-Wire Wire Line
-	8350 2350 9550 2350
-Wire Wire Line
-	9450 2850 10650 2850
 Text HLabel 950  5450 0    60   Output ~ 12
 CO_H
@@
 $EndComp
 $Comp
-L chromogram:GND #PWR019
+L chromogram:GND #PWR016
 U 1 1 5A470153
 P 1150 4750
-F 0 "#PWR019" H 1150 4750 30  0001 C CNN
+F 0 "#PWR016" H 1150 4750 30  0001 C CNN
 F 1 "GND" H 1150 4680 30  0001 C CNN
 F 2 "" H 1150 4750 60  0001 C CNN
@@
 $EndComp
 Wire Wire Line
-	1150 4150 1150 4700
+	1150 4150 1150 4750
 Connection ~ 1800 5200
 Wire Wire Line
@@
 Connection ~ 1800 4700
 Wire Wire Line
-	950  4700 1150 4700
+	950  4700 9550 4700
 Wire Wire Line
 	10800 5450 10800 3950
@@
 	1800 4700 1800 4750
 Wire Wire Line
-	950  5200 1800 5200
+	950  5200 10650 5200
 Connection ~ 1150 4700
 $Comp
@@
 DO_H
 Wire Wire Line
-	1800 5200 2250 5200
-Wire Wire Line
-	1800 4700 2350 4700
-Wire Wire Line
-	1150 4700 1150 4750
-Wire Wire Line
-	1150 4700 1800 4700
-Wire Wire Line
-	2350 4700 3550 4700
-Wire Wire Line
-	2250 5200 3450 5200
-Wire Wire Line
-	3450 5200 4650 5200
-Wire Wire Line
-	3550 4700 4750 4700
-Wire Wire Line
-	4650 5200 5850 5200
-Wire Wire Line
-	4750 4700 5950 4700
-Wire Wire Line
-	5850 5200 7050 5200
-Wire Wire Line
-	5950 4700 7150 4700
-Wire Wire Line
-	7050 5200 8250 5200
-Wire Wire Line
-	7150 4700 8350 4700
-Wire Wire Line
-	8250 5200 9450 5200
-Wire Wire Line
-	8350 4700 9550 4700
-Wire Wire Line
-	9450 5200 10650 5200
-Wire Wire Line
-	950  3350 950  3750
+	950  3750 950  3350
 Wire Wire Line
 	750  3100 750  3950

Commit message: WIP schematic
Parts:
- C15, C16: symbol chromogram:C2 -> chromogram:C_NP
Connections:
- wire segments 118 -> 152
Changed lines of the file:
@@
-EESchema Schematic File Version 2
+EESchema Schematic File Version 4
 LIBS:chromogram
-LIBS:wyolum_kicad_symbols
 LIBS:chromogram-cache
-EELAYER 25 0
+EELAYER 26 0
 EELAYER END
 $Descr A4 11693 8268
@@
 5V
 $Comp
-L chromogram:C2 C15
+L chromogram:C_NP C15
 U 1 1 51168961
 P 1800 2600
@@
 $EndComp
 Wire Wire Line
-	1150 1800 1150 2400
+	1150 1800 1150 2350
 Connection ~ 1800 2850
 Wire Wire Line
-	1800 2850 1800 2800
+	1800 2850 1800 2750
 Connection ~ 1800 2350
 Wire Wire Line
-	950  2350 9550 2350
+	950  2350 1150 2350
 Wire Wire Line
 	10800 3100 10800 1600
 Wire Wire Line
-	1800 2350 1800 2400
-Wire Wire Line
-	950  2850 10650 2850
+	1800 2350 1800 2450
+Wire Wire Line
+	950  2850 1800 2850
 Connection ~ 1150 2350
 Text HLabel 950  2850 0    60   Input ~ 12
@@
 CO_H
 $Comp
-L chromogram:C2 C16
+L chromogram:C_NP C16
 U 1 1 5A47014C
 P 1800 4950
@@
 $EndComp
 Wire Wire Line
-	1150 4150 1150 4750
+	1150 4150 1150 4700
 Connection ~ 1800 5200
 Wire Wire Line
-	1800 5200 1800 5150
+	1800 5200 1800 5100
 Wire Wire Line
 	950  5450 10800 5450
 Connection ~ 1800 4700
 Wire Wire Line
-	950  4700 9550 4700
+	950  4700 1150 4700
 Wire Wire Line
 	10800 5450 10800 3950
 Wire Wire Line
-	1800 4700 1800 4750
-Wire Wire Line
-	950  5200 10650 5200
+	1800 4700 1800 4800
+Wire Wire Line
+	950  5200 1800 5200
 Connection ~ 1150 4700
 $Comp
@@
 Wire Wire Line
 	750  3950 1300 3950
+Wire Wire Line
+	1800 2850 2250 2850
+Wire Wire Line
+	1800 2350 2350 2350
+Wire Wire Line
+	1150 2350 1150 2400
+Wire Wire Line
+	1150 2350 1800 2350
+Wire Wire Line
+	2350 2350 3550 2350
+Wire Wire Line
+	2250 2850 3450 2850
+Wire Wire Line
+	3450 2850 4650 2850
+Wire Wire Line
+	3550 2350 4750 2350
+Wire Wire Line
+	4650 2850 5850 2850
+Wire Wire Line
+	4750 2350 5950 2350
+Wire Wire Line
+	5850 2850 7050 2850
+Wire Wire Line
+	5950 2350 7150 2350
+Wire Wire Line
+	7050 2850 8250 2850
+Wire Wire Line
+	7150 2350 8350 2350
+Wire Wire Line
+	8250 2850 9450 2850
+Wire Wire Line
+	8350 2350 9550 2350
+Wire Wire Line
+	9450 2850 10650 2850
+Wire Wire Line
+	1800 5200 2250 5200
+Wire Wire Line
+	1800 4700 2350 4700
+Wire Wire Line
+	1150 4700 1150 4750
+Wire Wire Line
+	1150 4700 1800 4700
+Wire Wire Line
+	2350 4700 3550 4700
+Wire Wire Line
+	2250 5200 3450 5200
+Wire Wire Line
+	3450 5200 4650 5200
+Wire Wire Line
+	3550 4700 4750 4700
+Wire Wire Line
+	4650 5200 5850 5200
+Wire Wire Line
+	4750 4700 5950 4700
+Wire Wire Line
+	5850 5200 7050 5200
+Wire Wire Line
+	5950 4700 7150 4700
+Wire Wire Line
+	7050 5200 8250 5200
+Wire Wire Line
+	7150 4700 8350 4700
+Wire Wire Line
+	8250 5200 9450 5200
+Wire Wire Line
+	8350 4700 9550 4700
+Wire Wire Line
+	9450 5200 10650 5200
 $EndSCHEMATC

Commit message: making progress on PCB
Connections:
- wire segments 152 -> 118
Changed lines of the file:
@@
-EESchema Schematic File Version 4
+EESchema Schematic File Version 2
 LIBS:chromogram
+LIBS:wyolum_kicad_symbols
 LIBS:chromogram-cache
-EELAYER 26 0
+EELAYER 25 0
 EELAYER END
 $Descr A4 11693 8268
@@
 $EndComp
 Wire Wire Line
-	1150 1800 1150 2350
+	1150 1800 1150 2400
 Connection ~ 1800 2850
 Wire Wire Line
@@
 Connection ~ 1800 2350
 Wire Wire Line
-	950  2350 1150 2350
+	950  2350 9550 2350
 Wire Wire Line
 	10800 3100 10800 1600
@@
 	1800 2350 1800 2450
 Wire Wire Line
-	950  2850 1800 2850
+	950  2850 10650 2850
 Connection ~ 1150 2350
 Text HLabel 950  2850 0    60   Input ~ 12
@@
 $EndComp
 Wire Wire Line
-	1150 4150 1150 4700
+	1150 4150 1150 4750
 Connection ~ 1800 5200
 Wire Wire Line
@@
 Connection ~ 1800 4700
 Wire Wire Line
-	950  4700 1150 4700
+	950  4700 9550 4700
 Wire Wire Line
 	10800 5450 10800 3950
@@
 	1800 4700 1800 4800
 Wire Wire Line
-	950  5200 1800 5200
+	950  5200 10650 5200
 Connection ~ 1150 4700
 $Comp
@@
 Wire Wire Line
 	750  3950 1300 3950
-Wire Wire Line
-	1800 2850 2250 2850
-Wire Wire Line
-	1800 2350 2350 2350
-Wire Wire Line
-	1150 2350 1150 2400
-Wire Wire Line
-	1150 2350 1800 2350
-Wire Wire Line
-	2350 2350 3550 2350
-Wire Wire Line
-	2250 2850 3450 2850
-Wire Wire Line
-	3450 2850 4650 2850
-Wire Wire Line
-	3550 2350 4750 2350
-Wire Wire Line
-	4650 2850 5850 2850
-Wire Wire Line
-	4750 2350 5950 2350
-Wire Wire Line
-	5850 2850 7050 2850
-Wire Wire Line
-	5950 2350 7150 2350
-Wire Wire Line
-	7050 2850 8250 2850
-Wire Wire Line
-	7150 2350 8350 2350
-Wire Wire Line
-	8250 2850 9450 2850
-Wire Wire Line
-	8350 2350 9550 2350
-Wire Wire Line
-	9450 2850 10650 2850
-Wire Wire Line
-	1800 5200 2250 5200
-Wire Wire Line
-	1800 4700 2350 4700
-Wire Wire Line
-	1150 4700 1150 4750
-Wire Wire Line
-	1150 4700 1800 4700
-Wire Wire Line
-	2350 4700 3550 4700
-Wire Wire Line
-	2250 5200 3450 5200
-Wire Wire Line
-	3450 5200 4650 5200
-Wire Wire Line
-	3550 4700 4750 4700
-Wire Wire Line
-	4650 5200 5850 5200
-Wire Wire Line
-	4750 4700 5950 4700
-Wire Wire Line
-	5850 5200 7050 5200
-Wire Wire Line
-	5950 4700 7150 4700
-Wire Wire Line
-	7050 5200 8250 5200
-Wire Wire Line
-	7150 4700 8350 4700
-Wire Wire Line
-	8250 5200 9450 5200
-Wire Wire Line
-	8350 4700 9550 4700
-Wire Wire Line
-	9450 5200 10650 5200
 $EndSCHEMATC
