File: kicad/chromogram.sch (KiCad schematic (older format))
At the start: 72 parts, among them P1 ICSP, P10 Marquee, P2 FTDI, P3 PWR_IN, P5 PWR_IN, P6 5VEN_L, P7 I2C_L, P8 5VEN_R, P9 I2C_R, SW1 SW_RST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

Commit message: schematic WIP
Parts:
- removed A6, A7, B2, D7: CONN_1, C4_Pretty:BreakOutPad, symbol CONN_1
- removed C3: 100n, C4_Pretty:c_0805, symbol CAP_NP
- removed C5, C7: 22p, C4_Pretty:c_0805, symbol CAP_NP
- removed L3: Wyolum, C4_Pretty:Logo-WL3, symbol Logos
- removed L4: Chronogram, C4_Pretty:Logo_silk_OSHW_6x6mm, symbol Logos
- removed L5: Logo, C4_Pretty:Logo_silk_OSHW_6x6mm, symbol Logos
- removed R12, R13: 0R, C4_Pretty:r_0805, symbol R
- removed S1, S2, S3, S4: CONN_1, C4_Pretty:Screw_3mm, symbol CONN_1
- removed S10, S11, S12, S13: CONN_1, C4_Pretty:Slot_tiewrap, symbol CONN_1
- removed S5, S6: CONN_1, C4_Pretty:MtgHole_3mm, symbol CONN_1
- removed X1: 16MHz, C4_Pretty:Xtal_SMD3, symbol CRYSTAL_3
- added R2: 470R, C4_Pretty:r_0805, symbol chromogram:R
- BT1: symbol Batt_RTC -> chromogram:Batt_RTC
- C?: renamed from C6; symbol CAP_NP -> chromogram:CAP_NP
- C?: renamed from C8; symbol CAP_NP -> chromogram:CAP_NP
- C?: renamed from C9; symbol CAP_NP -> chromogram:CAP_NP
- C?: renamed from C1; symbol CAP_NP -> chromogram:CAP_NP
- C?: renamed from C11; symbol CAP_NP -> chromogram:CAP_NP
- C?: renamed from C10; symbol C_POL_1 -> chromogram:C_POL_1
- C?: renamed from C194; symbol C_POL_1 -> chromogram:C_POL_1
- C?: renamed from C195; symbol C_POL_1 -> chromogram:C_POL_1
- C?: renamed from C196; symbol C_POL_1 -> chromogram:C_POL_1
- C?: renamed from C197; symbol CAP_NP -> chromogram:CAP_NP
- C?: renamed from C198; symbol CAP_NP -> chromogram:CAP_NP
- C?: renamed from C199; symbol CAP_NP -> chromogram:CAP_NP
- D?: renamed from D1; symbol DIODE_ZENER -> chromogram:DIODE_ZENER
- F1: symbol FUSE -> chromogram:FUSE
- L1: symbol Logos -> ultim8x8_sym:OSHW; manf# (none) -> Value
- L2: symbol Logos -> ultim8x8_sym:LOGO_WL; manf# (none) -> Value
- LDR1, LDR2, LDR3, LDR4: symbol VR -> chromogram:VR
- P10: symbol CONN_4 -> chromogram:CONN_4
- P?: renamed from P2; symbol CONN_6 -> chromogram:CONN_6
- P?: renamed from P1; symbol CONN_6 -> chromogram:CONN_6
- P?: renamed from P9; symbol CONN_4 -> chromogram:CONN_4
- P?: renamed from P7; symbol CONN_4 -> chromogram:CONN_4
- P?: renamed from P6; symbol R -> chromogram:R
- P?: renamed from P8; symbol R -> chromogram:R
- P?: renamed from P5; symbol CONN_3 -> chromogram:CONN_3
- P?: renamed from P3; symbol CONN_3 -> chromogram:CONN_3
- R1: symbol R -> chromogram:R
- R?: renamed from R2; symbol R -> chromogram:R
- R?: renamed from R8; symbol R -> chromogram:R
- R?: renamed from R9; symbol R -> chromogram:R
- R?: renamed from R6; symbol R -> chromogram:R
- R?: renamed from R7; symbol R -> chromogram:R
- R?: renamed from R10; symbol R -> chromogram:R
- R?: renamed from R11; symbol R -> chromogram:R
- R?: renamed from R15; symbol R -> chromogram:R
- R?: renamed from R3; symbol R -> chromogram:R
- R?: renamed from R4; symbol R -> chromogram:R
- R?: renamed from R5; symbol R -> chromogram:R
- R?: renamed from R14; symbol R -> chromogram:R
- R?: renamed from R16; symbol R -> chromogram:R
- SW1, SW2, SW3: symbol SW_PUSH -> chromogram:SW_PUSH
- U?: renamed from U2; symbol DS3231N -> chromogram:DS3231N
- U?: symbol ESP-wroom-32 -> chromogram:ESP-wroom-32
Connections:
- net labels added: CI_A, CI_B, CI_C, CI_D, CI_E, CI_F, CI_G, CI_H, CLK_IN, CLK_OUT, DAT_IN, DAT_OUT, DI_A, DI_B, DI_C, DI_D, DI_E, DI_F, DI_G, DI_H
- net labels removed: A to B, A6, A7, AREF, B to C, B2, C to D, D to E, D7, E to F, F to G, G to H, H to I, I to J, J to K, K to L, L to M, M to NC, R to Matrix Input
- wire segments 290 -> 319
- no-connect marks 11 -> 0
Other:
- note added: "16 x 8 pixel matrix"
- note removed: "14 x 13 pixel matrix"
- note removed: "Breakout pins"
- note removed: "Logos"
- note removed: "Mounting Screws"
- note removed: "Power cord ancorage holes"
- note removed: "Solder Bridges for\nHW Addressing"
- note removed: "Spare holes"
- moved on the sheet: P?, R1

Commit message: schematic WIP
Parts:
- removed C? (x5): 100n, C4_Pretty:c_0805, symbol chromogram:CAP_NP
- removed L1: OSHW, C4_Pretty:Logo_silk_OSHW_6x6mm, symbol ultim8x8_sym:OSHW
- removed L2: Wyolum, C4_Pretty:Logo-WL3, symbol ultim8x8_sym:LOGO_WL
- removed P10: Marquee, C4_Pretty:Header_4x1, symbol chromogram:CONN_4
- removed P?: FTDI, C4_Pretty:Header_FTDI, symbol chromogram:CONN_6
- removed P?: I2C_R, C4_Pretty:STACK-R, symbol chromogram:CONN_4
- removed P?: I2C_L, C4_Pretty:STACK-L, symbol chromogram:CONN_4
- removed P?: 5VEN_L, C4_Pretty:r_0805, symbol chromogram:R
- removed P?: 5VEN_R, C4_Pretty:r_0805, symbol chromogram:R
- removed R? (x2): 10K, C4_Pretty:r_0805, symbol chromogram:R
- removed R?: 470R, C4_Pretty:r_0805, symbol chromogram:R
- removed SW1: SW_RST, C4_Pretty:SW_SMD, symbol chromogram:SW_PUSH
- BT1: footprint C4_Pretty:CR2032_SMD2 -> chromogram_libs:CR2032_SMD
- C21, C22, C28: renamed from C?; footprint C4_Pretty:c_0805 -> chromogram_libs:c_0805
- C24, C25, C26, C27: renamed from C?; footprint C4_Pretty:c_2917 -> chromogram_libs:c_2917
- D1: renamed from D?; footprint C4_Pretty:diode-DO214AA -> chromogram_libs:diode-DO214AA
- F1: footprint C4_Pretty:f_1812 -> chromogram_libs:f_1812
- LDR1, LDR2, LDR3, LDR4: footprint C4_Pretty:r_0805_ldr -> chromogram_libs:r_0805_ldr
- P5: renamed from P?; footprint C4_Pretty:ISP -> chromogram_libs:ISP
- P8, P9: renamed from P?; footprint C4_Pretty:Header_3x1_PWR -> chromogram_libs:Header_3x1_PWR
- R1, R2: footprint C4_Pretty:r_0805 -> chromogram_libs:r_0805
- R10, R11, R12, R13, R14, R15, R6, R7, R8, R9: renamed from R?; footprint C4_Pretty:r_0805 -> chromogram_libs:r_0805
- SW2, SW3: footprint C4_Pretty:SW_SMD -> chromogram_libs:SW_SMD
- U130: renamed from U?; footprint C4_Pretty:DS3231 -> chromogram_libs:DS3231
- gave numbers to parts that had none: 1
Connections:
- net labels removed: 5V_L, 5V_R
- wire segments 319 -> 262
Other:
- note removed: "Arduino"
- note removed: "FTDI Header"
- note removed: "Header for Marquee"
- note removed: "I2C Connectors"

Commit message: schematic dev in progress
Parts:
- removed BT1: Batt_RTC, chromogram_libs:CR2032_SMD, symbol chromogram:Batt_RTC
- removed C21, C22, C28: 100n, chromogram_libs:c_0805, symbol chromogram:CAP_NP
- removed C24, C25, C26, C27: 47u, chromogram_libs:c_2917, symbol chromogram:C_POL_1
- removed D1: SMBJ5339B, chromogram_libs:diode-DO214AA, symbol chromogram:DIODE_ZENER
- removed F1: miniSMDC200F/16, chromogram_libs:f_1812, symbol chromogram:FUSE
- removed P5: ICSP, chromogram_libs:ISP, symbol chromogram:CONN_6
- removed P8, P9: PWR_IN, chromogram_libs:Header_3x1_PWR, symbol chromogram:CONN_3
- removed R6, R7: 10K, chromogram_libs:r_0805, symbol chromogram:R
- removed R8, R9: 4K7, chromogram_libs:r_0805, symbol chromogram:R
- removed U130: DS3231N, chromogram_libs:DS3231, symbol chromogram:DS3231N
- U129: footprint (none) -> chromogram_libs:esp_wroom_32; manf# (none) -> mfr_pn
Connections:
- net labels added: RST
- net labels removed: BAT, RESET, VCC
- wire segments 262 -> 155
Other:
- note removed: "ICSP Header"
- note removed: "Power supply"
- note removed: "RTC"

Commit message: schematic WIP
Parts:
- removed LDR1, LDR2, LDR3, LDR4: LDR, chromogram_libs:r_0805_ldr, symbol chromogram:VR
- removed SW2: SW_L, chromogram_libs:SW_SMD, symbol chromogram:SW_PUSH
- removed SW3: SW_R, chromogram_libs:SW_SMD, symbol chromogram:SW_PUSH
- added LDR1, LDR2, LDR3, LDR4: LDR, Opto-Devices:Resistor_LDR_10x8.5_RM7.6, symbol chromogram:LDR03
- added S1: SW-L, symbol chromogram:SW-SPST-M
- added S2: SW-R, symbol chromogram:SW-SPST-M
Connections:
- net labels added: 3V3
- wire segments 155 -> 213
- no-connect marks 0 -> 1

Commit message: making progress on schematic
Parts:
- added P2: OUT_CLK_DAT, Pin_Headers:Pin_Header_Straight_1x02, symbol CONN_2
- LDR1, LDR2, LDR3, LDR4: footprint Opto-Devices:Resistor_LDR_10x8.5_RM7.6 -> chromogram_libs:r_0805_ldr
- S1, S2: footprint (none) -> chromogram_libs:SW_SMD
Connections:
- net labels added: ACTIVE, DCD, DSR, DTR, EN, IO0, IO13, IO15, RXD0, TXD0
- net labels removed: MARQUEE_DATA, MARQUEE_SENSE, MATRIX_PIN, MISO, MOSI, RXD, SCK, TXD
- wire segments 213 -> 209
- no-connect marks 1 -> 28
Other:
- moved on the sheet: R1, R2

Commit message: WIP schematic
Parts:
- added C27: 100uF/6V3, chromogram_libs:c_2917, symbol chromogram:C_POL
- added C28: 1uF/10V, chromogram_libs:c_0805, symbol chromogram:C_NP
- added R10, R11: 10K, chromogram_libs:r_0805, symbol chromogram:R
- added S1: SW-ENTER, chromogram_libs:SW_SMD, symbol chromogram:SW-SPST-M
- added S2: SW-INC, chromogram_libs:SW_SMD, symbol chromogram:SW-SPST-M
- P2: footprint Pin_Headers:Pin_Header_Straight_1x02 -> chromogram_libs:Pin_Header_Straight_1x02; symbol CONN_2 -> chromogram:CONN_2; manf# (none) -> Value
- S5: renamed from S1; value SW-L -> SW-DEC
- S6: renamed from S2; value SW-R -> SW-MODE
- renumbered R10 to R24, R11 to R25
Connections:
- net labels added: SW_D, SW_E, SW_I, SW_M
- net labels removed: ACTIVE, DCD, DSR, SW_L, SW_R
- wire segments 209 -> 236
- no-connect marks 28 -> 16
Other:
- note added: "BUTTONS"
- note added: "I2C"
- note added: "LDR"
- note added: "LED CLK/DAT"
- note added: "SERIAL"
- moved on the sheet: R12, R13, R14, R15, R24, R25, S5, S6

Commit message: making progress on PCB
Connections:
- wire segments 236 -> 212
Changed lines of the file:
@@
-EESchema Schematic File Version 4
+EESchema Schematic File Version 2
 LIBS:chromogram
+LIBS:wyolum_kicad_symbols
 LIBS:chromogram-cache
-EELAYER 26 0
+EELAYER 25 0
 EELAYER END
 $Descr A4 11693 8268
@@
 Text Notes 8175 550  0    40   ~ 8
 16 x 8 pixel matrix
+Text Label 1825 3050 0    40   ~ 0
+SCL
 Text Label 1825 3150 0    40   ~ 0
-SCL
-Text Label 1825 3050 0    40   ~ 0
 SDA
 Text Label 8400 1300 0    40   ~ 0
@@
 Text Label 1825 2650 0    40   ~ 0
 LDR1_PIN
-Text Label 4075 3050 2    40   ~ 0
+Text Label 4075 3150 2    40   ~ 0
 DAT_IN
 Text Label 1825 2750 0    40   ~ 0
@@
 	8375 4100 8875 4100
 Wire Wire Line
-	5950 5275 5950 5300
-Wire Wire Line
-	6450 5275 6450 5300
+	5950 5275 5950 5550
+Wire Wire Line
+	6450 5275 6450 5550
 Wire Wire Line
 	5950 5425 6150 5425
@@
 Connection ~ 6450 5425
 Wire Wire Line
-	6450 5850 6450 5975
-Wire Wire Line
-	6450 5975 5950 5975
+	6450 5975 6450 5850
+Wire Wire Line
+	4950 5975 6450 5975
 Wire Wire Line
 	5950 5975 5950 5850
 Wire Wire Line
-	5950 4775 5950 4950
-Wire Wire Line
-	5950 4775 6450 4775
-Wire Wire Line
-	6450 4775 6450 4950
+	5950 4775 5950 4975
+Wire Wire Line
+	4950 4775 6450 4775
+Wire Wire Line
+	6450 4775 6450 4975
 $Comp
 L chromogram:R R12
@@
 	4950 6425 4950 6575
 Wire Wire Line
-	4950 6875 4950 7025
+	4950 6875 4950 7150
 Wire Wire Line
 	4950 7450 4950 7625
@@
 Connection ~ 4950 7025
 Wire Wire Line
-	4950 6425 5450 6425
-Wire Wire Line
-	4950 7625 5450 7625
+	4950 6425 6450 6425
+Wire Wire Line
+	4950 7625 6450 7625
 $Comp
 L chromogram:R R13
@@
 	5450 6425 5450 6575
 Wire Wire Line
-	5450 6875 5450 7025
-Wire Wire Line
-	5450 7450 5450 7625
+	5450 6875 5450 7150
+Wire Wire Line
+	5450 7625 5450 7450
 Wire Wire Line
 	5450 7025 5550 7025
@@
 	5950 6425 5950 6575
 Wire Wire Line
-	5950 6875 5950 7025
-Wire Wire Line
-	5950 7450 5950 7625
+	5950 6875 5950 7150
+Wire Wire Line
+	5950 7625 5950 7450
 Wire Wire Line
 	5950 7025 6050 7025
@@
 	6450 6425 6450 6575
 Wire Wire Line
-	6450 6875 6450 7025
-Wire Wire Line
-	6450 7450 6450 7625
+	6450 6875 6450 7150
+Wire Wire Line
+	6450 7625 6450 7450
 Wire Wire Line
 	6450 7025 6550 7025
@@
 Text Label 2000 5600 0    40   ~ 0
 DTR
-Text Label 4075 3150 2    40   ~ 0
+Text Label 4075 3050 2    40   ~ 0
 CLK_IN
 $Comp
@@
 Wire Wire Line
 	10350 6350 10350 6375
-Wire Wire Line
-	5950 5425 5950 5550
-Wire Wire Line
-	6450 5425 6450 5550
-Wire Wire Line
-	4950 7025 4950 7150
-Wire Wire Line
-	5450 7025 5450 7150
-Wire Wire Line
-	5950 7025 5950 7150
-Wire Wire Line
-	6450 7025 6450 7150
-Wire Wire Line
-	5950 5300 5950 5425
-Wire Wire Line
-	6450 5300 6450 5425
-Wire Wire Line
-	6450 4950 6450 4975
-Wire Wire Line
-	5950 4950 5950 4975
 $Comp
 L chromogram:R R10
@@
 5V
 Wire Wire Line
-	4950 5275 4950 5300
-Wire Wire Line
-	5450 5275 5450 5300
+	4950 5275 4950 5550
+Wire Wire Line
+	5450 5275 5450 5550
 Wire Wire Line
 	4950 5425 5150 5425
@@
 	5450 5850 5450 5975
 Wire Wire Line
-	5450 5975 4950 5975
-Wire Wire Line
 	4950 5975 4950 5850
 Wire Wire Line
-	4950 4775 4950 4950
-Wire Wire Line
-	4950 4775 5450 4775
-Wire Wire Line
-	5450 4775 5450 4950
+	4950 4775 4950 4975
+Wire Wire Line
+	5450 4775 5450 4975
 $Comp
 L chromogram:SW-SPST-M S1
@@
 	5000 4950 4950 4950
 Connection ~ 4950 4950
-Wire Wire Line
-	4950 5425 4950 5550
-Wire Wire Line
-	5450 5425 5450 5550
-Wire Wire Line
-	4950 5300 4950 5425
-Wire Wire Line
-	5450 5300 5450 5425
-Wire Wire Line
-	5450 4950 5450 4975
-Wire Wire Line
-	4950 4950 4950 4975
-Wire Wire Line
-	5950 4775 5450 4775
 Connection ~ 5950 4775
 Connection ~ 5450 4775
-Wire Wire Line
-	5950 5975 5450 5975
 Connection ~ 5950 5975
 Connection ~ 5450 5975
@@
 Text Notes 1675 2700 2    40   ~ 0
 LDR
-Wire Wire Line
-	5450 6425 5950 6425
 Connection ~ 5450 6425
-Wire Wire Line
-	5950 6425 6450 6425
 Connection ~ 5950 6425
-Wire Wire Line
-	5450 7625 5950 7625
-Wire Wire Line
-	5950 7625 6450 7625
 Connection ~ 5950 7625
 Connection ~ 5450 7625
@@
 	800  2050 800  2150
 Wire Wire Line
-	800  2050 1100 2050
-Wire Wire Line
-	1100 2150 1100 2050
+	800  2050 2100 2050
+Wire Wire Line
+	1100 2050 1100 2150
 Connection ~ 1100 2050
-Wire Wire Line
-	1100 2050 2100 2050
 Wire Wire Line
 	800  2450 800  2725
@@
 NoConn ~ 4075 2450
 NoConn ~ 1825 3250
+Wire Wire Line
+	3800 1850 4075 1850
+Text Label 4075 1850 2    40   ~ 0
+GND
 $EndSCHEMATC

Commit message: WIP PCB layout
Connections:
- net labels added: LDR1, LDR2, LDR3, LDR4
- net labels removed: LDR1_PIN, LDR2_PIN, LDR3_PIN, LDR4_PIN
- wire segments 212 -> 230
