File: kicad/chromogram.sch (KiCad schematic (older format))
At the start: 22 parts, among them P2 OUT_CLK_DAT, U129 ESP-wroom-32

Commit message: almost done with PCB
Connections:
- net labels removed: RST
- wire segments 230 -> 229
Changed lines of the file:
@@
 F2 "5V" I L 2300 5950 40
 F3 "GND" I L 2300 6025 40
-F4 "RST" I L 2300 6100 40
 F5 "SDA" I L 2300 6175 40
 F6 "SCL" I L 2300 6250 40
@@
 	2000 6025 2300 6025
 Wire Wire Line
-	2300 6100 2000 6100
-Wire Wire Line
 	2000 6175 2300 6175
 Wire Wire Line
@@
 Text Label 2000 6025 0    40   ~ 0
 GND
-Text Label 2000 6100 0    40   ~ 0
-RST
 Text Label 2000 6175 0    40   ~ 0
 SDA
@@
 	3800 3150 4050 3150
 Wire Wire Line
-	4075 3250 3800 3250
+	4050 3250 3800 3250
 Wire Wire Line
 	2500 3650 2500 3925
@@
 Text Label 2600 3925 1    40   ~ 0
 IO13
-Text Label 4075 3250 2    40   ~ 0
+Text Label 4050 3250 2    40   ~ 0
 IO0
 Wire Wire Line

Commit message: modified diode footprints
Parts:
- added G1: LOGO_WL, chromogram_libs:Logo-WL3, symbol chromogram:LOGO_WL
- added G2: KiCad, chromogram_libs:KiCad-Logo2_6mm_SilkScreen, symbol chromogram:KiCad
- added G3: OSHW, chromogram_libs:OSHW_6mm, symbol chromogram:OSHW
- R10, R11, R12, R13, R14, R15, R24, R25: value 10K -> 10k
Changed lines of the file:
@@
 P 3150 5450
 F 0 "R24" H 3225 5300 40  0000 C CNN
-F 1 "10K" V 3157 5451 40  0000 C CNN
+F 1 "10k" V 3157 5451 40  0000 C CNN
 F 2 "chromogram_libs:r_0805" V 3080 5450 30  0001 C CNN
 F 3 "~" H 3150 5450 30  0000 C CNN
@@
 P 3650 5450
 F 0 "R25" H 3725 5300 40  0000 C CNN
-F 1 "10K" V 3657 5451 40  0000 C CNN
+F 1 "10k" V 3657 5451 40  0000 C CNN
 F 2 "chromogram_libs:r_0805" V 3580 5450 30  0001 C CNN
 F 3 "~" H 3650 5450 30  0000 C CNN
@@
 P 2150 7050
 F 0 "R12" H 2225 6900 40  0000 C CNN
-F 1 "10K" V 2157 7051 40  0000 C CNN
+F 1 "10k" V 2157 7051 40  0000 C CNN
 F 2 "chromogram_libs:r_0805" V 2080 7050 30  0001 C CNN
 F 3 "~" H 2150 7050 30  0000 C CNN
@@
 P 2650 7050
 F 0 "R13" H 2725 6900 40  0000 C CNN
-F 1 "10K" V 2657 7051 40  0000 C CNN
+F 1 "10k" V 2657 7051 40  0000 C CNN
 F 2 "chromogram_libs:r_0805" V 2580 7050 30  0001 C CNN
 F 3 "~" H 2650 7050 30  0000 C CNN
@@
 P 3150 7050
 F 0 "R14" H 3225 6900 40  0000 C CNN
-F 1 "10K" V 3157 7051 40  0000 C CNN
+F 1 "10k" V 3157 7051 40  0000 C CNN
 F 2 "chromogram_libs:r_0805" V 3080 7050 30  0001 C CNN
 F 3 "~" H 3150 7050 30  0000 C CNN
@@
 P 3650 7050
 F 0 "R15" H 3725 6900 40  0000 C CNN
-F 1 "10K" V 3657 7051 40  0000 C CNN
+F 1 "10k" V 3657 7051 40  0000 C CNN
 F 2 "chromogram_libs:r_0805" V 3580 7050 30  0001 C CNN
 F 3 "~" H 3650 7050 30  0000 C CNN
@@
 P 2150 5450
 F 0 "R10" H 2225 5300 40  0000 C CNN
-F 1 "10K" V 2157 5451 40  0000 C CNN
+F 1 "10k" V 2157 5451 40  0000 C CNN
 F 2 "chromogram_libs:r_0805" V 2080 5450 30  0001 C CNN
 F 3 "~" H 2150 5450 30  0000 C CNN
@@
 P 2650 5450
 F 0 "R11" H 2725 5300 40  0000 C CNN
-F 1 "10K" V 2657 5451 40  0000 C CNN
+F 1 "10k" V 2657 5451 40  0000 C CNN
 F 2 "chromogram_libs:r_0805" V 2580 5450 30  0001 C CNN
 F 3 "~" H 2650 5450 30  0000 C CNN
@@
 Text Label 5450 3525 0    40   ~ 0
 GND
+$Comp
+L chromogram:LOGO_WL G1
+U 1 1 5A4DA853
+P 8350 6700
+F 0 "G1" H 8350 6564 60  0001 C CNN
+F 1 "LOGO_WL" H 8350 6836 60  0001 C CNN
+F 2 "chromogram_libs:Logo-WL3" H 8350 6700 60  0001 C CNN
+F 3 "" H 8350 6700 60  0001 C CNN
+F 4 "Value" H 8350 6700 50  0001 C CNN "manf#"
+	1    8350 6700
+	1    0    0    -1
+$EndComp
+$Comp
+L chromogram:OSHW G3
+U 1 1 5A4DB491
+P 10850 7000
+F 0 "G3" H 10850 6950 40  0001 C CNN
+F 1 "OSHW" H 10850 7100 40  0001 C CNN
+F 2 "chromogram_libs:OSHW_6mm" H 10850 7000 60  0001 C CNN
+F 3 "" H 10850 7000 60  0000 C CNN
+F 4 "Value" H 10850 7000 50  0001 C CNN "manf#"
+	1    10850 7000
+	1    0    0    -1
+$EndComp
+$Comp
+L chromogram:KiCad G2
+U 1 1 5A5061ED
+P 9550 6850
+F 0 "G2" H 9550 6582 60  0001 C CNN
+F 1 "KiCad" H 9550 7118 60  0001 C CNN
+F 2 "chromogram_libs:KiCad-Logo2_6mm_SilkScreen" H 9550 6850 60  0001 C CNN
+F 3 "" H 9550 6850 60  0001 C CNN
+F 4 "Value" H 9550 6850 50  0001 C CNN "manf#"
+	1    9550 6850
+	1    0    0    -1
+$EndComp
 $EndSCHEMATC

Commit message: modified mounting holes
Parts:
- LDR1, LDR2, LDR3, LDR4: footprint chromogram_libs:r_0805_ldr -> Opto-Devices:Resistor_LDR_10x8.5_RM7.6
- R24, R25: footprint chromogram_libs:r_0805 -> chromogram_libs:r_0805_ldr
Changed lines of the file:
@@
 F 1 "470R" V 9025 650 40  0000 C CNN
 F 2 "chromogram_libs:r_0805" V 8955 650 30  0001 C CNN
-F 3 "~" H 9025 650 30  0000 C CNN
+F 3 "" H 9025 650 30  0000 C CNN
 	1    9025 650
 	0    -1   -1   0
@@
 F 0 "R24" H 3225 5300 40  0000 C CNN
 F 1 "10k" V 3157 5451 40  0000 C CNN
-F 2 "chromogram_libs:r_0805" V 3080 5450 30  0001 C CNN
-F 3 "~" H 3150 5450 30  0000 C CNN
+F 2 "chromogram_libs:r_0805_ldr" V 3080 5450 30  0001 C CNN
+F 3 "" H 3150 5450 30  0000 C CNN
 	1    3150 5450
 	1    0    0    -1
@@
 F 0 "R25" H 3725 5300 40  0000 C CNN
 F 1 "10k" V 3657 5451 40  0000 C CNN
-F 2 "chromogram_libs:r_0805" V 3580 5450 30  0001 C CNN
-F 3 "~" H 3650 5450 30  0000 C CNN
+F 2 "chromogram_libs:r_0805_ldr" V 3580 5450 30  0001 C CNN
+F 3 "" H 3650 5450 30  0000 C CNN
 	1    3650 5450
 	1    0    0    -1
@@
 F 1 "10k" V 2157 7051 40  0000 C CNN
 F 2 "chromogram_libs:r_0805" V 2080 7050 30  0001 C CNN
-F 3 "~" H 2150 7050 30  0000 C CNN
+F 3 "" H 2150 7050 30  0000 C CNN
 	1    2150 7050
 	1    0    0    -1
@@
 F 1 "10k" V 2657 7051 40  0000 C CNN
 F 2 "chromogram_libs:r_0805" V 2580 7050 30  0001 C CNN
-F 3 "~" H 2650 7050 30  0000 C CNN
+F 3 "" H 2650 7050 30  0000 C CNN
 	1    2650 7050
 	1    0    0    -1
@@
 F 1 "10k" V 3157 7051 40  0000 C CNN
 F 2 "chromogram_libs:r_0805" V 3080 7050 30  0001 C CNN
-F 3 "~" H 3150 7050 30  0000 C CNN
+F 3 "" H 3150 7050 30  0000 C CNN
 	1    3150 7050
 	1    0    0    -1
@@
 F 1 "10k" V 3657 7051 40  0000 C CNN
 F 2 "chromogram_libs:r_0805" V 3580 7050 30  0001 C CNN
-F 3 "~" H 3650 7050 30  0000 C CNN
+F 3 "" H 3650 7050 30  0000 C CNN
 	1    3650 7050
 	1    0    0    -1
@@
 F 1 "470R" V 9025 800 40  0000 C CNN
 F 2 "chromogram_libs:r_0805" V 8955 800 30  0001 C CNN
-F 3 "~" H 9025 800 30  0000 C CNN
+F 3 "" H 9025 800 30  0000 C CNN
 	1    9025 800
 	0    -1   -1   0
@@
 F 0 "LDR1" H 2175 6325 40  0000 L CNN
 F 1 "LDR" V 2150 6425 40  0000 L CNN
-F 2 "chromogram_libs:r_0805_ldr" V 2325 6475 50  0001 C CNN
+F 2 "Opto-Devices:Resistor_LDR_10x8.5_RM7.6" V 2325 6475 50  0001 C CNN
 F 3 "" H 2150 6425 50  0000 C CNN
 	1    2150 6475
@@
 F 0 "LDR2" H 2675 6325 40  0000 L CNN
 F 1 "LDR" V 2650 6425 40  0000 L CNN
-F 2 "chromogram_libs:r_0805_ldr" V 2825 6475 50  0001 C CNN
+F 2 "Opto-Devices:Resistor_LDR_10x8.5_RM7.6" V 2825 6475 50  0001 C CNN
 F 3 "" H 2650 6425 50  0000 C CNN
 	1    2650 6475
@@
 F 0 "LDR3" H 3175 6325 40  0000 L CNN
 F 1 "LDR" V 3150 6425 40  0000 L CNN
-F 2 "chromogram_libs:r_0805_ldr" V 3325 6475 50  0001 C CNN
+F 2 "Opto-Devices:Resistor_LDR_10x8.5_RM7.6" V 3325 6475 50  0001 C CNN
 F 3 "" H 3150 6425 50  0000 C CNN
 	1    3150 6475
@@
 F 0 "LDR4" H 3675 6325 40  0000 L CNN
 F 1 "LDR" V 3650 6425 40  0000 L CNN
-F 2 "chromogram_libs:r_0805_ldr" V 3825 6475 50  0001 C CNN
+F 2 "Opto-Devices:Resistor_LDR_10x8.5_RM7.6" V 3825 6475 50  0001 C CNN
 F 3 "" H 3650 6425 50  0000 C CNN
 	1    3650 6475
@@
 F 1 "10k" V 2157 5451 40  0000 C CNN
 F 2 "chromogram_libs:r_0805" V 2080 5450 30  0001 C CNN
-F 3 "~" H 2150 5450 30  0000 C CNN
+F 3 "" H 2150 5450 30  0000 C CNN
 	1    2150 5450
 	1    0    0    -1
@@
 F 1 "10k" V 2657 5451 40  0000 C CNN
 F 2 "chromogram_libs:r_0805" V 2580 5450 30  0001 C CNN
-F 3 "~" H 2650 5450 30  0000 C CNN
+F 3 "" H 2650 5450 30  0000 C CNN
 	1    2650 5450
 	1    0    0    -1

Commit message: added Gerbers
Parts:
- LDR1, LDR2, LDR3, LDR4: footprint Opto-Devices:Resistor_LDR_10x8.5_RM7.6 -> chromogram_libs:r_0805_ldr
- R24, R25: footprint chromogram_libs:r_0805_ldr -> chromogram_libs:r_0805
Changed lines of the file:
@@
 F 0 "R24" H 3225 5300 40  0000 C CNN
 F 1 "10k" V 3157 5451 40  0000 C CNN
-F 2 "chromogram_libs:r_0805_ldr" V 3080 5450 30  0001 C CNN
+F 2 "chromogram_libs:r_0805" V 3080 5450 30  0001 C CNN
 F 3 "" H 3150 5450 30  0000 C CNN
 	1    3150 5450
@@
 F 0 "R25" H 3725 5300 40  0000 C CNN
 F 1 "10k" V 3657 5451 40  0000 C CNN
-F 2 "chromogram_libs:r_0805_ldr" V 3580 5450 30  0001 C CNN
+F 2 "chromogram_libs:r_0805" V 3580 5450 30  0001 C CNN
 F 3 "" H 3650 5450 30  0000 C CNN
 	1    3650 5450
@@
 F 0 "LDR1" H 2175 6325 40  0000 L CNN
 F 1 "LDR" V 2150 6425 40  0000 L CNN
-F 2 "Opto-Devices:Resistor_LDR_10x8.5_RM7.6" V 2325 6475 50  0001 C CNN
+F 2 "chromogram_libs:r_0805_ldr" V 2325 6475 50  0001 C CNN
 F 3 "" H 2150 6425 50  0000 C CNN
 	1    2150 6475
@@
 F 0 "LDR2" H 2675 6325 40  0000 L CNN
 F 1 "LDR" V 2650 6425 40  0000 L CNN
-F 2 "Opto-Devices:Resistor_LDR_10x8.5_RM7.6" V 2825 6475 50  0001 C CNN
+F 2 "chromogram_libs:r_0805_ldr" V 2825 6475 50  0001 C CNN
 F 3 "" H 2650 6425 50  0000 C CNN
 	1    2650 6475
@@
 F 0 "LDR3" H 3175 6325 40  0000 L CNN
 F 1 "LDR" V 3150 6425 40  0000 L CNN
-F 2 "Opto-Devices:Resistor_LDR_10x8.5_RM7.6" V 3325 6475 50  0001 C CNN
+F 2 "chromogram_libs:r_0805_ldr" V 3325 6475 50  0001 C CNN
 F 3 "" H 3150 6425 50  0000 C CNN
 	1    3150 6475
@@
 F 0 "LDR4" H 3675 6325 40  0000 L CNN
 F 1 "LDR" V 3650 6425 40  0000 L CNN
-F 2 "Opto-Devices:Resistor_LDR_10x8.5_RM7.6" V 3825 6475 50  0001 C CNN
+F 2 "chromogram_libs:r_0805_ldr" V 3825 6475 50  0001 C CNN
 F 3 "" H 3650 6425 50  0000 C CNN
 	1    3650 6475

Commit message: added Gerbers
Connections:
- net labels added: CLK, CMD, IO12, IO14, IO16, IO2, IO22, IO23, IO27, IO4, SD2, SD3, SDI, SDO, SENSOR_VN, SENSOR_VP
Changed lines of the file:
@@
 Text Notes 8175 550  0    40   ~ 8
 16 x 8 pixel matrix
-Text Label 1850 2650 0    40   ~ 0
+Text Label 1850 2450 0    40   ~ 0
 SCL
-Text Label 1850 2750 0    40   ~ 0
+Text Label 1850 2550 0    40   ~ 0
 SDA
 Text Label 8400 1300 0    40   ~ 0
@@
 Text Label 8325 650  0    40   ~ 0
 DAT_IN
-Text Label 1850 3150 0    40   ~ 0
+Text Label 1850 2950 0    40   ~ 0
 LDR1
-Text Label 4050 3150 2    40   ~ 0
+Text Label 4050 2950 2    40   ~ 0
 DAT_IN
-Text Label 1850 2850 0    40   ~ 0
+Text Label 1850 2650 0    40   ~ 0
 LDR2
-Text Label 1850 2950 0    40   ~ 0
+Text Label 1850 2750 0    40   ~ 0
 LDR3
 Text Label 8475 1850 0    40   ~ 0
@@
 	3650 6775 3750 6775
 Connection ~ 3650 6775
-Text Label 1850 3050 0    40   ~ 0
+Text Label 1850 2850 0    40   ~ 0
 LDR4
 $Comp
@@
 	2100 2150 1850 2150
 Wire Wire Line
+	2100 2650 1850 2650
+Wire Wire Line
+	1850 2750 2100 2750
+Wire Wire Line
 	2100 2850 1850 2850
 Wire Wire Line
 	1850 2950 2100 2950
 Wire Wire Line
-	2100 3050 1850 3050
-Wire Wire Line
-	1850 3150 2100 3150
-Wire Wire Line
-	2100 2650 1850 2650
-Wire Wire Line
-	1850 2750 2100 2750
+	2100 2450 1850 2450
+Wire Wire Line
+	1850 2550 2100 2550
 Wire Wire Line
 	4050 1950 3800 1950
@@
 	4050 2350 3800 2350
 Wire Wire Line
+	4050 2450 3800 2450
+Wire Wire Line
+	3800 2550 4050 2550
+Wire Wire Line
 	4050 2650 3800 2650
 Wire Wire Line
@@
 Wire Wire Line
 	3800 2950 4050 2950
-Wire Wire Line
-	4050 3050 3800 3050
-Wire Wire Line
-	3800 3150 4050 3150
 Wire Wire Line
 	4050 3250 3800 3250
@@
 Text Label 2500 3925 1    40   ~ 0
 GND
-NoConn ~ 3800 2550
+NoConn ~ 3800 3150
 Text Label 4050 1950 2    40   ~ 0
 GND
@@
 Text Label 5450 2000 0    40   ~ 0
 DTR
-Text Label 4050 3050 2    40   ~ 0
+Text Label 4050 2850 2    40   ~ 0
 CLK_IN
 $Comp
@@
 Connection ~ 3150 5725
 Connection ~ 2650 5725
+Text Label 4050 2450 2    40   ~ 0
+SW_E
+Text Label 4050 2550 2    40   ~ 0
+SW_I
 Text Label 4050 2650 2    40   ~ 0
-SW_E
+SW_D
 Text Label 4050 2750 2    40   ~ 0
-SW_I
-Text Label 4050 2850 2    40   ~ 0
-SW_D
-Text Label 4050 2950 2    40   ~ 0
 SW_M
 Wire Notes Line
-	4125 2650 4175 2650
-Wire Notes Line
-	4175 2650 4175 2950
+	4125 2450 4175 2450
+Wire Notes Line
+	4175 2450 4175 2750
+Wire Notes Line
+	4175 2750 4125 2750
+Wire Notes Line
+	4125 2850 4175 2850
+Wire Notes Line
+	4175 2850 4175 2950
 Wire Notes Line
 	4175 2950 4125 2950
 Wire Notes Line
-	4125 3050 4175 3050
-Wire Notes Line
-	4175 3050 4175 3150
-Wire Notes Line
-	4175 3150 4125 3150
-Wire Notes Line
-	1750 2650 1700 2650
-Wire Notes Line
-	1700 2650 1700 2750
-Wire Notes Line
-	1700 2750 1750 2750
-Text Notes 4175 2700 0    40   ~ 0
+	1750 2450 1700 2450
+Wire Notes Line
+	1700 2450 1700 2550
+Wire Notes Line
+	1700 2550 1750 2550
+Text Notes 4175 2500 0    40   ~ 0
 BUTTONS
-Text Notes 4175 3100 0    40   ~ 0
+Text Notes 4175 2900 0    40   ~ 0
 LED CLK/DAT
-Text Notes 1675 2700 2    40   ~ 0
+Text Notes 1675 2500 2    40   ~ 0
 I2C
 Wire Notes Line
@@
 SERIAL
 Wire Notes Line
-	1750 3150 1700 3150
-Wire Notes Line
-	1700 3150 1700 2850
-Wire Notes Line
-	1700 2850 1750 2850
-Text Notes 1675 2900 2    40   ~ 0
+	1750 2950 1700 2950
+Wire Notes Line
+	1700 2950 1700 2650
+Wire Notes Line
+	1700 2650 1750 2650
+Text Notes 1675 2700 2    40   ~ 0
 LDR
 Connection ~ 2650 6175
@@
 NoConn ~ 2100 2250
 NoConn ~ 2100 2350
-NoConn ~ 2100 2450
-NoConn ~ 2100 2550
 NoConn ~ 3400 3650
 NoConn ~ 3200 3650
@@
 NoConn ~ 3800 2050
 NoConn ~ 3800 2150
-NoConn ~ 3800 2450
+NoConn ~ 3800 3050
 NoConn ~ 2100 3250
 Wire Wire Line
@@
 	1    0    0    -1
 $EndComp
+NoConn ~ 2100 3150
+NoConn ~ 2100 3050
+Text Label 2100 2250 2    40   ~ 0
+SENSOR_VP
+Text Label 2100 2350 2    40   ~ 0
+SENSOR_VN
+Text Label 2100 3050 2    40   ~ 0
+IO27
+Text Label 2100 3150 2    40   ~ 0
+IO14
+Text Label 2100 3250 2    40   ~ 0
+IO12
+Text Label 2700 3650 3    40   ~ 0
+SD2
+Text Label 2800 3650 3    40   ~ 0
+SD3
+Text Label 2900 3650 3    40   ~ 0
+CMD
+Text Label 3000 3650 3    40   ~ 0
+CLK
+Text Label 3100 3650 3    40   ~ 0
+SDO
+Text Label 3200 3650 3    40   ~ 0
+SDI
+Text Label 3400 3650 3    40   ~ 0
+IO2
+Text Label 3800 3150 0    40   ~ 0
+IO4
+Text Label 3800 3050 0    40   ~ 0
+IO16
+Text Label 3800 2150 0    40   ~ 0
+IO22
+Text Label 3800 2050 0    40   ~ 0
+IO23
 $EndSCHEMATC
