File: kicad/chromogram.kicad_pcb (KiCad board)
At the start: 2 copper layers, 162.6 x 142.2 mm, 217 parts, among them SW2 SW_L, SW3 SW_R, U1 APA102, U10 APA102, U100 APA102, U101 APA102, U102 APA102, U103 APA102, U104 APA102, U105 APA102, U106 APA102, U107 APA102, U108 APA102, U109 APA102, U11 APA102, U110 APA102, U111 APA102, U112 APA102, U113 APA102, U114 APA102, U115 APA102, U116 APA102, U117 APA102, U118 APA102, U119 APA102, U12 APA102, U120 APA102, U121 APA102, U122 APA102, U123 APA102, U124 APA102, U125 APA102, U126 APA102, U127 APA102, U128 APA102, U13 APA102, U130 DS3231N, U14 APA102, U15 APA102, U16 APA102, U17 APA102, U18 APA102, U19 APA102, U2 APA102, U20 APA102, U21 APA102, U22 APA102, U23 APA102, U24 APA102, U25 APA102, U26 APA102, U27 APA102, U28 APA102, U29 APA102, U3 APA102, U30 APA102, U31 APA102, U32 APA102, U33 APA102, U34 APA102, U35 APA102, U36 APA102, U37 APA102, U38 APA102, U39 APA102, U4 APA102, U40 APA102, U41 APA102, U42 APA102, U43 APA102, U44 APA102, U45 APA102, U46 APA102, U47 APA102, U48 APA102, U49 APA102, U5 APA102, U50 APA102, U51 APA102, U52 APA102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

Commit message: schematic dev in progress
Parts:
- removed C21, C28: 100n, chromogram_libs:c_0805
- removed C24, C25, C26, C27: 47u, chromogram_libs:c_2917
- removed D1: SMBJ5339B, chromogram_libs:diode-DO214AA
- removed F1: miniSMDC200F/16, chromogram_libs:f_1812
- added U129: ESP-wroom-32, chromogram_libs:esp_wroom_32, B.Cu at (127.0, 176.5)
Connections:
- net /BAT renamed /rtc_ds3231/BAT
- net 5V renamed /5V
- U128 pad 5: /CLK_OUT -> (no net)
- U128 pad 6: /DAT_OUT -> (no net)
- U130 pad 4: /RESET -> (no net)

Commit message: schematic WIP
Parts:
- moved U129 109.2 mm to (127.0, 67.3), turned to 180 degrees

Commit message: WIP schematic
Parts:
- removed SW2: SW_L, chromogram_libs:SW_SMD
- removed SW3: SW_R, chromogram_libs:SW_SMD
- added C17: 10uF/25V, chromogram_libs:c_2917, B.Cu at (299.7, 86.4)
- added C18: 22uF/25V, chromogram_libs:c_2917, B.Cu at (306.1, 78.7)
- added C19: 1nF, chromogram_libs:c_0805, B.Cu at (349.9, 87.6)
- added C20: 1nF, chromogram_libs:c_0805, B.Cu at (58.4, 16.5)
- added C21: 1nF, chromogram_libs:c_0805, B.Cu at (134.6, 16.5)
- added C23: 10uF/25V, chromogram_libs:c_2917, B.Cu at (343.5, 76.2)
- added C24: 100nF, chromogram_libs:c_0805, B.Cu at (348.0, 76.2)
- added C25: 10uF/25V, chromogram_libs:c_2917, B.Cu at (338.5, 76.2)
- added C26: 100nF, chromogram_libs:c_0805, B.Cu at (348.6, 71.1)
- added C27: 100uF/6V3, chromogram_libs:c_2917, B.Cu at (170.8, 7.62)
- added C28: 1uF/10V, chromogram_libs:c_0805, B.Cu at (171.4, 3.17)
- added D1: 1N5819, chromogram_libs:D_SOD-123, B.Cu at (323.2, 78.7)
- added D2: LED_PWR, chromogram_libs:LED-0805, B.Cu at (292.1, 81.3)
- added D3: VESD05A1B, chromogram_libs:D_SOD-123, B.Cu at (328.9, 81.3)
- added D4: VESD05A1B, chromogram_libs:D_SOD-123, B.Cu at (328.9, 78.7)
- added HB45: hole_baffle, chromogram_libs:MtgHole_3mm, F.Cu at (49.5, 2.54)
- added HB46: hole_baffle, chromogram_libs:MtgHole_3mm, F.Cu at (204.5, 2.54)
- added HB47: hole_baffle, chromogram_libs:MtgHole_3mm, F.Cu at (50.8, 36.8)
- added HB48: hole_baffle, chromogram_libs:MtgHole_3mm, F.Cu at (203.2, 36.8)
- added HB49: hole_baffle, chromogram_libs:MtgHole_3mm, F.Cu at (50.8, 189.2)
- added HB50: hole_baffle, chromogram_libs:MtgHole_3mm, F.Cu at (203.2, 189.2)
- added HB51: hole_baffle, chromogram_libs:MtgHole_3mm, F.Cu at (49.5, 223.5)
- added HB52: hole_baffle, chromogram_libs:MtgHole_3mm, F.Cu at (204.5, 223.5)
- added JP1: PWR_LED_EN, chromogram_libs:R_0402, B.Cu at (292.1, 86.4)
- added P1: USB_micro, chromogram_libs:USB_Micro-B_Molex-105017-0001, B.Cu at (47.6, 26.7)
- added P2: OUT_CLK_DAT, chromogram_libs:Pin_Header_Straight_1x02, F.Cu at (50.8, 180.3)
- added Q1: DDC114TU, chromogram_libs:SOT-363_SC-70-6, B.Cu at (348.0, 83.8)
- added R16: 470R, chromogram_libs:r_0805, B.Cu at (58.4, 19.7)
- added R18: 470R, chromogram_libs:r_0805, B.Cu at (134.6, 19.7)
- added R19: 0R NC, chromogram_libs:r_0805, B.Cu at (360.7, 83.2)
- added R20: 0R NC, chromogram_libs:r_0805, B.Cu at (358.1, 83.2)
- added R21: 0R, chromogram_libs:r_0805, B.Cu at (355.6, 83.2)
- added R22: 470R, chromogram_libs:r_0805, B.Cu at (353.1, 83.2)
- added R23: 0R, chromogram_libs:r_0805, B.Cu at (353.1, 87.6)
- added R24: 10K, chromogram_libs:r_0805, B.Cu at (88.9, 16.5)
- added R25: 10K, chromogram_libs:r_0805, B.Cu at (73.7, 16.5)
- added R3: 10k, chromogram_libs:r_0805, B.Cu at (347.3, 87.6)
- added R4: 2k, chromogram_libs:r_0805, B.Cu at (294.6, 81.3)
- added S1: SW-ENTER, chromogram_libs:SW_SMD, B.Cu at (119.4, 8.89)
- added S2: SW-INC, chromogram_libs:SW_SMD, B.Cu at (104.1, 8.89)
- added S3: EN, chromogram_libs:SW_SMD, B.Cu at (58.4, 8.89)
- added S4: BOOT, chromogram_libs:SW_SMD, B.Cu at (134.6, 8.89)
- added S5: SW-DEC, chromogram_libs:SW_SMD, B.Cu at (88.9, 8.89)
- added S6: SW-MODE, chromogram_libs:SW_SMD, B.Cu at (73.7, 8.89)
- added U131: AP1117-15, chromogram_libs:SOT-223-3_TabPin2, B.Cu at (299.7, 78.7)
- added U132: CP2102N-A01-GQFN28, chromogram_libs:QFN-28-1EP_5x5mm_Pitch0.5mm, B.Cu at (355.6, 76.2)
- C13: value C2 -> 100nF
- C22: value 100n -> 100nF
- moved BT1 126.4 mm to (195.6, 18.4), turned to 90 degrees
- moved R10 118.4 mm to (119.4, 16.5), turned to 0 degrees
- moved R7 108.8 mm to (173.4, 13.3), turned to 90 degrees
- moved R6 107.3 mm to (175.9, 13.3), turned to 90 degrees
- moved R9 105.8 mm to (178.4, 13.3), turned to 90 degrees
- moved R8 104.4 mm to (181.0, 13.3), turned to 90 degrees
- moved R11 104.0 mm to (104.8, 16.5), turned to 0 degrees
- moved U130 95.8 mm to (177.2, 21.6), turned to 270 degrees
- moved C22 86.4 mm to (177.2, 29.2), turned to 270 degrees
- moved U129 61.1 mm to (151.8, 11.4)
- turned R1 to 90 degrees
- turned R2 to 90 degrees
Connections:
- R1 pad 1: (no net) -> /DAT_IN
- R10 pad 1: /SW_L -> /SW_E
- R11 pad 1: /SW_R -> /SW_I
- R2 pad 1: (no net) -> /CLK_IN
- U128 pad 5: (no net) -> /CLK_OUT
- U128 pad 6: (no net) -> /DAT_OUT
- U129 pad 1: (no net) -> GND
- U129 pad 10: (no net) -> /LDR3_PIN
- U129 pad 11: (no net) -> /LDR4_PIN
- U129 pad 12: (no net) -> /SDA
- U129 pad 13: (no net) -> /SCL
- U129 pad 14: (no net) -> Net-(J5-Pad1)
- U129 pad 15: (no net) -> GND
- U129 pad 16: (no net) -> /IO13
- U129 pad 17: (no net) -> Net-(J6-Pad1)
- U129 pad 18: (no net) -> Net-(J7-Pad1)
- U129 pad 19: (no net) -> Net-(J8-Pad1)
- U129 pad 2: (no net) -> /3V3
- U129 pad 20: (no net) -> Net-(J9-Pad1)
- U129 pad 21: (no net) -> Net-(J10-Pad1)
- U129 pad 22: (no net) -> Net-(J11-Pad1)
- U129 pad 23: (no net) -> /IO15
- U129 pad 24: (no net) -> Net-(J12-Pad1)
- U129 pad 25: Net-(U129-Pad25) -> /IO0
- U129 pad 26: (no net) -> /CLK_IN
- U129 pad 27: (no net) -> /DAT_IN
- U129 pad 28: (no net) -> /SW_M
- U129 pad 29: (no net) -> /SW_D
- U129 pad 3: (no net) -> /EN
- U129 pad 30: (no net) -> /SW_I
- U129 pad 31: (no net) -> /SW_E
- U129 pad 33: (no net) -> Net-(J13-Pad1)
- U129 pad 34: (no net) -> /RXD0
- U129 pad 35: (no net) -> /TXD0
- U129 pad 36: (no net) -> Net-(J14-Pad1)
- U129 pad 37: (no net) -> Net-(J15-Pad1)
- U129 pad 38: (no net) -> GND
- U129 pad 4: (no net) -> Net-(J1-Pad1)
- U129 pad 5: (no net) -> Net-(J2-Pad1)
- U129 pad 6: (no net) -> Net-(J3-Pad1)
- U129 pad 7: (no net) -> Net-(J4-Pad1)
- U129 pad 8: (no net) -> /LDR1_PIN
- U129 pad 9: (no net) -> /LDR2_PIN
Routing:
- net GND: track 2030.3 -> 2253.9 mm, vias 0 -> 8
- net /5V: track 1800.5 -> 1842.8 mm
- net /CI_A: track 0.00 -> 10.4 mm, vias 0 -> 1
- net /CLK_OUT: track 0.00 -> 8.47 mm
- net /DI_A: track 0.00 -> 5.94 mm, vias 0 -> 1
- net /DAT_OUT: track 0.00 -> 5.47 mm
- net /LDR2_PIN: track 0.00 -> 4.43 mm
- net /LDR4_PIN: track 0.00 -> 4.43 mm
- net /LDR1_PIN: track 0.00 -> 4.43 mm
- net /LDR3_PIN: track 0.00 -> 4.43 mm

Commit message: WIP schematic
Parts:
- moved D4 281.3 mm to (52.7, 25.4), turned to 270 degrees
- moved D3 279.3 mm to (55.2, 25.4), turned to 270 degrees
- moved D1 273.8 mm to (54.0, 29.2), turned to 0 degrees
- moved C25 253.6 mm to (89.5, 27.9)
- moved U132 251.9 mm to (108.6, 26.7)
- moved C23 251.1 mm to (97.2, 27.9)
- moved C24 249.8 mm to (102.9, 27.9)
- moved C17 247.7 mm to (59.1, 27.9), turned to 270 degrees
- moved C26 247.0 mm to (106.7, 21.6)
- moved Q1 244.9 mm to (108.6, 32.4)
- moved R23 244.9 mm to (113.7, 36.2)
- moved R3 244.2 mm to (108.6, 36.2)
- moved C19 244.2 mm to (111.1, 36.2)
- moved R19 241.5 mm to (123.8, 36.2)
- moved R21 241.5 mm to (118.7, 36.2)
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Other:
- board size 162.6 x 142.2 mm -> 162.6 x 228.6 mm

Commit message: making progress on PCB
Parts:
- removed HB51, HB52: hole_baffle, chromogram_libs:MtgHole_3mm
- added HB48: hole_baffle, chromogram_libs:MtgHole_3mm, F.Cu at (162.6, 37.5)
- added HB48: hole_baffle, chromogram_libs:MtgHole_3mm, F.Cu at (152.4, 80.6)
- added HB48: hole_baffle, chromogram_libs:MtgHole_3mm, F.Cu at (142.2, 80.6)
- added HB48: hole_baffle, chromogram_libs:MtgHole_3mm, F.Cu at (132.1, 80.6)
- added HB48: hole_baffle, chromogram_libs:MtgHole_3mm, F.Cu at (121.9, 80.6)
- added HB48: hole_baffle, chromogram_libs:MtgHole_3mm, F.Cu at (111.8, 80.6)
- added HB48: hole_baffle, chromogram_libs:MtgHole_3mm, F.Cu at (101.6, 80.6)
- added HB48: hole_baffle, chromogram_libs:MtgHole_3mm, F.Cu at (91.4, 80.6)
- added HB48: hole_baffle, chromogram_libs:MtgHole_3mm, F.Cu at (152.4, 37.5)
- added HB48: hole_baffle, chromogram_libs:MtgHole_3mm, F.Cu at (142.2, 37.5)
- added HB48: hole_baffle, chromogram_libs:MtgHole_3mm, F.Cu at (91.4, 37.5)
- added HB48: hole_baffle, chromogram_libs:MtgHole_3mm, F.Cu at (101.6, 37.5)
- added HB48: hole_baffle, chromogram_libs:MtgHole_3mm, F.Cu at (111.8, 37.5)
- added HB48: hole_baffle, chromogram_libs:MtgHole_3mm, F.Cu at (121.9, 37.5)
- added HB48: hole_baffle, chromogram_libs:MtgHole_3mm, F.Cu at (132.1, 37.5)
- added HB48: hole_baffle, chromogram_libs:MtgHole_3mm, F.Cu at (162.6, 80.6)
- moved U132 45.7 mm to (62.9, 26.7)
- moved C24 43.9 mm to (60.3, 17.1), turned to 90 degrees
- moved C26 41.5 mm to (65.4, 17.1)
- moved C23 41.2 mm to (56.5, 21.0), turned to 0 degrees
- moved JP1 35.1 mm to (100.1, 29.8), turned to 180 degrees
- moved D2 31.9 mm to (97.2, 29.8), turned to 0 degrees
- moved C17 31.3 mm to (90.2, 24.1)
- moved R4 28.6 mm to (94.0, 29.8), turned to 90 degrees
- moved U131 26.4 mm to (96.5, 22.9)
- moved R23 23.9 mm to (134.6, 24.8), turned to 0 degrees
- moved C18 21.9 mm to (103.5, 24.1)
- moved C25 21.5 mm to (69.2, 21.0), turned to 180 degrees
- moved R21 21.1 mm to (134.6, 22.2), turned to 0 degrees
- moved HB31 20.3 mm to (71.1, 59.7)
- moved HB32 20.3 mm to (71.1, 77.5)
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Connections:
- net /esp_pwr_uart/USB_DN renamed /esp_pwr_uart/USB_D-
- net /esp_pwr_uart/USB_DP renamed /esp_pwr_uart/USB_D+
- U129 pad 12: /SDA -> /SCL
- U129 pad 13: /SCL -> /SDA
- U129 pad 26: /CLK_IN -> /DAT_IN
- U129 pad 27: /DAT_IN -> /CLK_IN
- U129 pad 32: (no net) -> Net-(U129-Pad32)
Routing:
- net /3V3: track 0.00 -> 215.2 mm, vias 0 -> 2
- net /5V: track 1842.8 -> 2035.1 mm, vias 0 -> 3
- net /EN: track 0.00 -> 175.1 mm, vias 0 -> 3
- net GND: track 2253.9 -> 2397.3 mm, vias 8 -> 10
- net /SW_M: track 0.00 -> 87.8 mm, vias 0 -> 2
- net /esp_pwr_uart/RTS: track 0.00 -> 86.6 mm, vias 0 -> 2
- net /esp_pwr_uart/RXD: track 0.00 -> 84.6 mm, vias 0 -> 2
- net Net-(R22-Pad2): track 0.00 -> 84.5 mm, vias 0 -> 2
- net /DTR: track 0.00 -> 78.9 mm, vias 0 -> 2
- net /SW_D: track 0.00 -> 75.1 mm, vias 0 -> 2
- net /esp_pwr_uart/CTS: track 0.00 -> 72.6 mm
- net /SW_I: track 0.00 -> 59.3 mm, vias 0 -> 2
- net /SW_E: track 0.00 -> 43.6 mm, vias 0 -> 2
- net /IO0: track 0.00 -> 34.6 mm
- net /rtc_ds3231/BAT: track 0.00 -> 32.5 mm
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Other:
- board size 162.6 x 228.6 mm -> 162.6 x 195.6 mm
- net class 8 mil added: clearance 0.0381, trace_width 0.1524, via_dia 0.889, via_drill 0.635
- net class Default: clearance 0.254 -> 0.1016
- rule trace_clearance: 0.254 -> 0.1016
- rule trace_min: 0.254 -> 0.08

Commit message: WIP PCB layout
Parts:
- removed the HB48 at (162.6, 37.5)
- removed the HB48 at (152.4, 80.6)
- removed the HB48 at (142.2, 80.6)
- removed the HB48 at (132.1, 80.6)
- removed the HB48 at (121.9, 80.6)
- removed the HB48 at (111.8, 80.6)
- removed the HB48 at (101.6, 80.6)
- removed the HB48 at (91.4, 80.6)
- removed the HB48 at (152.4, 37.5)
- removed the HB48 at (142.2, 37.5)
- removed the HB48 at (91.4, 37.5)
- removed the HB48 at (101.6, 37.5)
- removed the HB48 at (111.8, 37.5)
- removed the HB48 at (121.9, 37.5)
- removed the HB48 at (132.1, 37.5)
- removed the HB48 at (162.6, 80.6)
- added HB51: hole_baffle, chromogram_libs:MtgHole_3mm, F.Cu at (91.4, 98.4)
- added HB52: hole_baffle, chromogram_libs:MtgHole_3mm, F.Cu at (162.6, 98.4)
- added HB53: hole_baffle, chromogram_libs:MtgHole_3mm, F.Cu at (162.6, 169.5)
- added HB54: hole_baffle, chromogram_libs:MtgHole_3mm, F.Cu at (91.4, 169.5)
- added J1: CLK_IN, chromogram_libs:1pin, F.Cu at (91.4, 37.5)
- added J10: DAT_IN, chromogram_libs:1pin, F.Cu at (101.6, 80.6)
- added J11: LDR1, chromogram_libs:1pin, F.Cu at (111.8, 80.6)
- added J12: LDR2, chromogram_libs:1pin, F.Cu at (162.6, 80.6)
- added J13: LDR3, chromogram_libs:1pin, F.Cu at (152.4, 80.6)
- added J14: LDR4, chromogram_libs:1pin, F.Cu at (121.9, 80.6)
- added J15: 5V, chromogram_libs:1pin, F.Cu at (142.2, 80.6)
- added J16: GND, chromogram_libs:1pin, F.Cu at (132.1, 80.6)
- added J2: DAT_IN, chromogram_libs:1pin, F.Cu at (101.6, 37.5)
- added J3: LDR1, chromogram_libs:1pin, F.Cu at (111.8, 37.5)
- added J4: LDR2, chromogram_libs:1pin, F.Cu at (162.6, 37.5)
- added J5: LDR3, chromogram_libs:1pin, F.Cu at (152.4, 37.5)
- added J6: LDR4, chromogram_libs:1pin, F.Cu at (121.9, 37.5)
- added J7: 5V, chromogram_libs:1pin, F.Cu at (142.2, 37.5)
- added J8: GND, chromogram_libs:1pin, F.Cu at (132.1, 37.5)
- added J9: CLK_IN, chromogram_libs:1pin, F.Cu at (91.4, 80.6)
- moved JP1 15.9 mm to (84.5, 26.7), turned to 90 degrees
- moved C21 11.2 mm to (127.0, 5.71), turned to 0 degrees
- moved D2 10.6 mm to (87.0, 26.7), turned to 90 degrees
- moved C17 8.84 mm to (81.9, 21.0), turned to 0 degrees
- moved R4 4.49 mm to (90.8, 26.7)
- moved R14 2.54 mm to (193.0, 176.5), turned to 180 degrees
- moved R15 2.54 mm to (61.0, 176.5), turned to 180 degrees
- moved P1 1.42 mm to (48.3, 26.7)
- moved LDR3 0.64 mm to (193.0, 181.0), turned to 0 degrees
- moved LDR4 0.64 mm to (61.0, 181.0)
- moved P2 0.63 mm to (50.8, 181.0)
- turned C22 to 270 degrees
- turned LDR1 to 180 degrees
- turned R12 to 0 degrees
Connections:
- LDR1 pad 2: /LDR1_PIN -> /LDR1
- LDR2 pad 2: /LDR2_PIN -> /LDR2
- LDR3 pad 2: /LDR3_PIN -> /LDR3
- LDR4 pad 2: /LDR4_PIN -> /LDR4
- P1 pad 4: (no net) -> Net-(P1-Pad4)
- R12 pad 1: /LDR1_PIN -> /LDR1
- R13 pad 1: /LDR2_PIN -> /LDR2
- R14 pad 1: /LDR3_PIN -> /LDR3
- R15 pad 1: /LDR4_PIN -> /LDR4
- U129 pad 10: /LDR3_PIN -> /LDR2
- U129 pad 11: /LDR4_PIN -> /LDR3
- U129 pad 12: /SCL -> /LDR4
- U129 pad 13: /SDA -> /LDR1
- U129 pad 8: /LDR1_PIN -> /SCL
- U129 pad 9: /LDR2_PIN -> /SDA
- U130 pad 4: (no net) -> /RST
- U132 pad 1: (no net) -> /esp_pwr_uart/DCD
- U132 pad 10: (no net) -> Net-(U132-Pad10)
- U132 pad 11: (no net) -> /esp_pwr_uart/ACTIVE
- U132 pad 12: (no net) -> Net-(U132-Pad12)
- U132 pad 13: (no net) -> Net-(U132-Pad13)
- U132 pad 14: (no net) -> Net-(U132-Pad14)
- U132 pad 15: (no net) -> Net-(U132-Pad15)
- U132 pad 16: (no net) -> Net-(U132-Pad16)
- U132 pad 17: (no net) -> Net-(U132-Pad17)
- U132 pad 18: (no net) -> Net-(U132-Pad18)
- U132 pad 19: (no net) -> Net-(U132-Pad19)
- U132 pad 2: (no net) -> /esp_pwr_uart/RI
- U132 pad 20: (no net) -> Net-(U132-Pad20)
- U132 pad 21: (no net) -> Net-(U132-Pad21)
- U132 pad 22: (no net) -> Net-(U132-Pad22)
- U132 pad 27: (no net) -> /esp_pwr_uart/DSR
- U132 pad 9: (no net) -> Net-(U132-Pad9)
Routing:
- net GND: track 2397.3 -> 2851.4 mm, vias 10 -> 8
- net /LDR4: track 0.00 -> 275.6 mm
- net /5V: track 2035.1 -> 2292.2 mm, vias 3 -> 6
- net /LDR3: track 0.00 -> 224.8 mm
- net /LDR1: track 0.00 -> 170.4 mm, vias 0 -> 1
- net /DAT_IN: track 2.50 -> 158.9 mm, vias 0 -> 4
- net /CLK_IN: track 2.50 -> 151.5 mm, vias 0 -> 4
- net /LDR2: track 0.00 -> 110.1 mm, vias 0 -> 1
- net /rtc_ds3231/BAT: track 32.5 -> 67.0 mm, vias 0 -> 2
- net /EN: track 175.1 -> 184.8 mm
- net /LDR2_PIN: track 6.93 -> 0.00 mm
- net /LDR4_PIN: track 6.93 -> 0.00 mm
- net /LDR1_PIN: track 6.93 -> 0.00 mm
- net /LDR3_PIN: track 6.93 -> 0.00 mm
- net /3V3: track 215.2 -> 218.6 mm, vias 2 -> 15
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- added copper zone on B.Cu, net /3V3
- added copper zone on F.Cu, net /3V3
- added copper zone on F.Cu, net /5V
- added copper zone on B.Cu, net GND
Other:
- board size 162.6 x 195.6 mm -> 162.6 x 194.3 mm

Commit message: almost done with PCB
Parts:
- added TP1: ~RST, chromogram_libs:BreakOutPad, B.Cu at (191.1, 54.0)
- moved R12 52.9 mm to (65.4, 99.7)
- moved R13 52.8 mm to (196.2, 99.7)
- moved LDR2 52.3 mm to (197.5, 96.5)
- moved LDR1 52.3 mm to (65.4, 96.5)
- moved R15 51.1 mm to (66.7, 227.3), turned to 0 degrees
- moved C10 51.0 mm to (136.5, 177.8)
- moved C13 51.0 mm to (55.2, 213.4)
- moved C14 51.0 mm to (136.5, 213.4)
- moved C18 51.0 mm to (108.0, 74.9)
- moved C5 51.0 mm to (55.2, 142.2)
- moved C6 51.0 mm to (136.5, 142.2)
- moved C7 51.0 mm to (207.6, 149.9)
- moved C8 51.0 mm to (126.4, 149.9)
- moved C9 51.0 mm to (55.2, 177.8)
- moved D1 51.0 mm to (57.8, 81.9)
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Connections:
- net Net-(R6-Pad2) renamed /rtc_ds3231/SQR
- net Net-(R7-Pad2) renamed /rtc_ds3231/32kHz
- U130 pad 4: /RST -> /rtc_ds3231/RESET
Routing:
- net GND: track 2851.4 -> 1638.6 mm
- net /5V: track 2292.2 -> 2350.2 mm
- net /EN: track 184.8 -> 152.6 mm
- net /rtc_ds3231/RESET: track 0.00 -> 27.8 mm, vias 0 -> 1
- net /3V3: track 218.6 -> 198.1 mm
- net /LDR4: track 275.6 -> 271.9 mm
- net /CLK_IN: track 151.5 -> 155.0 mm
- net /LDR1: track 170.4 -> 172.6 mm
- net /DAT_IN: track 158.9 -> 160.8 mm
- net /LDR2: track 110.1 -> 111.9 mm
- net /esp_pwr_uart/RTS: track 86.4 -> 88.0 mm
- net /IO13: track 32.5 -> 33.8 mm
Other:
- board text added: "3V3"
- board text added: "5V"
- board text added: "CLK_IN"
- board text added: "DAT_IN"
- board text added: "EN"
- board text added: "GND"
- board text added: "IO0"
- board text added: "IO13"
- board text added: "IO15"
- board text added: "LDR1"
- board text added: "LDR2"
- board text added: "LDR3"
- board text added: "LDR4"
- board text added: "RXD0"
- board text added: "SCL"
- board text added: "SDA"
- board text added: "SW_D"
- board text added: "SW_E"
- board text added: "SW_I"
- board text added: "SW_M"
- board text added: "TXD0"

Commit message: PCB cleanup
Parts:
- added BITE1: Mouse_Bite, chromogram_libs:mouse-bite-2.54mm-slot, F.Cu at (54.0, 92.7)
- added BITE2: Mouse_Bite, chromogram_libs:mouse-bite-2.54mm-slot, F.Cu at (208.9, 92.7)
- added BITE3: Mouse_Bite, chromogram_libs:mouse-bite-2.54mm-slot, F.Cu at (53.3, 234.9)
- added BITE4: Mouse_Bite, chromogram_libs:mouse-bite-2.54mm-slot, F.Cu at (95.9, 234.9)
- added BITE5: Mouse_Bite, chromogram_libs:mouse-bite-2.54mm-slot, F.Cu at (126.4, 234.9)
- added BITE6: Mouse_Bite, chromogram_libs:mouse-bite-2.54mm-slot, F.Cu at (136.5, 234.9)
- added BITE7: Mouse_Bite, chromogram_libs:mouse-bite-2.54mm-slot, F.Cu at (167.0, 234.9)
- added BITE8: Mouse_Bite, chromogram_libs:mouse-bite-2.54mm-slot, F.Cu at (209.6, 234.9)
- HB45, HB46, HB47, HB48, HB49, HB50, HB51, HB52, HB53, HB54: footprint chromogram_libs:MtgHole_3mm -> chromogram_libs:mtg_hole_3mm_vias_2
- JP1: value PWR_LED_EN -> LED_PWR_EN
Routing:
- net GND: track 1638.6 -> 1674.0 mm
- net /5V: track 2350.2 -> 2372.5 mm
- net /SW_M: vias 2 -> 1
- net /SW_I: vias 2 -> 1
- net /SW_E: vias 2 -> 1
- net /SW_D: vias 2 -> 1
- net /3V3: vias 15 -> 47
Other:
- board text added: "CONNECT MOAR LEDS HERE"
- board text added: "DAT|CLK"
