File: kicad/chromogram.kicad_pcb (KiCad board)
At the start: 2 copper layers, 162.6 x 194.3 mm, 281 parts, among them J1 CLK_IN, J10 DAT_IN, J11 LDR1, J12 LDR2, J13 LDR3, J14 LDR4, J15 5V, J16 GND, J2 DAT_IN, J3 LDR1, J4 LDR2, J5 LDR3, J6 LDR4, J7 5V, J8 GND, J9 CLK_IN, P1 USB_micro, P2 OUT_CLK_DAT, Q1 DDC114TU, U1 APA102, U10 APA102, U100 APA102, U101 APA102, U102 APA102, U103 APA102, U104 APA102, U105 APA102, U106 APA102, U107 APA102, U108 APA102, U109 APA102, U11 APA102, U110 APA102, U111 APA102, U112 APA102, U113 APA102, U114 APA102, U115 APA102, U116 APA102, U117 APA102, U118 APA102, U119 APA102, U12 APA102, U120 APA102, U121 APA102, U122 APA102, U123 APA102, U124 APA102, U125 APA102, U126 APA102, U127 APA102, U128 APA102, U129 ESP-wroom-32, U13 APA102, U130 DS3231N, U131 AP1117-15, U132 CP2102N-A01-GQFN28, U14 APA102, U15 APA102, U16 APA102, U17 APA102, U18 APA102, U19 APA102, U2 APA102, U20 APA102, U21 APA102, U22 APA102, U23 APA102, U24 APA102, U25 APA102, U26 APA102, U27 APA102, U28 APA102, U29 APA102, U3 APA102, U30 APA102, U31 APA102, U32 APA102, U33 APA102, U34 APA102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

Commit message: BoM
Routing:
- net /rtc_ds3231/BAT: track 67.0 -> 81.4 mm
- net /EN: track 152.6 -> 161.2 mm
- net /5V: track 2372.5 -> 2376.6 mm
- net /SW_D: track 75.1 -> 73.3 mm
- net /SW_I: track 59.3 -> 57.5 mm
- net /LDR3: track 225.1 -> 224.0 mm
- net /LDR4: track 271.9 -> 270.8 mm
- net /SW_M: track 90.8 -> 91.6 mm
Other:
- net class 8 mil: via_dia 0.889 -> 0.9; via_drill 0.635 -> 0.5
- net class Default: via_dia 0.889 -> 0.9; via_drill 0.635 -> 0.5
- net class Power: via_dia 0.889 -> 0.9; via_drill 0.635 -> 0.5
- rule via_min_drill: 0.508 -> 0.5
- rule via_min_size: 0.889 -> 0.9
