File: kicad/chromogram.kicad_pcb (KiCad board)
At the start: 2 copper layers, 162.6 x 194.3 mm, 281 parts, among them J1 CLK_IN, J10 DAT_IN, J11 LDR1, J12 LDR2, J13 LDR3, J14 LDR4, J15 5V, J16 GND, J2 DAT_IN, J3 LDR1, J4 LDR2, J5 LDR3, J6 LDR4, J7 5V, J8 GND, J9 CLK_IN, P1 USB_micro, P2 OUT_CLK_DAT, Q1 DDC114TU, U1 APA102, U10 APA102, U100 APA102, U101 APA102, U102 APA102, U103 APA102, U104 APA102, U105 APA102, U106 APA102, U107 APA102, U108 APA102, U109 APA102, U11 APA102, U110 APA102, U111 APA102, U112 APA102, U113 APA102, U114 APA102, U115 APA102, U116 APA102, U117 APA102, U118 APA102, U119 APA102, U12 APA102, U120 APA102, U121 APA102, U122 APA102, U123 APA102, U124 APA102, U125 APA102, U126 APA102, U127 APA102, U128 APA102, U129 ESP-wroom-32, U13 APA102, U130 DS3231N, U131 AP1117-15, U132 CP2102N-A01-GQFN28, U14 APA102, U15 APA102, U16 APA102, U17 APA102, U18 APA102, U19 APA102, U2 APA102, U20 APA102, U21 APA102, U22 APA102, U23 APA102, U24 APA102, U25 APA102, U26 APA102, U27 APA102, U28 APA102, U29 APA102, U3 APA102, U30 APA102, U31 APA102, U32 APA102, U33 APA102, U34 APA102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

Commit message: library edits
Connections:
- P1 pad 4: Net-(P1-Pad4) -> (no net)
- U132 pad 1: /esp_pwr_uart/DCD -> (no net)
- U132 pad 10: Net-(U132-Pad10) -> (no net)
- U132 pad 11: /esp_pwr_uart/ACTIVE -> (no net)
- U132 pad 12: Net-(U132-Pad12) -> (no net)
- U132 pad 13: Net-(U132-Pad13) -> (no net)
- U132 pad 14: Net-(U132-Pad14) -> (no net)
- U132 pad 15: Net-(U132-Pad15) -> (no net)
- U132 pad 16: Net-(U132-Pad16) -> (no net)
- U132 pad 17: Net-(U132-Pad17) -> (no net)
- U132 pad 18: Net-(U132-Pad18) -> (no net)
- U132 pad 19: Net-(U132-Pad19) -> (no net)
- U132 pad 2: /esp_pwr_uart/RI -> (no net)
- U132 pad 20: Net-(U132-Pad20) -> (no net)
- U132 pad 21: Net-(U132-Pad21) -> (no net)
- U132 pad 22: Net-(U132-Pad22) -> (no net)
- U132 pad 27: /esp_pwr_uart/DSR -> (no net)
- U132 pad 9: Net-(U132-Pad9) -> (no net)
Changed lines of the file:
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@@
-(kicad_pcb (version 20171130) (host pcbnew no-vcs-found-5ca5783~61~ubuntu16.04.1)
+(kicad_pcb (version 20171130) (host pcbnew no-vcs-found-70f516b~61~ubuntu16.04.1)
   (general
     (thickness 1.6)
@@
     (zones 0)
     (modules 281)
-    (nets 331)
+    (nets 313)
   )
   (page A3)
@@
     (pad_to_mask_clearance 0)
     (aux_axis_origin 50.8 50.8)
-    (visible_elements 7FFEFF7F)
+    (visible_elements 7FFFFF7F)
     (pcbplotparams
       (layerselection 0x00130_ffffffff)
@@
   (net 311 /rtc_ds3231/SQR)
   (net 312 /rtc_ds3231/32kHz)
-  (net 313 "Net-(P1-Pad4)")
-  (net 314 /esp_pwr_uart/DSR)
-  (net 315 "Net-(U132-Pad22)")
-  (net 316 "Net-(U132-Pad21)")
-  (net 317 "Net-(U132-Pad20)")
-  (net 318 "Net-(U132-Pad19)")
-  (net 319 "Net-(U132-Pad18)")
-  (net 320 "Net-(U132-Pad17)")
-  (net 321 "Net-(U132-Pad16)")
-  (net 322 "Net-(U132-Pad15)")
-  (net 323 "Net-(U132-Pad14)")
-  (net 324 "Net-(U132-Pad13)")
-  (net 325 "Net-(U132-Pad12)")
-  (net 326 /esp_pwr_uart/ACTIVE)
-  (net 327 "Net-(U132-Pad10)")
-  (net 328 "Net-(U132-Pad9)")
-  (net 329 /esp_pwr_uart/RI)
-  (net 330 /esp_pwr_uart/DCD)
   (net_class Default "This is the default net class."
     (clearance 0.1016)
@@
     (add_net /SW_M)
     (add_net /TXD0)
-    (add_net /esp_pwr_uart/ACTIVE)
     (add_net /esp_pwr_uart/CTS)
-    (add_net /esp_pwr_uart/DCD)
-    (add_net /esp_pwr_uart/DSR)
-    (add_net /esp_pwr_uart/RI)
     (add_net /esp_pwr_uart/RTS)
     (add_net /esp_pwr_uart/RXD)
@@
     (add_net "Net-(D2-Pad1)")
     (add_net "Net-(D2-Pad2)")
-    (add_net "Net-(P1-Pad4)")
     (add_net "Net-(R22-Pad2)")
     (add_net "Net-(U1-Pad5)")
@@
     (add_net "Net-(U13-Pad5)")
     (add_net "Net-(U13-Pad6)")
-    (add_net "Net-(U132-Pad10)")
-    (add_net "Net-(U132-Pad12)")
-    (add_net "Net-(U132-Pad13)")
-    (add_net "Net-(U132-Pad14)")
-    (add_net "Net-(U132-Pad15)")
-    (add_net "Net-(U132-Pad16)")
-    (add_net "Net-(U132-Pad17)")
-    (add_net "Net-(U132-Pad18)")
-    (add_net "Net-(U132-Pad19)")
-    (add_net "Net-(U132-Pad20)")
-    (add_net "Net-(U132-Pad21)")
-    (add_net "Net-(U132-Pad22)")
-    (add_net "Net-(U132-Pad9)")
     (add_net "Net-(U14-Pad5)")
     (add_net "Net-(U14-Pad6)")
@@
     (pad 28 smd oval (at -1.5 2.45 270) (size 0.85 0.3) (layers B.Cu B.Paste B.Mask)
       (net 271 /DTR))
-    (pad 27 smd oval (at -1 2.45 270) (size 0.85 0.3) (layers B.Cu B.Paste B.Mask)
-      (net 314 /esp_pwr_uart/DSR))
+    (pad 27 smd oval (at -1 2.45 270) (size 0.85 0.3) (layers B.Cu B.Paste B.Mask))
     (pad 26 smd oval (at -0.5 2.45 270) (size 0.85 0.3) (layers B.Cu B.Paste B.Mask)
       (net 284 "Net-(R22-Pad2)"))
@@
     (pad 23 smd oval (at 1 2.45 270) (size 0.85 0.3) (layers B.Cu B.Paste B.Mask)
       (net 279 /esp_pwr_uart/CTS))
-    (pad 22 smd oval (at 1.5 2.45 270) (size 0.85 0.3) (layers B.Cu B.Paste B.Mask)
-      (net 315 "Net-(U132-Pad22)"))
-    (pad 21 smd oval (at 2.45 1.5) (size 0.85 0.3) (layers B.Cu B.Paste B.Mask)
-      (net 316 "Net-(U132-Pad21)"))
-    (pad 20 smd oval (at 2.45 1) (size 0.85 0.3) (layers B.Cu B.Paste B.Mask)
-      (net 317 "Net-(U132-Pad20)"))
-    (pad 19 smd oval (at 2.45 0.5) (size 0.85 0.3) (layers B.Cu B.Paste B.Mask)
-      (net 318 "Net-(U132-Pad19)"))
-    (pad 18 smd oval (at 2.45 0) (size 0.85 0.3) (layers B.Cu B.Paste B.Mask)
-      (net 319 "Net-(U132-Pad18)"))
-    (pad 17 smd oval (at 2.45 -0.5) (size 0.85 0.3) (layers B.Cu B.Paste B.Mask)
-      (net 320 "Net-(U132-Pad17)"))
-    (pad 16 smd oval (at 2.45 -1) (size 0.85 0.3) (layers B.Cu B.Paste B.Mask)
-      (net 321 "Net-(U132-Pad16)"))
-    (pad 15 smd oval (at 2.45 -1.5) (size 0.85 0.3) (layers B.Cu B.Paste B.Mask)
-      (net 322 "Net-(U132-Pad15)"))
-    (pad 14 smd oval (at 1.5 -2.45 270) (size 0.85 0.3) (layers B.Cu B.Paste B.Mask)
-      (net 323 "Net-(U132-Pad14)"))
-    (pad 13 smd oval (at 1 -2.45 270) (size 0.85 0.3) (layers B.Cu B.Paste B.Mask)
-      (net 324 "Net-(U132-Pad13)"))
-    (pad 12 smd oval (at 0.5 -2.45 270) (size 0.85 0.3) (layers B.Cu B.Paste B.Mask)
-      (net 325 "Net-(U132-Pad12)"))
-    (pad 11 smd oval (at 0 -2.45 270) (size 0.85 0.3) (layers B.Cu B.Paste B.Mask)
-      (net 326 /esp_pwr_uart/ACTIVE))
-    (pad 10 smd oval (at -0.5 -2.45 270) (size 0.85 0.3) (layers B.Cu B.Paste B.Mask)
-      (net 327 "Net-(U132-Pad10)"))
-    (pad 9 smd oval (at -1 -2.45 270) (size 0.85 0.3) (layers B.Cu B.Paste B.Mask)
-      (net 328 "Net-(U132-Pad9)"))
+    (pad 22 smd oval (at 1.5 2.45 270) (size 0.85 0.3) (layers B.Cu B.Paste B.Mask))
+    (pad 21 smd oval (at 2.45 1.5) (size 0.85 0.3) (layers B.Cu B.Paste B.Mask))
+    (pad 20 smd oval (at 2.45 1) (size 0.85 0.3) (layers B.Cu B.Paste B.Mask))
+    (pad 19 smd oval (at 2.45 0.5) (size 0.85 0.3) (layers B.Cu B.Paste B.Mask))
+    (pad 18 smd oval (at 2.45 0) (size 0.85 0.3) (layers B.Cu B.Paste B.Mask))
+    (pad 17 smd oval (at 2.45 -0.5) (size 0.85 0.3) (layers B.Cu B.Paste B.Mask))
+    (pad 16 smd oval (at 2.45 -1) (size 0.85 0.3) (layers B.Cu B.Paste B.Mask))
+    (pad 15 smd oval (at 2.45 -1.5) (size 0.85 0.3) (layers B.Cu B.Paste B.Mask))
+    (pad 14 smd oval (at 1.5 -2.45 270) (size 0.85 0.3) (layers B.Cu B.Paste B.Mask))
+    (pad 13 smd oval (at 1 -2.45 270) (size 0.85 0.3) (layers B.Cu B.Paste B.Mask))
+    (pad 12 smd oval (at 0.5 -2.45 270) (size 0.85 0.3) (layers B.Cu B.Paste B.Mask))
+    (pad 11 smd oval (at 0 -2.45 270) (size 0.85 0.3) (layers B.Cu B.Paste B.Mask))
+    (pad 10 smd oval (at -0.5 -2.45 270) (size 0.85 0.3) (layers B.Cu B.Paste B.Mask))
+    (pad 9 smd oval (at -1 -2.45 270) (size 0.85 0.3) (layers B.Cu B.Paste B.Mask))
     (pad 8 smd oval (at -1.5 -2.45 270) (size 0.85 0.3) (layers B.Cu B.Paste B.Mask)
       (net 261 /5V))
@@
     (pad 3 smd oval (at -2.45 0.5) (size 0.85 0.3) (layers B.Cu B.Paste B.Mask)
       (net 1 GND))
-    (pad 2 smd oval (at -2.45 1) (size 0.85 0.3) (layers B.Cu B.Paste B.Mask)
-      (net 329 /esp_pwr_uart/RI))
-    (pad 1 smd oval (at -2.45 1.5) (size 0.85 0.3) (layers B.Cu B.Paste B.Mask)
-      (net 330 /esp_pwr_uart/DCD))
+    (pad 2 smd oval (at -2.45 1) (size 0.85 0.3) (layers B.Cu B.Paste B.Mask))
+    (pad 1 smd oval (at -2.45 1.5) (size 0.85 0.3) (layers B.Cu B.Paste B.Mask))
     (pad 29 thru_hole circle (at -0.635 0.635) (size 0.8 0.8) (drill 0.5) (layers *.Cu *.Mask)
       (net 1 GND))
@@
     (pad 5 smd rect (at 1.3 2.35 90) (size 0.4 1.35) (layers B.Cu B.Paste B.Mask)
       (net 1 GND))
-    (pad 4 smd rect (at 0.65 2.35 90) (size 0.4 1.35) (layers B.Cu B.Paste B.Mask)
-      (net 313 "Net-(P1-Pad4)"))
+    (pad 4 smd rect (at 0.65 2.35 90) (size 0.4 1.35) (layers B.Cu B.Paste B.Mask))
     (pad 3 smd rect (at 0 2.35 90) (size 0.4 1.35) (layers B.Cu B.Paste B.Mask)
       (net 304 /esp_pwr_uart/USB_D+))
