File: kicad/mechanical.sch (KiCad schematic (older format))
At the start: 44 parts

Commit message: WIP schematic
Parts:
- added HB45, HB46, HB47, HB48, HB49, HB50, HB51, HB52: hole_baffle, chromogram_libs:MtgHole_3mm, symbol chromogram:SCREW
Other:
- note added: "<- 6.0" ->"
- note added: "<- 6.1" ->"
- note added: "<- 8.7" ->"
- note added: "Mounting holes for\nC3jr compatibility\n3 mm diameter\nplated"
Changed lines of the file:
@@
-EESchema Schematic File Version 2
+EESchema Schematic File Version 4
 LIBS:chromogram
-LIBS:wyolum_kicad_symbols
 LIBS:chromogram-cache
-EELAYER 25 0
+EELAYER 26 0
 EELAYER END
 $Descr A4 11693 8268
@@
 F 4 "Value" H 2000 3400 50  0001 C CNN "manf#"
 	1    2000 3400
-	0    -1   -1   0
+	0    1    1    0
 $EndComp
 $Comp
@@
 F 4 "Value" H 2200 3400 50  0001 C CNN "manf#"
 	1    2200 3400
-	0    -1   -1   0
+	0    1    1    0
 $EndComp
 $Comp
@@
 F 4 "Value" H 2400 3400 50  0001 C CNN "manf#"
 	1    2400 3400
-	0    -1   -1   0
+	0    1    1    0
 $EndComp
 $Comp
@@
 F 4 "Value" H 2600 3400 50  0001 C CNN "manf#"
 	1    2600 3400
-	0    -1   -1   0
+	0    1    1    0
 $EndComp
 $Comp
@@
 F 4 "Value" H 2800 3400 50  0001 C CNN "manf#"
 	1    2800 3400
-	0    -1   -1   0
+	0    1    1    0
 $EndComp
 $Comp
@@
 F 4 "Value" H 3000 3400 50  0001 C CNN "manf#"
 	1    3000 3400
-	0    -1   -1   0
+	0    1    1    0
 $EndComp
 $Comp
@@
 F 4 "Value" H 3200 3400 50  0001 C CNN "manf#"
 	1    3200 3400
-	0    -1   -1   0
+	0    1    1    0
 $EndComp
 $Comp
@@
 F 4 "Value" H 3400 3400 50  0001 C CNN "manf#"
 	1    3400 3400
-	0    -1   -1   0
+	0    1    1    0
 $EndComp
 $Comp
@@
 F 4 "Value" H 3600 3400 50  0001 C CNN "manf#"
 	1    3600 3400
-	0    -1   -1   0
+	0    1    1    0
 $EndComp
 $Comp
@@
 F 4 "Value" H 3800 3400 50  0001 C CNN "manf#"
 	1    3800 3400
-	0    -1   -1   0
+	0    1    1    0
 $EndComp
 $Comp
@@
 F 4 "Value" H 4000 3400 50  0001 C CNN "manf#"
 	1    4000 3400
-	0    -1   -1   0
+	0    1    1    0
 $EndComp
 $Comp
@@
 F 4 "Value" H 4200 3400 50  0001 C CNN "manf#"
 	1    4200 3400
-	0    -1   -1   0
+	0    1    1    0
 $EndComp
 $Comp
@@
 F 4 "Value" H 4400 3400 50  0001 C CNN "manf#"
 	1    4400 3400
-	0    -1   -1   0
+	0    1    1    0
 $EndComp
 $Comp
@@
 F 4 "Value" H 4600 3400 50  0001 C CNN "manf#"
 	1    4600 3400
-	0    -1   -1   0
+	0    1    1    0
 $EndComp
 $Comp
@@
 F 4 "Value" H 4800 3400 50  0001 C CNN "manf#"
 	1    4800 3400
-	0    -1   -1   0
+	0    1    1    0
 $EndComp
 $Comp
@@
 F 4 "Value" H 1600 2100 50  0001 C CNN "manf#"
 	1    1600 2100
-	0    -1   -1   0
+	0    1    1    0
 $EndComp
 $Comp
@@
 F 4 "Value" H 1600 2300 50  0001 C CNN "manf#"
 	1    1600 2300
-	1    0    0    -1
+	-1   0    0    1
 $EndComp
 $Comp
@@
 F 4 "Value" H 1600 2500 50  0001 C CNN "manf#"
 	1    1600 2500
-	1    0    0    -1
+	-1   0    0    1
 $EndComp
 $Comp
@@
 F 4 "Value" H 1600 2700 50  0001 C CNN "manf#"
 	1    1600 2700
-	1    0    0    -1
+	-1   0    0    1
 $EndComp
 $Comp
@@
 F 4 "Value" H 1600 2900 50  0001 C CNN "manf#"
 	1    1600 2900
-	1    0    0    -1
+	-1   0    0    1
 $EndComp
 $Comp
@@
 F 4 "Value" H 1600 3100 50  0001 C CNN "manf#"
 	1    1600 3100
-	1    0    0    -1
+	-1   0    0    1
 $EndComp
 $Comp
@@
 F 4 "Value" H 1600 3300 50  0001 C CNN "manf#"
 	1    1600 3300
-	1    0    0    -1
+	-1   0    0    1
 $EndComp
 $Comp
@@
 Text Notes 3150 2700 0    50   ~ 10
 Guide holes for\nBaffle mounting\n2 mm diameter\nnon-plated
+$Comp
+L chromogram:SCREW HB45
+U 1 1 5A4A80D0
+P 1675 4400
+F 0 "HB45" V 1675 4322 40  0000 R CNN
+F 1 "hole_baffle" H 1675 4500 40  0001 C CNN
+F 2 "chromogram_libs:MtgHole_3mm" H 1753 4363 60  0001 L CNN
+F 3 "" H 1675 4400 60  0000 C CNN
+F 4 "Value" H 1675 4400 50  0001 C CNN "manf#"
+	1    1675 4400
+	0    -1   -1   0
+$EndComp
+$Comp
+L chromogram:SCREW HB46
+U 1 1 5A4A8341
+P 3175 4400
+F 0 "HB46" V 3175 4322 40  0000 R CNN
+F 1 "hole_baffle" H 3175 4500 40  0001 C CNN
+F 2 "chromogram_libs:MtgHole_3mm" H 3253 4363 60  0001 L CNN
+F 3 "" H 3175 4400 60  0000 C CNN
+F 4 "Value" H 3175 4400 50  0001 C CNN "manf#"
+	1    3175 4400
+	0    1    1    0
+$EndComp
+$Comp
+L chromogram:SCREW HB51
+U 1 1 5A4A86FB
+P 1675 6400
+F 0 "HB51" V 1675 6322 40  0000 R CNN
+F 1 "hole_baffle" H 1675 6500 40  0001 C CNN
+F 2 "chromogram_libs:MtgHole_3mm" H 1753 6363 60  0001 L CNN
+F 3 "" H 1675 6400 60  0000 C CNN
+F 4 "Value" H 1675 6400 50  0001 C CNN "manf#"
+	1    1675 6400
+	0    -1   -1   0
+$EndComp
+$Comp
+L chromogram:SCREW HB52
+U 1 1 5A4A8702
+P 3175 6400
+F 0 "HB52" V 3175 6322 40  0000 R CNN
+F 1 "hole_baffle" H 3175 6500 40  0001 C CNN
+F 2 "chromogram_libs:MtgHole_3mm" H 3253 6363 60  0001 L CNN
+F 3 "" H 3175 6400 60  0000 C CNN
+F 4 "Value" H 3175 6400 50  0001 C CNN "manf#"
+	1    3175 6400
+	0    1    1    0
+$EndComp
+$Comp
+L chromogram:SCREW HB47
+U 1 1 5A4A8811
+P 1725 4900
+F 0 "HB47" V 1725 4822 40  0000 R CNN
+F 1 "hole_baffle" H 1725 5000 40  0001 C CNN
+F 2 "chromogram_libs:MtgHole_3mm" H 1803 4863 60  0001 L CNN
+F 3 "" H 1725 4900 60  0000 C CNN
+F 4 "Value" H 1725 4900 50  0001 C CNN "manf#"
+	1    1725 4900
+	0    -1   -1   0
+$EndComp
+$Comp
+L chromogram:SCREW HB48
+U 1 1 5A4A8818
+P 3125 4900
+F 0 "HB48" V 3125 4822 40  0000 R CNN
+F 1 "hole_baffle" H 3125 5000 40  0001 C CNN
+F 2 "chromogram_libs:MtgHole_3mm" H 3203 4863 60  0001 L CNN
+F 3 "" H 3125 4900 60  0000 C CNN
+F 4 "Value" H 3125 4900 50  0001 C CNN "manf#"
+	1    3125 4900
+	0    1    1    0
+$EndComp
+$Comp
+L chromogram:SCREW HB49
+U 1 1 5A4A8943
+P 1725 5900
+F 0 "HB49" V 1725 5822 40  0000 R CNN
+F 1 "hole_baffle" H 1725 6000 40  0001 C CNN
+F 2 "chromogram_libs:MtgHole_3mm" H 1803 5863 60  0001 L CNN
+F 3 "" H 1725 5900 60  0000 C CNN
+F 4 "Value" H 1725 5900 50  0001 C CNN "manf#"
+	1    1725 5900
+	0    -1   -1   0
+$EndComp
+$Comp
+L chromogram:SCREW HB50
+U 1 1 5A4A894A
+P 3125 5900
+F 0 "HB50" V 3125 5822 40  0000 R CNN
+F 1 "hole_baffle" H 3125 6000 40  0001 C CNN
+F 2 "chromogram_libs:MtgHole_3mm" H 3203 5863 60  0001 L CNN
+F 3 "" H 3125 5900 60  0000 C CNN
+F 4 "Value" H 3125 5900 50  0001 C CNN "manf#"
+	1    3125 5900
+	0    1    1    0
+$EndComp
+Text Notes 2275 4425 0    40   ~ 0
+<- 6.1" ->
+Text Notes 2275 4925 0    40   ~ 0
+<- 6.0" ->
+Text Notes 2275 5925 0    40   ~ 0
+<- 6.0" ->
+Text Notes 2275 6425 0    40   ~ 0
+<- 6.1" ->
+Text Notes 1750 5600 1    40   ~ 0
+<- 6.0" ->
+Text Notes 3150 5600 1    40   ~ 0
+<- 6.0" ->
+Text Notes 3225 5600 1    40   ~ 0
+<- 8.7" ->
+Text Notes 1675 5600 1    40   ~ 0
+<- 8.7" ->
+Wire Notes Line
+	1575 4300 3275 4300
+Wire Notes Line
+	3275 4300 3275 6500
+Wire Notes Line
+	3275 6500 1575 6500
+Wire Notes Line
+	1575 6500 1575 4300
+Text Notes 2150 5525 0    50   ~ 10
+Mounting holes for\nC3jr compatibility\n3 mm diameter\nplated
 $EndSCHEMATC

Commit message: WIP PCB layout
Parts:
- added HB53, HB54: hole_baffle, chromogram_libs:MtgHole_3mm, symbol chromogram:SCREW
- added J1, J9: CLK_IN, chromogram_libs:1pin, symbol chromogram:Conn_01x01
- added J10, J2: DAT_IN, chromogram_libs:1pin, symbol chromogram:Conn_01x01
- added J11, J3: LDR1, chromogram_libs:1pin, symbol chromogram:Conn_01x01
- added J12, J4: LDR2, chromogram_libs:1pin, symbol chromogram:Conn_01x01
- added J13, J5: LDR3, chromogram_libs:1pin, symbol chromogram:Conn_01x01
- added J14, J6: LDR4, chromogram_libs:1pin, symbol chromogram:Conn_01x01
- added J15, J7: 5V, chromogram_libs:1pin, symbol chromogram:Conn_01x01
- added J16, J8: GND, chromogram_libs:1pin, symbol chromogram:Conn_01x01
Connections:
- net labels added: 5V, CLK_IN, DAT_IN, GND, LDR1, LDR2, LDR3, LDR4
- wire segments 0 -> 16
Other:
- note added: "<- 1.35" ->"
- note added: "<- 2.8" ->"
- note added: "<- 4.45" ->"
- note added: "Mechanical mounting holes\nfor LED matrix\n3 mm diameter\nplated"
- note added: "Mounting holes for\npiggy back attachment\nof "snap-off" control board.\nUse M3 HEX posts to connect\nLED board to control board"
- note removed: "<- 8.7" ->"

Commit message: almost done with PCB
Other:
- note added: "<- 0.575" ->"
- note removed: "<- 4.45" ->"
Changed lines of the file:
@@
 P 5450 4375
 F 0 "J7" H 5275 4425 40  0000 L CNN
-F 1 "5V" H 5525 4400 50  0000 L CNN
+F 1 "5V" H 5525 4400 40  0000 L CNN
 F 2 "chromogram_libs:1pin" H 5450 4375 50  0001 C CNN
 F 3 "~" H 5450 4375 50  0001 C CNN
@@
 	0    1    1    0
 $EndComp
-Text Notes 7400 5275 0    40   ~ 0
+Text Notes 7350 5250 0    40   ~ 0
 <- 2.8" ->
-Text Notes 6875 4950 1    40   ~ 0
-<- 4.45" ->
+Text Notes 7175 4950 1    40   ~ 0
+<- 2.8" ->
 Wire Notes Line
 	6700 3650 8400 3650
@@
 Mechanical mounting holes\nfor LED matrix\n3 mm diameter\nplated
 Wire Notes Line
-	7450 4750 7650 4750
-Wire Notes Line
 	7550 4650 7550 4850
 Wire Notes Line
@@
 Wire Notes Line
 	2450 4650 2450 4850
+Text Notes 8100 4775 1    40   ~ 0
+<- 0.575" ->
+Wire Notes Line
+	7450 4750 8025 4750
 $EndSCHEMATC

Commit message: PCB cleanup
Parts:
- added BITE1, BITE2, BITE3, BITE4, BITE5, BITE6, BITE7, BITE8: Mouse_Bite, chromogram_libs:mouse-bite-2.54mm-slot, symbol ultim_bus:Mouse_Bite
- HB45, HB46, HB47, HB48, HB49, HB50, HB51, HB52, HB53, HB54: footprint chromogram_libs:MtgHole_3mm -> chromogram_libs:mtg_hole_3mm_vias_2
Other:
- note added: "MOUSEBITES\nfor board separation"
