File: kicad/mechanical.sch (KiCad schematic (older format))
At the start: 78 parts, among them J1 CLK_IN, J10 DAT_IN, J11 LDR1, J12 LDR2, J13 LDR3, J14 LDR4, J15 5V, J16 GND, J2 DAT_IN, J3 LDR1, J4 LDR2, J5 LDR3, J6 LDR4, J7 5V, J8 GND, J9 CLK_IN

Commit message: library edits
Parts:
- BITE1, BITE2, BITE3, BITE4, BITE5, BITE6, BITE7, BITE8: symbol ultim_bus:Mouse_Bite -> chromogram:Mouse_Bite; manf# (none) -> mfr_pn
Changed lines of the file:
@@
 encoding utf-8
 Sheet 10 12
-Title ""
-Date ""
-Rev ""
-Comp ""
-Comment1 ""
+Title "Chromogram"
+Date "2017-12-26"
+Rev "rev 1"
+Comp "WyoLum"
+Comment1 "www.wyolum.com"
 Comment2 ""
 Comment3 ""
@@
 	4650 4750 5225 4750
 $Comp
-L ultim_bus:Mouse_Bite BITE1
+L chromogram:Mouse_Bite BITE1
 U 1 1 5A49F376
 P 8100 4900
@@
 F 2 "chromogram_libs:mouse-bite-2.54mm-slot" H 8100 4900 60  0001 C CNN
 F 3 "" H 8100 4900 60  0000 C CNN
+F 4 "mfr_pn" H 8100 4900 50  0001 C CNN "manf#"
 	1    8100 4900
 	1    0    0    -1
 $EndComp
 $Comp
-L ultim_bus:Mouse_Bite BITE2
+L chromogram:Mouse_Bite BITE2
 U 1 1 5A4A147E
 P 8900 4900
@@
 F 2 "chromogram_libs:mouse-bite-2.54mm-slot" H 8900 4900 60  0001 C CNN
 F 3 "" H 8900 4900 60  0000 C CNN
+F 4 "mfr_pn" H 8900 4900 50  0001 C CNN "manf#"
 	1    8900 4900
 	1    0    0    -1
 $EndComp
 $Comp
-L ultim_bus:Mouse_Bite BITE5
+L chromogram:Mouse_Bite BITE5
 U 1 1 5A4A2BA0
 P 8100 5700
@@
 F 2 "chromogram_libs:mouse-bite-2.54mm-slot" H 8100 5700 60  0001 C CNN
 F 3 "" H 8100 5700 60  0000 C CNN
+F 4 "mfr_pn" H 8100 5700 50  0001 C CNN "manf#"
 	1    8100 5700
 	1    0    0    -1
 $EndComp
 $Comp
-L ultim_bus:Mouse_Bite BITE6
+L chromogram:Mouse_Bite BITE6
 U 1 1 5A4A2BA6
 P 8900 5700
@@
 F 2 "chromogram_libs:mouse-bite-2.54mm-slot" H 8900 5700 60  0001 C CNN
 F 3 "" H 8900 5700 60  0000 C CNN
+F 4 "mfr_pn" H 8900 5700 50  0001 C CNN "manf#"
 	1    8900 5700
 	1    0    0    -1
 $EndComp
 $Comp
-L ultim_bus:Mouse_Bite BITE7
+L chromogram:Mouse_Bite BITE7
 U 1 1 5A4A2F4F
 P 9700 5700
@@
 F 2 "chromogram_libs:mouse-bite-2.54mm-slot" H 9700 5700 60  0001 C CNN
 F 3 "" H 9700 5700 60  0000 C CNN
+F 4 "mfr_pn" H 9700 5700 50  0001 C CNN "manf#"
 	1    9700 5700
 	1    0    0    -1
 $EndComp
 $Comp
-L ultim_bus:Mouse_Bite BITE8
+L chromogram:Mouse_Bite BITE8
 U 1 1 5A4A2F55
 P 10500 5700
@@
 F 2 "chromogram_libs:mouse-bite-2.54mm-slot" H 10500 5700 60  0001 C CNN
 F 3 "" H 10500 5700 60  0000 C CNN
+F 4 "mfr_pn" H 10500 5700 50  0001 C CNN "manf#"
 	1    10500 5700
 	1    0    0    -1
 $EndComp
 $Comp
-L ultim_bus:Mouse_Bite BITE3
+L chromogram:Mouse_Bite BITE3
 U 1 1 5A4A335C
 P 6500 5700
@@
 F 2 "chromogram_libs:mouse-bite-2.54mm-slot" H 6500 5700 60  0001 C CNN
 F 3 "" H 6500 5700 60  0000 C CNN
+F 4 "mfr_pn" H 6500 5700 50  0001 C CNN "manf#"
 	1    6500 5700
 	1    0    0    -1
 $EndComp
 $Comp
-L ultim_bus:Mouse_Bite BITE4
+L chromogram:Mouse_Bite BITE4
 U 1 1 5A4A3362
 P 7300 5700
@@
 F 2 "chromogram_libs:mouse-bite-2.54mm-slot" H 7300 5700 60  0001 C CNN
 F 3 "" H 7300 5700 60  0000 C CNN
+F 4 "mfr_pn" H 7300 5700 50  0001 C CNN "manf#"
 	1    7300 5700
 	1    0    0    -1

Commit message: modified diode footprints
Parts:
- added G4: LOGO_WL, chromogram_libs:Logo-WL3, symbol chromogram:LOGO_WL
- added G5: KiCad, chromogram_libs:KiCad-Logo2_6mm_SilkScreen, symbol chromogram:KiCad
- added G6: OSHW, chromogram_libs:OSHW_6mm, symbol chromogram:OSHW
Changed lines of the file:
@@
 Text Notes 8150 5350 0    50   ~ 10
 MOUSEBITES\nfor board separation
+$Comp
+L chromogram:KiCad G5
+U 1 1 5A50766D
+P 9350 6850
+F 0 "G5" H 9350 6582 60  0001 C CNN
+F 1 "KiCad" H 9350 7118 60  0001 C CNN
+F 2 "chromogram_libs:KiCad-Logo2_6mm_SilkScreen" H 9350 6850 60  0001 C CNN
+F 3 "" H 9350 6850 60  0001 C CNN
+F 4 "Value" H 9350 6850 50  0001 C CNN "manf#"
+	1    9350 6850
+	1    0    0    -1
+$EndComp
+$Comp
+L chromogram:OSHW G6
+U 1 1 5A5077CE
+P 10800 7000
+F 0 "G6" H 10800 6950 40  0001 C CNN
+F 1 "OSHW" H 10800 7100 40  0001 C CNN
+F 2 "chromogram_libs:OSHW_6mm" H 10800 7000 60  0001 C CNN
+F 3 "" H 10800 7000 60  0000 C CNN
+F 4 "Value" H 10800 7000 50  0001 C CNN "manf#"
+	1    10800 7000
+	1    0    0    -1
+$EndComp
+$Comp
+L chromogram:LOGO_WL G4
+U 1 1 5A5079CB
+P 8200 6750
+F 0 "G4" H 8200 6614 60  0001 C CNN
+F 1 "LOGO_WL" H 8200 6886 60  0001 C CNN
+F 2 "chromogram_libs:Logo-WL3" H 8200 6750 60  0001 C CNN
+F 3 "" H 8200 6750 60  0001 C CNN
+F 4 "Value" H 8200 6750 50  0001 C CNN "manf#"
+	1    8200 6750
+	1    0    0    -1
+$EndComp
 $EndSCHEMATC

Commit message: edited mousebites
Parts:
- BITE1, BITE2, BITE3, BITE4, BITE5, BITE6, BITE7, BITE8: footprint chromogram_libs:mouse-bite-2.54mm-slot -> chromogram_libs:mouse-bite-2.54mm-slot_OSH
Changed lines of the file:
@@
 F 0 "BITE1" H 8100 5050 40  0000 C CNN
 F 1 "Mouse_Bite" H 8100 5025 30  0001 C CNN
-F 2 "chromogram_libs:mouse-bite-2.54mm-slot" H 8100 4900 60  0001 C CNN
+F 2 "chromogram_libs:mouse-bite-2.54mm-slot_OSH" H 8100 4900 60  0001 C CNN
 F 3 "" H 8100 4900 60  0000 C CNN
 F 4 "mfr_pn" H 8100 4900 50  0001 C CNN "manf#"
@@
 F 0 "BITE2" H 8900 5050 40  0000 C CNN
 F 1 "Mouse_Bite" H 8900 5025 30  0001 C CNN
-F 2 "chromogram_libs:mouse-bite-2.54mm-slot" H 8900 4900 60  0001 C CNN
+F 2 "chromogram_libs:mouse-bite-2.54mm-slot_OSH" H 8900 4900 60  0001 C CNN
 F 3 "" H 8900 4900 60  0000 C CNN
 F 4 "mfr_pn" H 8900 4900 50  0001 C CNN "manf#"
@@
 F 0 "BITE5" H 8100 5850 40  0000 C CNN
 F 1 "Mouse_Bite" H 8100 5825 30  0001 C CNN
-F 2 "chromogram_libs:mouse-bite-2.54mm-slot" H 8100 5700 60  0001 C CNN
+F 2 "chromogram_libs:mouse-bite-2.54mm-slot_OSH" H 8100 5700 60  0001 C CNN
 F 3 "" H 8100 5700 60  0000 C CNN
 F 4 "mfr_pn" H 8100 5700 50  0001 C CNN "manf#"
@@
 F 0 "BITE6" H 8900 5850 40  0000 C CNN
 F 1 "Mouse_Bite" H 8900 5825 30  0001 C CNN
-F 2 "chromogram_libs:mouse-bite-2.54mm-slot" H 8900 5700 60  0001 C CNN
+F 2 "chromogram_libs:mouse-bite-2.54mm-slot_OSH" H 8900 5700 60  0001 C CNN
 F 3 "" H 8900 5700 60  0000 C CNN
 F 4 "mfr_pn" H 8900 5700 50  0001 C CNN "manf#"
@@
 F 0 "BITE7" H 9700 5850 40  0000 C CNN
 F 1 "Mouse_Bite" H 9700 5825 30  0001 C CNN
-F 2 "chromogram_libs:mouse-bite-2.54mm-slot" H 9700 5700 60  0001 C CNN
+F 2 "chromogram_libs:mouse-bite-2.54mm-slot_OSH" H 9700 5700 60  0001 C CNN
 F 3 "" H 9700 5700 60  0000 C CNN
 F 4 "mfr_pn" H 9700 5700 50  0001 C CNN "manf#"
@@
 F 0 "BITE8" H 10500 5850 40  0000 C CNN
 F 1 "Mouse_Bite" H 10500 5825 30  0001 C CNN
-F 2 "chromogram_libs:mouse-bite-2.54mm-slot" H 10500 5700 60  0001 C CNN
+F 2 "chromogram_libs:mouse-bite-2.54mm-slot_OSH" H 10500 5700 60  0001 C CNN
 F 3 "" H 10500 5700 60  0000 C CNN
 F 4 "mfr_pn" H 10500 5700 50  0001 C CNN "manf#"
@@
 F 0 "BITE3" H 6500 5850 40  0000 C CNN
 F 1 "Mouse_Bite" H 6500 5825 30  0001 C CNN
-F 2 "chromogram_libs:mouse-bite-2.54mm-slot" H 6500 5700 60  0001 C CNN
+F 2 "chromogram_libs:mouse-bite-2.54mm-slot_OSH" H 6500 5700 60  0001 C CNN
 F 3 "" H 6500 5700 60  0000 C CNN
 F 4 "mfr_pn" H 6500 5700 50  0001 C CNN "manf#"
@@
 F 0 "BITE4" H 7300 5850 40  0000 C CNN
 F 1 "Mouse_Bite" H 7300 5825 30  0001 C CNN
-F 2 "chromogram_libs:mouse-bite-2.54mm-slot" H 7300 5700 60  0001 C CNN
+F 2 "chromogram_libs:mouse-bite-2.54mm-slot_OSH" H 7300 5700 60  0001 C CNN
 F 3 "" H 7300 5700 60  0000 C CNN
 F 4 "mfr_pn" H 7300 5700 50  0001 C CNN "manf#"

Commit message: modified mounting holes
Parts:
- HB45, HB46: value hole_baffle -> mtg_hole_3mm_small; footprint chromogram_libs:mtg_hole_3mm_vias_2 -> chromogram_libs:MountingHole_3.2mm_M3
- HB47, HB48, HB49, HB50, HB51, HB52, HB53, HB54: value hole_baffle -> mtg_hole_3mm; footprint chromogram_libs:mtg_hole_3mm_vias_2 -> chromogram_libs:MountingHole_3.2mm_M3_Pad_Via
Changed lines of the file:
@@
 P 1700 3750
 F 0 "HB45" V 1700 3672 40  0000 R CNN
-F 1 "hole_baffle" H 1700 3850 40  0001 C CNN
-F 2 "chromogram_libs:mtg_hole_3mm_vias_2" H 1778 3713 60  0001 L CNN
+F 1 "mtg_hole_3mm_small" H 1700 3850 40  0001 C CNN
+F 2 "chromogram_libs:MountingHole_3.2mm_M3" H 1778 3713 60  0001 L CNN
 F 3 "" H 1700 3750 60  0000 C CNN
 F 4 "Value" H 1700 3750 50  0001 C CNN "manf#"
@@
 P 3200 3750
 F 0 "HB46" V 3200 3672 40  0000 R CNN
-F 1 "hole_baffle" H 3200 3850 40  0001 C CNN
-F 2 "chromogram_libs:mtg_hole_3mm_vias_2" H 3278 3713 60  0001 L CNN
+F 1 "mtg_hole_3mm_small" H 3200 3850 40  0001 C CNN
+F 2 "chromogram_libs:MountingHole_3.2mm_M3" H 3278 3713 60  0001 L CNN
 F 3 "" H 3200 3750 60  0000 C CNN
 F 4 "Value" H 3200 3750 50  0001 C CNN "manf#"
@@
 P 1750 4250
 F 0 "HB47" V 1750 4172 40  0000 R CNN
-F 1 "hole_baffle" H 1750 4350 40  0001 C CNN
-F 2 "chromogram_libs:mtg_hole_3mm_vias_2" H 1828 4213 60  0001 L CNN
+F 1 "mtg_hole_3mm" H 1750 4350 40  0001 C CNN
+F 2 "chromogram_libs:MountingHole_3.2mm_M3_Pad_Via" H 1828 4213 60  0001 L CNN
 F 3 "" H 1750 4250 60  0000 C CNN
 F 4 "Value" H 1750 4250 50  0001 C CNN "manf#"
@@
 P 3150 4250
 F 0 "HB48" V 3150 4172 40  0000 R CNN
-F 1 "hole_baffle" H 3150 4350 40  0001 C CNN
-F 2 "chromogram_libs:mtg_hole_3mm_vias_2" H 3228 4213 60  0001 L CNN
+F 1 "mtg_hole_3mm" H 3150 4350 40  0001 C CNN
+F 2 "chromogram_libs:MountingHole_3.2mm_M3_Pad_Via" H 3228 4213 60  0001 L CNN
 F 3 "" H 3150 4250 60  0000 C CNN
 F 4 "Value" H 3150 4250 50  0001 C CNN "manf#"
@@
 P 1750 5250
 F 0 "HB49" V 1750 5172 40  0000 R CNN
-F 1 "hole_baffle" H 1750 5350 40  0001 C CNN
-F 2 "chromogram_libs:mtg_hole_3mm_vias_2" H 1828 5213 60  0001 L CNN
+F 1 "mtg_hole_3mm" H 1750 5350 40  0001 C CNN
+F 2 "chromogram_libs:MountingHole_3.2mm_M3_Pad_Via" H 1828 5213 60  0001 L CNN
 F 3 "" H 1750 5250 60  0000 C CNN
 F 4 "Value" H 1750 5250 50  0001 C CNN "manf#"
@@
 P 3150 5250
 F 0 "HB50" V 3150 5172 40  0000 R CNN
-F 1 "hole_baffle" H 3150 5350 40  0001 C CNN
-F 2 "chromogram_libs:mtg_hole_3mm_vias_2" H 3228 5213 60  0001 L CNN
+F 1 "mtg_hole_3mm" H 3150 5350 40  0001 C CNN
+F 2 "chromogram_libs:MountingHole_3.2mm_M3_Pad_Via" H 3228 5213 60  0001 L CNN
 F 3 "" H 3150 5250 60  0000 C CNN
 F 4 "Value" H 3150 5250 50  0001 C CNN "manf#"
@@
 P 4350 4350
 F 0 "HB51" V 4350 4272 40  0000 R CNN
-F 1 "hole_baffle" H 4350 4450 40  0001 C CNN
-F 2 "chromogram_libs:mtg_hole_3mm_vias_2" H 4428 4313 60  0001 L CNN
+F 1 "mtg_hole_3mm" H 4350 4450 40  0001 C CNN
+F 2 "chromogram_libs:MountingHole_3.2mm_M3_Pad_Via" H 4428 4313 60  0001 L CNN
 F 3 "" H 4350 4350 60  0000 C CNN
 F 4 "Value" H 4350 4350 50  0001 C CNN "manf#"
@@
 P 5150 4350
 F 0 "HB52" V 5150 4272 40  0000 R CNN
-F 1 "hole_baffle" H 5150 4450 40  0001 C CNN
-F 2 "chromogram_libs:mtg_hole_3mm_vias_2" H 5228 4313 60  0001 L CNN
+F 1 "mtg_hole_3mm" H 5150 4450 40  0001 C CNN
+F 2 "chromogram_libs:MountingHole_3.2mm_M3_Pad_Via" H 5228 4313 60  0001 L CNN
 F 3 "" H 5150 4350 60  0000 C CNN
 F 4 "Value" H 5150 4350 50  0001 C CNN "manf#"
@@
 P 4350 5150
 F 0 "HB53" V 4350 5072 40  0000 R CNN
-F 1 "hole_baffle" H 4350 5250 40  0001 C CNN
-F 2 "chromogram_libs:mtg_hole_3mm_vias_2" H 4428 5113 60  0001 L CNN
+F 1 "mtg_hole_3mm" H 4350 5250 40  0001 C CNN
+F 2 "chromogram_libs:MountingHole_3.2mm_M3_Pad_Via" H 4428 5113 60  0001 L CNN
 F 3 "" H 4350 5150 60  0000 C CNN
 F 4 "Value" H 4350 5150 50  0001 C CNN "manf#"
@@
 P 5150 5150
 F 0 "HB54" V 5150 5072 40  0000 R CNN
-F 1 "hole_baffle" H 5150 5250 40  0001 C CNN
-F 2 "chromogram_libs:mtg_hole_3mm_vias_2" H 5228 5113 60  0001 L CNN
+F 1 "mtg_hole_3mm" H 5150 5250 40  0001 C CNN
+F 2 "chromogram_libs:MountingHole_3.2mm_M3_Pad_Via" H 5228 5113 60  0001 L CNN
 F 3 "" H 5150 5150 60  0000 C CNN
 F 4 "Value" H 5150 5150 50  0001 C CNN "manf#"

Commit message: renamed all files, fresh Gerbers
Parts:
- BITE1, BITE2, BITE3, BITE4, BITE5, BITE6, BITE7, BITE8: footprint chromogram_libs:mouse-bite-2.54mm-slot_OSH -> KlokTHREEjr_libs:mouse-bite-2.54mm-slot_OSH; symbol chromogram:Mouse_Bite -> KlokTHREEjr:Mouse_Bite
- G4: footprint chromogram_libs:Logo-WL3 -> KlokTHREEjr_libs:Logo-WL3; symbol chromogram:LOGO_WL -> KlokTHREEjr:LOGO_WL
- G5: footprint chromogram_libs:KiCad-Logo2_6mm_SilkScreen -> KlokTHREEjr_libs:KiCad-Logo2_6mm_SilkScreen; symbol chromogram:KiCad -> KlokTHREEjr:KiCad
- G6: footprint chromogram_libs:OSHW_6mm -> KlokTHREEjr_libs:OSHW_6mm; symbol chromogram:OSHW -> KlokTHREEjr:OSHW
- HB1, HB10, HB11, HB12, HB13, HB14, HB15, HB16, HB17, HB18, HB19, HB2, HB20, HB21, HB22, HB23, HB24, HB25, HB26, HB27, HB28, HB29, HB3, HB30, HB31, HB32, HB33, HB34, HB35, HB36, HB37, HB38, HB39, HB4, HB40, HB41, HB42, HB43, HB44, HB5, HB6, HB7, HB8, HB9: footprint chromogram_libs:hole_baffle_2mm -> KlokTHREEjr_libs:hole_baffle_2mm; symbol chromogram:SCREW -> KlokTHREEjr:SCREW
- HB45, HB46: footprint chromogram_libs:MountingHole_3.2mm_M3 -> KlokTHREEjr_libs:MountingHole_3.2mm_M3; symbol chromogram:SCREW -> KlokTHREEjr:SCREW
- HB47, HB48, HB49, HB50, HB51, HB52, HB53, HB54: footprint chromogram_libs:MountingHole_3.2mm_M3_Pad_Via -> KlokTHREEjr_libs:MountingHole_3.2mm_M3_Pad_Via; symbol chromogram:SCREW -> KlokTHREEjr:SCREW
- J1, J10, J11, J12, J13, J14, J15, J16, J2, J3, J4, J5, J6, J7, J8, J9: footprint chromogram_libs:1pin -> KlokTHREEjr_libs:1pin; symbol chromogram:Conn_01x01 -> KlokTHREEjr:Conn_01x01

Commit message: USB protection, LDR, Switches reconfigured
Parts:
- removed G4: LOGO_WL, KlokTHREEjr_libs:Logo-WL3, symbol KlokTHREEjr:LOGO_WL
- removed G5: KiCad, KlokTHREEjr_libs:KiCad-Logo2_6mm_SilkScreen, symbol KlokTHREEjr:KiCad
- removed G6: OSHW, KlokTHREEjr_libs:OSHW_6mm, symbol KlokTHREEjr:OSHW
- removed J11, J3: LDR1, KlokTHREEjr_libs:1pin, symbol KlokTHREEjr:Conn_01x01
- removed J12, J4: LDR2, KlokTHREEjr_libs:1pin, symbol KlokTHREEjr:Conn_01x01
- removed J13, J5: LDR3, KlokTHREEjr_libs:1pin, symbol KlokTHREEjr:Conn_01x01
- removed J14, J6: LDR4, KlokTHREEjr_libs:1pin, symbol KlokTHREEjr:Conn_01x01
Connections:
- net labels removed: LDR1, LDR2, LDR3, LDR4
- wire segments 16 -> 8
Changed lines of the file:
@@
-$EndComp
-$Comp
-L KlokTHREEjr:Conn_01x01 J3
-U 1 1 5A486F0A
-P 7200 1825
-F 0 "J3" H 7025 1875 40  0000 L CNN
-F 1 "LDR1" H 7275 1850 40  0000 L CNN
-F 2 "KlokTHREEjr_libs:1pin" H 7200 1825 50  0001 C CNN
-F 3 "~" H 7200 1825 50  0001 C CNN
-	1    7200 1825
-	0    1    1    0
-$EndComp
-$Comp
-L KlokTHREEjr:Conn_01x01 J4
-U 1 1 5A486F90
-P 7400 1825
-F 0 "J4" H 7225 1875 50  0000 L CNN
-F 1 "LDR2" H 7475 1850 40  0000 L CNN
-F 2 "KlokTHREEjr_libs:1pin" H 7400 1825 50  0001 C CNN
-F 3 "~" H 7400 1825 50  0001 C CNN
-	1    7400 1825
-	0    1    1    0
-$EndComp
-$Comp
-L KlokTHREEjr:Conn_01x01 J5
-U 1 1 5A4872FB
-P 7600 1825
-F 0 "J5" H 7425 1875 40  0000 L CNN
-F 1 "LDR3" H 7675 1850 40  0000 L CNN
-F 2 "KlokTHREEjr_libs:1pin" H 7600 1825 50  0001 C CNN
-F 3 "~" H 7600 1825 50  0001 C CNN
-	1    7600 1825
-	0    1    1    0
-$EndComp
-$Comp
-L KlokTHREEjr:Conn_01x01 J6
-U 1 1 5A487301
-P 7800 1825
-F 0 "J6" H 7625 1875 40  0000 L CNN
-F 1 "LDR4" H 7875 1850 40  0000 L CNN
-F 2 "KlokTHREEjr_libs:1pin" H 7800 1825 50  0001 C CNN
-F 3 "~" H 7800 1825 50  0001 C CNN
-	1    7800 1825
-	0    1    1    0
 $EndComp
 $Comp
@@
 $EndComp
 $Comp
-L KlokTHREEjr:Conn_01x01 J11
-U 1 1 5A4877AC
-P 7200 2450
-F 0 "J11" H 7025 2500 40  0000 L CNN
-F 1 "LDR1" H 7275 2475 40  0000 L CNN
-F 2 "KlokTHREEjr_libs:1pin" H 7200 2450 50  0001 C CNN
-F 3 "~" H 7200 2450 50  0001 C CNN
-	1    7200 2450
-	0    1    -1   0
-$EndComp
-$Comp
-L KlokTHREEjr:Conn_01x01 J12
-U 1 1 5A4877B2
-P 7400 2450
-F 0 "J12" H 7225 2500 40  0000 L CNN
-F 1 "LDR2" H 7475 2475 40  0000 L CNN
-F 2 "KlokTHREEjr_libs:1pin" H 7400 2450 50  0001 C CNN
-F 3 "~" H 7400 2450 50  0001 C CNN
-	1    7400 2450
-	0    1    -1   0
-$EndComp
-$Comp
-L KlokTHREEjr:Conn_01x01 J13
-U 1 1 5A4877B8
-P 7600 2450
-F 0 "J13" H 7425 2500 40  0000 L CNN
-F 1 "LDR3" H 7675 2475 40  0000 L CNN
-F 2 "KlokTHREEjr_libs:1pin" H 7600 2450 50  0001 C CNN
-F 3 "~" H 7600 2450 50  0001 C CNN
-	1    7600 2450
-	0    1    -1   0
-$EndComp
-$Comp
-L KlokTHREEjr:Conn_01x01 J14
-U 1 1 5A4877BE
-P 7800 2450
-F 0 "J14" H 7625 2500 40  0000 L CNN
-F 1 "LDR4" H 7875 2475 40  0000 L CNN
-F 2 "KlokTHREEjr_libs:1pin" H 7800 2450 50  0001 C CNN
-F 3 "~" H 7800 2450 50  0001 C CNN
-	1    7800 2450
-	0    1    -1   0
-$EndComp
-$Comp
 L KlokTHREEjr:Conn_01x01 J15
 U 1 1 5A4877C4
@@
 	7000 1375 7000 1625
 Wire Wire Line
-	7200 1375 7200 1625
-Wire Wire Line
-	7400 1375 7400 1625
-Wire Wire Line
-	7600 1375 7600 1625
-Wire Wire Line
-	7800 1375 7800 1625
-Wire Wire Line
 	8000 1375 8000 1625
 Wire Wire Line
@@
 Text Label 7000 1375 3    40   ~ 0
 DAT_IN
-Text Label 7200 1375 3    40   ~ 0
-LDR1
-Text Label 7400 1375 3    40   ~ 0
-LDR2
-Text Label 7600 1375 3    40   ~ 0
-LDR3
-Text Label 7800 1375 3    40   ~ 0
-LDR4
 Text Label 8000 1375 3    40   ~ 0
 5V
@@
 Wire Wire Line
 	7000 2650 7000 2900
-Wire Wire Line
-	7200 2650 7200 2900
-Wire Wire Line
-	7400 2650 7400 2900
-Wire Wire Line
-	7600 2650 7600 2900
-Wire Wire Line
-	7800 2650 7800 2900
 Wire Wire Line
 	8000 2650 8000 2900
@@
 Text Label 7000 2900 1    40   ~ 0
 DAT_IN
-Text Label 7200 2900 1    40   ~ 0
-LDR1
-Text Label 7400 2900 1    40   ~ 0
-LDR2
-Text Label 7600 2900 1    40   ~ 0
-LDR3
-Text Label 7800 2900 1    40   ~ 0
-LDR4
 Text Label 8000 2900 1    40   ~ 0
 5V
@@
 Text HLabel 7000 1375 1    40   Input ~ 0
 DAT_IN
-Text HLabel 7200 1375 1    40   Input ~ 0
-LDR1
-Text HLabel 7400 1375 1    40   Input ~ 0
-LDR2
-Text HLabel 7800 1375 1    40   Input ~ 0
-LDR4
-Text HLabel 7600 1375 1    40   Input ~ 0
-LDR3
 Text HLabel 8000 1375 1    40   Input ~ 0
 5V
@@
 Text Notes 8150 5350 0    50   ~ 10
 MOUSEBITES\nfor board separation
-$Comp
-L KlokTHREEjr:KiCad G5
-U 1 1 5A50766D
-P 9700 6850
-F 0 "G5" H 9700 6582 60  0001 C CNN
-F 1 "KiCad" H 9700 7118 60  0001 C CNN
-F 2 "KlokTHREEjr_libs:KiCad-Logo2_6mm_SilkScreen" H 9700 6850 60  0001 C CNN
-F 3 "" H 9700 6850 60  0001 C CNN
-F 4 "Value" H 9700 6850 50  0001 C CNN "manf#"
-	1    9700 6850
-	1    0    0    -1
-$EndComp
-$Comp
-L KlokTHREEjr:OSHW G6
-U 1 1 5A5077CE
-P 10850 7000
-F 0 "G6" H 10850 6950 40  0001 C CNN
-F 1 "OSHW" H 10850 7100 40  0001 C CNN
-F 2 "KlokTHREEjr_libs:OSHW_6mm" H 10850 7000 60  0001 C CNN
-F 3 "" H 10850 7000 60  0000 C CNN
-F 4 "Value" H 10850 7000 50  0001 C CNN "manf#"
-	1    10850 7000
-	1    0    0    -1
-$EndComp
-$Comp
-L KlokTHREEjr:LOGO_WL G4
-U 1 1 5A5079CB
-P 8450 6700
-F 0 "G4" H 8450 6564 60  0001 C CNN
-F 1 "LOGO_WL" H 8450 6836 60  0001 C CNN
-F 2 "KlokTHREEjr_libs:Logo-WL3" H 8450 6700 60  0001 C CNN
-F 3 "" H 8450 6700 60  0001 C CNN
-F 4 "Value" H 8450 6700 50  0001 C CNN "manf#"
-	1    8450 6700
-	1    0    0    -1
-$EndComp
 $EndSCHEMATC
