File: kicad/esp_pwr_uart.sch (KiCad schematic (older format))
At the start: 11 parts

Commit message: making progress on schematic
Parts:
- added C19, C20, C21: 1nF, chromogram_libs:c_0805, symbol C_NP
- added C23, C25: 10uF/25V, chromogram_libs:c_2917, symbol chromogram:C_POL
- added C24, C26: 100nF, chromogram_libs:c_0805, symbol C_NP
- added Q1, Q2: S8050, TO_SOT_Packages_SMD:SOT-23, symbol Q_NPN_BCE
- added R16, R18, R22: 470R, chromogram_libs:r_0805, symbol R
- added R17, R3, R5: 12k, chromogram_libs:r_0805, symbol R
- added R19, R20: 0R NC, chromogram_libs:r_0805, symbol R
- added R21, R23: 0R, chromogram_libs:r_0805, symbol R
- added S3: EN, chromogram_libs:SW_SMD, symbol SW-SPST-M
- added S4: BOOT, chromogram_libs:SW_SMD, symbol SW-SPST-M
- C17, C18: renamed from C?; footprint (none) -> chromogram_libs:c_2917
- D1: renamed from D?; footprint (none) -> Diodes_SMD:D_SOD-123
- D2: footprint (none) -> LEDs:LED-0805
- D3, D4: renamed from D?; value diode_sch -> VESD05A1B; footprint (none) -> Diodes_SMD:D_SOD-123
- JP1: renamed from JP?; footprint (none) -> Resistors_SMD:R_0402
- P1: renamed from P?; footprint (none) -> Connectors_USB:USB_Micro-B_Molex-105017-0001
- R4: renamed from R?; footprint (none) -> chromogram_libs:r_0805
- gave numbers to parts that had none: 2
Connections:
- net labels added: ACTIVE, CTS, DCD, DSR, DTR, EN, IO0, IO13, IO15, RI, RTS, RXD, RXD0, TXD, TXD0, USB_DN, USB_DP
- wire segments 45 -> 94
- no-connect marks 1 -> 3
Other:
- note added: "Auto program\nDTR RTS-->EN IO0\n 1 1 1 1\n 0 0 1 1\n 1 0 0 1\n 0 1 1 0"

Commit message: WIP schematic
Parts:
- removed Q1, Q2: S8050, TO_SOT_Packages_SMD:SOT-23, symbol Q_NPN_BCE
- removed R17, R5: 12k, chromogram_libs:r_0805, symbol R
- added Q1: DDC114TU, chromogram_libs:SOT-363_SC-70-6, symbol chromogram:DDC114TU
- C19, C20, C21, C24, C26: symbol C_NP -> chromogram:C_NP; manf# (none) -> Value
- D1, D3, D4: footprint Diodes_SMD:D_SOD-123 -> chromogram_libs:D_SOD-123
- D2: footprint LEDs:LED-0805 -> chromogram_libs:LED-0805
- JP1: footprint Resistors_SMD:R_0402 -> chromogram_libs:R_0402
- P1: footprint Connectors_USB:USB_Micro-B_Molex-105017-0001 -> chromogram_libs:USB_Micro-B_Molex-105017-0001
- R16, R18, R19, R20, R21, R22, R23: symbol R -> chromogram:R; manf# (none) -> Value
- R3: value 12k -> 10k; symbol R -> chromogram:R; manf# (none) -> Value
- S3, S4: symbol SW-SPST-M -> chromogram:SW-SPST-M; manf# (none) -> Value
- U131: footprint TO_SOT_Packages_SMD:SOT-223-3_TabPin2 -> chromogram_libs:SOT-223-3_TabPin2
- U132: footprint Housings_DFN_QFN:QFN-28-1EP_5x5mm_Pitch0.5mm -> chromogram_libs:QFN-28-1EP_5x5mm_Pitch0.5mm
Connections:
- wire segments 94 -> 128
- no-connect marks 3 -> 7

Commit message: making progress on PCB
Connections:
- net labels added: USB_D+, USB_D-
- net labels removed: USB_DN, USB_DP
- wire segments 128 -> 92
Changed lines of the file:
@@
-EESchema Schematic File Version 4
+EESchema Schematic File Version 2
 LIBS:chromogram
+LIBS:wyolum_kicad_symbols
 LIBS:chromogram-cache
-EELAYER 26 0
+EELAYER 25 0
 EELAYER END
 $Descr A4 11693 8268
@@
 $EndComp
 Wire Wire Line
-	1225 1300 1375 1300
-Wire Wire Line
-	1375 1250 1375 1300
+	1225 1300 1875 1300
+Wire Wire Line
+	1375 1250 1375 1400
 Wire Wire Line
 	1675 1300 1675 1400
 Connection ~ 1675 1300
 Wire Wire Line
-	2475 1300 2625 1300
-Wire Wire Line
-	2625 1250 2625 1300
+	2475 1300 2950 1300
+Wire Wire Line
+	2625 1250 2625 1400
 Wire Wire Line
 	2625 2575 2625 1700
 Wire Wire Line
-	1225 2575 1375 2575
+	1225 2575 2775 2575
 Wire Wire Line
 	1375 1800 1375 1700
 Wire Wire Line
-	1675 1700 1675 2575
+	1675 2575 1675 1700
 Connection ~ 1675 2575
 Wire Wire Line
-	2175 1600 2175 2575
+	2175 1600 2175 2675
 Connection ~ 2175 2575
 Wire Wire Line
 	1375 2100 1375 2200
 Wire Wire Line
-	1375 2400 1375 2575
+	1375 2575 1375 2400
 $Comp
 L chromogram:GND #PWR019
@@
 	1975 4550 1975 6025
 Wire Wire Line
-	4375 6025 3700 6025
+	4375 6025 1325 6025
 Wire Wire Line
 	4375 5250 4450 5250
@@
 Connection ~ 1975 6025
 Wire Wire Line
-	1875 4250 2325 4250
+	1875 4250 2750 4250
 Wire Wire Line
 	2325 4250 2325 4800
 Wire Wire Line
-	1875 4350 2125 4350
+	1875 4350 2850 4350
 Wire Wire Line
 	2125 4350 2125 4800
@@
 	4450 5150 4375 5150
 Wire Wire Line
-	4375 5150 4375 5250
-Wire Wire Line
-	3025 3950 3250 3950
+	4375 5150 4375 6025
+Wire Wire Line
+	3025 3950 4450 3950
 Wire Wire Line
 	4375 3950 4375 4050
@@
 	2850 4850 4450 4850
 Wire Wire Line
-	3475 4750 3700 4750
+	3475 4750 4450 4750
 Text Label 7400 4650 2    40   ~ 0
 DCD
@@
 Connection ~ 2325 4250
 Text Label 4100 4850 0    40   ~ 0
-USB_DP
+USB_D+
 Text Label 4100 4950 0    40   ~ 0
-USB_DN
+USB_D-
 Connection ~ 4375 3950
 Text Label 4100 4750 0    40   ~ 0
@@
 Connection ~ 3475 6025
 Wire Wire Line
-	3700 5625 3700 6025
+	3700 6025 3700 5625
 Connection ~ 3700 6025
 Wire Wire Line
 	3025 5325 3025 3950
 Wire Wire Line
-	3250 5325 3250 3950
+	3250 3950 3250 5325
 Connection ~ 3250 3950
 Wire Wire Line
 	3475 5325 3475 4750
 Wire Wire Line
-	3700 5325 3700 4750
+	3700 4750 3700 5325
 Connection ~ 3700 4750
 NoConn ~ 4450 4250
@@
 IO15
 Wire Wire Line
-	6800 1350 7150 1350
-Wire Wire Line
-	6800 2250 7000 2250
+	6800 1350 7675 1350
+Wire Wire Line
+	6800 2250 7675 2250
 Wire Wire Line
 	7150 1350 7150 2000
@@
 	7975 2450 7975 2500
 Wire Wire Line
-	7975 2500 9250 2500
-Wire Wire Line
-	7975 1100 8925 1100
+	7975 2500 10350 2500
+Wire Wire Line
+	7975 1100 10350 1100
 Wire Wire Line
 	7975 1100 7975 1150
@@
 $EndComp
 Wire Wire Line
-	8925 1000 8925 1100
+	8925 1000 8925 1600
 Connection ~ 8925 1100
 $Comp
@@
 	9575 2000 9575 1900
 Wire Wire Line
-	8925 2000 9250 2000
+	8925 2000 9575 2000
 Wire Wire Line
 	8925 2000 8925 1900
 Wire Wire Line
-	9250 1900 9250 2000
+	9250 2000 9250 1900
 Connection ~ 9250 2000
 Wire Wire Line
-	9525 1900 9525 2000
+	9525 2000 9525 1900
 Connection ~ 9525 2000
 Wire Wire Line
-	9250 1500 9250 1550
+	9250 1500 9250 1600
 Wire Wire Line
 	9575 1550 9575 1600
 Wire Wire Line
-	9250 1550 9525 1550
+	9250 1550 9575 1550
 Connection ~ 9250 1550
 Wire Wire Line
-	9525 1600 9525 1550
+	9525 1550 9525 1600
 Connection ~ 9525 1550
 Connection ~ 9250 1100
@@
 	9575 3400 9575 3300
 Wire Wire Line
-	9250 3400 9525 3400
+	9250 3400 9575 3400
 Wire Wire Line
 	9250 3300 9250 3400
 Wire Wire Line
-	9525 3300 9525 3400
+	9525 3400 9525 3300
 Connection ~ 9525 3400
 Wire Wire Line
-	9250 2900 9250 2950
+	9250 2900 9250 3000
 Wire Wire Line
 	9575 2950 9575 3000
 Wire Wire Line
-	9250 2950 9525 2950
+	9250 2950 9575 2950
 Connection ~ 9250 2950
 Wire Wire Line
-	9525 3000 9525 2950
+	9525 2950 9525 3000
 Connection ~ 9525 2950
 Connection ~ 9250 2500
@@
 	2775 2575 2775 2475
 Connection ~ 2625 2575
-Wire Wire Line
-	1675 1300 1875 1300
-Wire Wire Line
-	1675 2575 2175 2575
-Wire Wire Line
-	2175 2575 2175 2675
-Wire Wire Line
-	2175 2575 2625 2575
-Wire Wire Line
-	1375 2575 1675 2575
-Wire Wire Line
-	1375 1300 1675 1300
-Wire Wire Line
-	1375 1300 1375 1400
-Wire Wire Line
-	2625 1300 2950 1300
-Wire Wire Line
-	2625 1300 2625 1400
-Wire Wire Line
-	2125 6025 1975 6025
-Wire Wire Line
-	1975 6025 1325 6025
-Wire Wire Line
-	4375 5250 4375 6025
-Wire Wire Line
-	2325 6025 2125 6025
-Wire Wire Line
-	2125 4350 2850 4350
-Wire Wire Line
-	2325 4250 2750 4250
-Wire Wire Line
-	4375 3950 4450 3950
-Wire Wire Line
-	3025 6025 2325 6025
-Wire Wire Line
-	3250 6025 3025 6025
-Wire Wire Line
-	3475 6025 3250 6025
-Wire Wire Line
-	3700 6025 3475 6025
-Wire Wire Line
-	3250 3950 4375 3950
-Wire Wire Line
-	3700 4750 4450 4750
-Wire Wire Line
-	7150 1350 7675 1350
-Wire Wire Line
-	7000 2250 7675 2250
-Wire Wire Line
-	8925 1100 9250 1100
-Wire Wire Line
-	8925 1100 8925 1600
-Wire Wire Line
-	9250 2000 9525 2000
-Wire Wire Line
-	9525 2000 9575 2000
-Wire Wire Line
-	9250 1550 9250 1600
-Wire Wire Line
-	9525 1550 9575 1550
-Wire Wire Line
-	9250 1100 10350 1100
-Wire Wire Line
-	9525 3400 9575 3400
-Wire Wire Line
-	9250 2950 9250 3000
-Wire Wire Line
-	9525 2950 9575 2950
-Wire Wire Line
-	9250 2500 10350 2500
-Wire Wire Line
-	2625 2575 2775 2575
 NoConn ~ 4100 4550
 NoConn ~ 7400 4650

Commit message: almost done with PCB
Parts:
- U131: symbol regul:AP1117-15 -> chromogram:AP1117-15; manf# (none) -> mfr_pn
Connections:
- wire segments 92 -> 128
Changed lines of the file:
@@
 $EndComp
 $Comp
-L regul:AP1117-15 U131
+L chromogram:AP1117-15 U131
 U 1 1 5A4518D4
 P 2175 1300
@@
 F 2 "chromogram_libs:SOT-223-3_TabPin2" H 2175 1500 50  0001 C CNN
 F 3 "http://www.diodes.com/datasheets/AP1117.pdf" H 2275 1050 50  0001 C CNN
+F 4 "mfr_pn" H 2175 1300 50  0001 C CNN "manf#"
 	1    2175 1300
 	1    0    0    -1
 $EndComp
 Wire Wire Line
-	1225 1300 1875 1300
-Wire Wire Line
-	1375 1250 1375 1400
+	1225 1300 1375 1300
+Wire Wire Line
+	1375 1250 1375 1300
 Wire Wire Line
 	1675 1300 1675 1400
 Connection ~ 1675 1300
 Wire Wire Line
-	2475 1300 2950 1300
-Wire Wire Line
-	2625 1250 2625 1400
+	2475 1300 2625 1300
+Wire Wire Line
+	2625 1250 2625 1300
 Wire Wire Line
 	2625 2575 2625 1700
 Wire Wire Line
-	1225 2575 2775 2575
+	1225 2575 1375 2575
 Wire Wire Line
 	1375 1800 1375 1700
@@
 Connection ~ 1675 2575
 Wire Wire Line
-	2175 1600 2175 2675
+	2175 1600 2175 2575
 Connection ~ 2175 2575
 Wire Wire Line
@@
 	1975 4550 1975 6025
 Wire Wire Line
-	4375 6025 1325 6025
+	4375 6025 3700 6025
 Wire Wire Line
 	4375 5250 4450 5250
@@
 Connection ~ 1975 6025
 Wire Wire Line
-	1875 4250 2750 4250
+	1875 4250 2325 4250
 Wire Wire Line
 	2325 4250 2325 4800
 Wire Wire Line
-	1875 4350 2850 4350
+	1875 4350 2125 4350
 Wire Wire Line
 	2125 4350 2125 4800
@@
 	4450 5150 4375 5150
 Wire Wire Line
-	4375 5150 4375 6025
-Wire Wire Line
-	3025 3950 4450 3950
+	4375 5150 4375 5250
+Wire Wire Line
+	3025 3950 3250 3950
 Wire Wire Line
 	4375 3950 4375 4050
@@
 	2850 4850 4450 4850
 Wire Wire Line
-	3475 4750 4450 4750
+	3475 4750 3700 4750
 Text Label 7400 4650 2    40   ~ 0
 DCD
@@
 IO15
 Wire Wire Line
-	6800 1350 7675 1350
-Wire Wire Line
-	6800 2250 7675 2250
+	6800 1350 7150 1350
+Wire Wire Line
+	6800 2250 7000 2250
 Wire Wire Line
 	7150 1350 7150 2000
@@
 	7975 2450 7975 2500
 Wire Wire Line
-	7975 2500 10350 2500
-Wire Wire Line
-	7975 1100 10350 1100
+	7975 2500 9250 2500
+Wire Wire Line
+	7975 1100 8925 1100
 Wire Wire Line
 	7975 1100 7975 1150
@@
 $EndComp
 Wire Wire Line
-	8925 1000 8925 1600
+	8925 1000 8925 1100
 Connection ~ 8925 1100
 $Comp
@@
 	9575 2000 9575 1900
 Wire Wire Line
-	8925 2000 9575 2000
+	8925 2000 9250 2000
 Wire Wire Line
 	8925 2000 8925 1900
@@
 Connection ~ 9525 2000
 Wire Wire Line
-	9250 1500 9250 1600
+	9250 1500 9250 1550
 Wire Wire Line
 	9575 1550 9575 1600
 Wire Wire Line
-	9250 1550 9575 1550
+	9250 1550 9525 1550
 Connection ~ 9250 1550
 Wire Wire Line
@@
 	9575 3400 9575 3300
 Wire Wire Line
-	9250 3400 9575 3400
+	9250 3400 9525 3400
 Wire Wire Line
 	9250 3300 9250 3400
@@
 Connection ~ 9525 3400
 Wire Wire Line
-	9250 2900 9250 3000
+	9250 2900 9250 2950
 Wire Wire Line
 	9575 2950 9575 3000
 Wire Wire Line
-	9250 2950 9575 2950
+	9250 2950 9525 2950
 Connection ~ 9250 2950
 Wire Wire Line
@@
 	1    0    0    1
 $EndComp
+Wire Wire Line
+	1675 1300 1875 1300
+Wire Wire Line
+	1675 2575 2175 2575
+Wire Wire Line
+	2175 2575 2175 2675
+Wire Wire Line
+	2175 2575 2625 2575
+Wire Wire Line
+	1375 2575 1675 2575
+Wire Wire Line
+	1375 1300 1675 1300
+Wire Wire Line
+	1375 1300 1375 1400
+Wire Wire Line
+	2625 1300 2950 1300
+Wire Wire Line
+	2625 1300 2625 1400
+Wire Wire Line
+	2125 6025 1975 6025
+Wire Wire Line
+	1975 6025 1325 6025
+Wire Wire Line
+	4375 5250 4375 6025
+Wire Wire Line
+	2325 6025 2125 6025
+Wire Wire Line
+	2125 4350 2850 4350
+Wire Wire Line
+	2325 4250 2750 4250
+Wire Wire Line
+	4375 3950 4450 3950
+Wire Wire Line
+	3025 6025 2325 6025
+Wire Wire Line
+	3250 6025 3025 6025
+Wire Wire Line
+	3475 6025 3250 6025
+Wire Wire Line
+	3700 6025 3475 6025
+Wire Wire Line
+	3250 3950 4375 3950
+Wire Wire Line
+	3700 4750 4450 4750
+Wire Wire Line
+	7150 1350 7675 1350
+Wire Wire Line
+	7000 2250 7675 2250
+Wire Wire Line
+	8925 1100 9250 1100
+Wire Wire Line
+	8925 1100 8925 1600
+Wire Wire Line
+	9250 2000 9525 2000
+Wire Wire Line
+	9525 2000 9575 2000
+Wire Wire Line
+	9250 1550 9250 1600
+Wire Wire Line
+	9525 1550 9575 1550
+Wire Wire Line
+	9250 1100 10350 1100
+Wire Wire Line
+	9525 3400 9575 3400
+Wire Wire Line
+	9250 2950 9250 3000
+Wire Wire Line
+	9525 2950 9575 2950
+Wire Wire Line
+	9250 2500 10350 2500
+Wire Wire Line
+	2625 2575 2775 2575
 $EndSCHEMATC

Commit message: PCB cleanup
Parts:
- JP1: value PWR_LED_EN -> LED_PWR_EN
Changed lines of the file:
@@
 P 1375 2300
 F 0 "JP1" V 1375 2250 40  0000 R CNN
-F 1 "PWR_LED_EN" H 1550 2400 40  0000 R CNN
+F 1 "LED_PWR_EN" H 1550 2400 40  0000 R CNN
 F 2 "chromogram_libs:R_0402" H 1375 2300 50  0001 C CNN
 F 3 "" H 1375 2300 50  0001 C CNN

Commit message: modified diode footprints
Parts:
- D3, D4: footprint chromogram_libs:D_SOD-123 -> chromogram_libs:D_LLP1006-2L
- R4: value 2k -> 1k
- U131: value AP1117-15 -> 1117-33
Changed lines of the file:
@@
 P 1375 1550
 F 0 "R4" H 1400 1400 40  0000 L CNN
-F 1 "2k" V 1375 1475 40  0000 L CNN
+F 1 "1k" V 1375 1475 40  0000 L CNN
 F 2 "chromogram_libs:r_0805" V 1305 1550 30  0001 C CNN
 F 3 "" H 1375 1550 30  0000 C CNN
@@
 P 2175 1300
 F 0 "U131" H 2175 1540 50  0000 C CNN
-F 1 "AP1117-15" H 2175 1450 50  0000 C CNN
+F 1 "1117-33" H 2175 1450 50  0000 C CNN
 F 2 "chromogram_libs:SOT-223-3_TabPin2" H 2175 1500 50  0001 C CNN
 F 3 "http://www.diodes.com/datasheets/AP1117.pdf" H 2275 1050 50  0001 C CNN
@@
 F 0 "D3" V 2225 4925 40  0000 R CNN
 F 1 "VESD05A1B" H 2025 4900 40  0000 R CNN
-F 2 "chromogram_libs:D_SOD-123" H 2125 4950 60  0001 C CNN
+F 2 "chromogram_libs:D_LLP1006-2L" H 2125 4950 60  0001 C CNN
 F 3 "" H 2125 4950 60  0000 C CNN
 	1    2125 4950
@@
 F 0 "D4" V 2425 4925 40  0000 R CNN
 F 1 "VESD05A1B" H 2225 4900 40  0000 R CNN
-F 2 "chromogram_libs:D_SOD-123" H 2325 4950 60  0001 C CNN
+F 2 "chromogram_libs:D_LLP1006-2L" H 2325 4950 60  0001 C CNN
 F 3 "" H 2325 4950 60  0000 C CNN
 	1    2325 4950
