File: kicad/esp_pwr_uart.sch (KiCad schematic (older format))
At the start: 29 parts, among them P1 USB_micro, Q1 DDC114TU, U131 1117-33, U132 CP2102N-A01-GQFN28

Commit message: renamed all files, fresh Gerbers
Parts:
- C17, C18, C23, C25: footprint chromogram_libs:c_2917 -> KlokTHREEjr_libs:c_2917; symbol chromogram:C_POL -> KlokTHREEjr:C_POL
- C19, C20, C21, C24, C26: footprint chromogram_libs:c_0805 -> KlokTHREEjr_libs:c_0805; symbol chromogram:C_NP -> KlokTHREEjr:C_NP
- D1: footprint chromogram_libs:D_SOD-123 -> KlokTHREEjr_libs:D_SOD-123; symbol chromogram:diode_zener -> KlokTHREEjr:diode_zener
- D2: footprint chromogram_libs:LED-0805 -> KlokTHREEjr_libs:LED-0805; symbol chromogram:LED -> KlokTHREEjr:LED
- D3, D4: footprint chromogram_libs:D_LLP1006-2L -> KlokTHREEjr_libs:D_LLP1006-2L; symbol chromogram:diode_sch -> KlokTHREEjr:diode_sch
- JP1: footprint chromogram_libs:R_0402 -> KlokTHREEjr_libs:R_0402; symbol chromogram:Jumper_NC_Small -> KlokTHREEjr:Jumper_NC_Small
- P1: footprint chromogram_libs:USB_Micro-B_Molex-105017-0001 -> KlokTHREEjr_libs:USB_Micro-B_Molex-105017-0001; symbol chromogram:USB_micro -> KlokTHREEjr:USB_micro
- Q1: footprint chromogram_libs:SOT-363_SC-70-6 -> KlokTHREEjr_libs:SOT-363_SC-70-6; symbol chromogram:DDC114TU -> KlokTHREEjr:DDC114TU
- R16, R18, R19, R20, R21, R22, R23, R3, R4: footprint chromogram_libs:r_0805 -> KlokTHREEjr_libs:r_0805; symbol chromogram:R -> KlokTHREEjr:R
- S3, S4: footprint chromogram_libs:SW_SMD -> KlokTHREEjr_libs:SW_SMD; symbol chromogram:SW-SPST-M -> KlokTHREEjr:SW-SPST-M
- U131: footprint chromogram_libs:SOT-223-3_TabPin2 -> KlokTHREEjr_libs:SOT-223-3_TabPin2; symbol chromogram:AP1117-15 -> KlokTHREEjr:AP1117-15
- U132: footprint chromogram_libs:QFN-28-1EP_5x5mm_Pitch0.5mm -> KlokTHREEjr_libs:QFN-28-1EP_5x5mm_Pitch0.5mm; symbol chromogram:CP2102N-A01-GQFN28 -> KlokTHREEjr:CP2102N-A01-GQFN28

Commit message: KlokTHREEjr final. Kontroller pending
Parts:
- added G7: LOGO_WL, KlokTHREEjr_libs:Logo-WL3, symbol KlokTHREEjr:LOGO_WL
- added G8: KiCad, KlokTHREEjr_libs:KiCad-Logo2_6mm_SilkScreen, symbol KlokTHREEjr:KiCad
- added G9: OSHW, KlokTHREEjr_libs:OSHW_6mm, symbol KlokTHREEjr:OSHW
- S3: value EN -> SW-EN
- S4: value BOOT -> SW-BOOT
Changed lines of the file:
@@
 P 9575 1750
 F 0 "S3" V 9525 1975 40  0000 C CNB
-F 1 "EN" V 9625 1975 40  0000 C CNB
+F 1 "SW-EN" V 9625 2050 40  0000 C CNB
 F 2 "KlokTHREEjr_libs:SW_SMD" H 9575 1750 60  0001 C CNN
 F 3 "" H 9575 1750 60  0000 C CNN
@@
 P 9575 3150
 F 0 "S4" V 9525 3375 40  0000 C CNB
-F 1 "BOOT" V 9625 3425 40  0000 C CNB
+F 1 "SW-BOOT" V 9650 3475 40  0000 C CNB
 F 2 "KlokTHREEjr_libs:SW_SMD" H 9575 3150 60  0001 C CNN
 F 3 "" H 9575 3150 60  0000 C CNN
@@
 Wire Wire Line
 	2625 2575 2775 2575
+$Comp
+L KlokTHREEjr:OSHW G9
+U 1 1 5AA76142
+P 10825 7000
+F 0 "G9" H 10825 6950 40  0001 C CNN
+F 1 "OSHW" H 10825 7100 40  0001 C CNN
+F 2 "KlokTHREEjr_libs:OSHW_6mm" H 11250 7000 60  0001 L CNN
+F 3 "" H 10825 7000 60  0000 C CNN
+F 4 "mfr_pn" H 10825 7000 50  0001 C CNN "manf#"
+	1    10825 7000
+	1    0    0    -1
+$EndComp
+$Comp
+L KlokTHREEjr:KiCad G8
+U 1 1 5AA75FE2
+P 9725 6850
+F 0 "G8" H 9725 6582 60  0001 C CNN
+F 1 "KiCad" H 9725 7118 60  0001 C CNN
+F 2 "KlokTHREEjr_libs:KiCad-Logo2_6mm_SilkScreen" H 9725 6850 60  0001 C CNN
+F 3 "" H 9725 6850 60  0001 C CNN
+F 4 "mfr_pn" H 9725 6850 50  0001 C CNN "manf#"
+	1    9725 6850
+	1    0    0    -1
+$EndComp
+$Comp
+L KlokTHREEjr:LOGO_WL G7
+U 1 1 5AA760BF
+P 8700 6775
+F 0 "G7" H 8700 6639 60  0001 C CNN
+F 1 "LOGO_WL" H 8700 6911 60  0001 C CNN
+F 2 "KlokTHREEjr_libs:Logo-WL3" H 8700 6775 60  0001 C CNN
+F 3 "" H 8700 6775 60  0001 C CNN
+F 4 "mfr_pn" H 8700 6775 50  0001 C CNN "manf#"
+	1    8700 6775
+	1    0    0    -1
+$EndComp
 $EndSCHEMATC

Commit message: USB protection, LDR, Switches reconfigured
Parts:
- removed D1: 1N5819, KlokTHREEjr_libs:D_SOD-123, symbol KlokTHREEjr:diode_zener
- removed D3, D4: VESD05A1B, KlokTHREEjr_libs:D_LLP1006-2L, symbol KlokTHREEjr:diode_sch
- added D1: RClamp0854P.TCT, KlokTHREEjr_libs:SOT-143, symbol KlokTHREEjr:Diode_TVS
- added L1: 330E, KlokTHREEjr_libs:r_0805, symbol KlokTHREEjr:IND_FERRITE_BEAD
Changed lines of the file:
@@
 	1    0    0    -1
 $EndComp
-$Comp
-L KlokTHREEjr:diode_sch D3
-U 1 1 5A73F3F4
-P 2125 4950
-F 0 "D3" V 2225 4925 40  0000 R CNN
-F 1 "VESD05A1B" H 2025 4900 40  0000 R CNN
-F 2 "KlokTHREEjr_libs:D_LLP1006-2L" H 2125 4950 60  0001 C CNN
-F 3 "" H 2125 4950 60  0000 C CNN
-	1    2125 4950
-	0    -1   -1   0
-$EndComp
-$Comp
-L KlokTHREEjr:diode_sch D4
-U 1 1 5A73F4E3
-P 2325 4950
-F 0 "D4" V 2425 4925 40  0000 R CNN
-F 1 "VESD05A1B" H 2225 4900 40  0000 R CNN
-F 2 "KlokTHREEjr_libs:D_LLP1006-2L" H 2325 4950 60  0001 C CNN
-F 3 "" H 2325 4950 60  0000 C CNN
-	1    2325 4950
-	0    -1   -1   0
-$EndComp
-$Comp
-L KlokTHREEjr:diode_zener D1
-U 1 1 5A73F53E
-P 2125 3850
-F 0 "D1" V 2170 3795 40  0000 R CNN
-F 1 "1N5819" V 2080 3795 40  0000 R CNN
-F 2 "KlokTHREEjr_libs:D_SOD-123" H 1950 3875 60  0001 C CNN
-F 3 "" H 1950 3875 60  0000 C CNN
-	1    2125 3850
-	0    -1   -1   0
-$EndComp
-Wire Wire Line
-	2125 4000 2125 4150
-Wire Wire Line
-	2125 4150 1875 4150
+Wire Wire Line
+	2175 4000 2175 4150
+Wire Wire Line
+	2175 4150 1875 4150
 Wire Wire Line
 	1875 4550 1975 4550
@@
 Wire Wire Line
 	4375 5250 4450 5250
-Wire Wire Line
-	2325 6025 2325 5100
-Wire Wire Line
-	2125 6025 2125 5100
-Connection ~ 2125 6025
-Wire Wire Line
-	1325 6025 1325 4700
 Connection ~ 1975 6025
-Wire Wire Line
-	1875 4250 2325 4250
-Wire Wire Line
-	2325 4250 2325 4800
-Wire Wire Line
-	1875 4350 2125 4350
-Wire Wire Line
-	2125 4350 2125 4800
 NoConn ~ 1875 4450
-Wire Wire Line
-	2125 3700 2125 3625
-Text Label 2125 3625 2    40   ~ 0
+Text Label 2825 4000 2    40   ~ 0
 5V
 Wire Wire Line
@@
 RI
 Connection ~ 4375 5250
-Connection ~ 2325 6025
 Wire Wire Line
 	2850 4350 2850 4850
-Connection ~ 2125 4350
 Wire Wire Line
 	2750 4250 2750 4950
-Connection ~ 2325 4250
 Text Label 4100 4850 0    40   ~ 0
 USB_D+
@@
 	2625 1300 2625 1400
 Wire Wire Line
-	2125 6025 1975 6025
-Wire Wire Line
 	1975 6025 1325 6025
 Wire Wire Line
 	4375 5250 4375 6025
 Wire Wire Line
-	2325 6025 2125 6025
-Wire Wire Line
-	2125 4350 2850 4350
-Wire Wire Line
-	2325 4250 2750 4250
-Wire Wire Line
 	4375 3950 4450 3950
-Wire Wire Line
-	3025 6025 2325 6025
 Wire Wire Line
 	3250 6025 3025 6025
@@
 	1    0    0    -1
 $EndComp
+$Comp
+L KlokTHREEjr:Diode_TVS D1
+U 1 1 5AFE0C2C
+P 2275 5100
+F 0 "D1" H 2500 5000 50  0000 L CNN
+F 1 "RClamp0854P.TCT" H 2200 4900 50  0000 L CNN
+F 2 "KlokTHREEjr_libs:SOT-143" H 2275 5100 50  0001 C CNN
+F 3 "" H 2275 5100 50  0001 C CNN
+	1    2275 5100
+	1    0    0    -1
+$EndComp
+Wire Wire Line
+	1975 6025 2175 6025
+Wire Wire Line
+	1875 4350 2425 4350
+Wire Wire Line
+	1875 4250 2325 4250
+Wire Wire Line
+	2175 4850 2175 4150
+Connection ~ 2175 4150
+Wire Wire Line
+	2325 4850 2325 4250
+Connection ~ 2325 4250
+Wire Wire Line
+	2325 4250 2750 4250
+Wire Wire Line
+	2425 4850 2425 4350
+Connection ~ 2425 4350
+Wire Wire Line
+	2425 4350 2850 4350
+Wire Wire Line
+	2175 5350 2175 6025
+Connection ~ 2175 6025
+Wire Wire Line
+	2175 6025 3025 6025
+$Comp
+L KlokTHREEjr:IND_FERRITE_BEAD L1
+U 1 1 5AFF9108
+P 2450 4000
+F 0 "L1" H 2450 4175 40  0000 C CNN
+F 1 "330E" H 2450 4100 40  0000 C CNN
+F 2 "KlokTHREEjr_libs:r_0805" H 2450 4000 60  0001 C CNN
+F 3 "" H 2415 4090 60  0000 C CNN
+	1    2450 4000
+	1    0    0    -1
+$EndComp
+Wire Wire Line
+	2175 4000 2250 4000
+Wire Wire Line
+	2650 4000 2825 4000
+Wire Wire Line
+	1325 4700 1325 6025
 $EndSCHEMATC

Commit message: ready for seeed submission
Parts:
- added L2: 330E, KlokTHREEjr_libs:r_0805, symbol KlokTHREEjr:IND_FERRITE_BEAD
Connections:
- wire segments 128 -> 129
Changed lines of the file:
@@
 Wire Wire Line
 	2650 4000 2825 4000
+$Comp
+L KlokTHREEjr:IND_FERRITE_BEAD L2
+U 1 1 5AB0DB2F
+P 1325 5100
+F 0 "L2" V 1200 5200 40  0000 C CNN
+F 1 "330E" V 1275 5250 40  0000 C CNN
+F 2 "KlokTHREEjr_libs:r_0805" H 1325 5100 60  0001 C CNN
+F 3 "" H 1290 5190 60  0000 C CNN
+	1    1325 5100
+	0    1    1    0
+$EndComp
 Wire Wire Line
-	1325 4700 1325 6025
+	1325 4700 1325 4900
+Wire Wire Line
+	1325 5300 1325 6025
 $EndSCHEMATC
