File: kicad/rtc_ds3231.sch (KiCad schematic (older format))
At the start: 7 parts, among them U130 DS3231N

Commit message: schematic WIP
Parts:
- removed C22: 100n, chromogram_libs:c_0805, symbol chromogram:CAP_NP
- added C22: 100nF, symbol chromogram:C_NP
Connections:
- wire segments 35 -> 54
Other:
- note removed: "RTC"
Changed lines of the file:
@@
-EESchema Schematic File Version 2
-LIBS:power
+EESchema Schematic File Version 4
 LIBS:chromogram-cache
-EELAYER 25 0
+EELAYER 26 0
 EELAYER END
 $Descr A4 11693 8268
 encoding utf-8
-Sheet 11 11
+Sheet 11 12
 Title ""
 Date ""
@@
 Comment4 ""
 $EndDescr
-Text Notes 1800 4225 0    40   ~ 8
-RTC
-$Comp
-L chromogram:CAP_NP C22
-U 1 1 5A44891D
-P 2175 3225
-F 0 "C22" H 2250 3325 40  0000 C CNN
-F 1 "100n" H 2275 3150 40  0000 C CNN
-F 2 "chromogram_libs:c_0805" H 2175 3225 60  0001 C CNN
-F 3 "" H 2175 3225 60  0000 C CNN
-	1    2175 3225
-	1    0    0    -1
-$EndComp
 $Comp
 L chromogram:R R8
@@
 Connection ~ 4650 2250
 Wire Wire Line
-	4650 2250 4650 2325
-Wire Wire Line
-	2525 2250 5575 2250
-Wire Wire Line
-	4800 2250 4800 2325
-Wire Wire Line
-	2000 2350 2000 2975
+	4650 2250 4650 2425
+Wire Wire Line
+	2525 2250 2675 2250
+Wire Wire Line
+	4800 2250 4800 2425
+Wire Wire Line
+	2000 2350 2000 2425
 Wire Wire Line
 	4575 3025 5575 3025
 Wire Wire Line
-	4625 3275 4625 4125
+	4625 3275 4625 3375
 Wire Wire Line
 	4625 3675 4575 3675
@@
 	2000 2425 3425 2425
 Wire Wire Line
-	2000 3425 2000 4125
-Wire Wire Line
-	2175 2875 2175 3125
-Wire Wire Line
-	2000 2875 2175 2875
+	2000 3425 2000 3500
+Wire Wire Line
+	2200 2875 2200 3050
+Wire Wire Line
+	2000 2875 2200 2875
 Connection ~ 2000 2875
 Wire Wire Line
-	2175 3300 2175 3500
-Wire Wire Line
-	2175 3500 2000 3500
+	2200 3350 2200 3500
+Wire Wire Line
+	2200 3500 2000 3500
 Connection ~ 2000 3500
 Connection ~ 2000 2425
 Wire Wire Line
-	2000 4125 5575 4125
-Wire Wire Line
-	3675 4075 3675 4200
+	2000 4125 3675 4125
+Wire Wire Line
+	3675 4075 3675 4125
 Wire Wire Line
 	3875 4125 3875 4075
@@
 Connection ~ 4075 4125
 Wire Wire Line
-	2525 2250 2525 2525
-Wire Wire Line
-	2675 2250 2675 2525
-Wire Wire Line
-	2675 3025 2675 4450
+	2525 2250 2525 2625
+Wire Wire Line
+	2675 2250 2675 2625
+Wire Wire Line
+	2675 2925 2675 3175
 Wire Wire Line
 	2675 3175 2775 3175
 Wire Wire Line
-	2525 3025 2525 4575
+	2525 2925 2525 3325
 Wire Wire Line
 	2525 3325 2775 3325
@@
 	4575 2875 4650 2875
 Wire Wire Line
-	4650 2875 4650 2825
-Wire Wire Line
-	4800 2825 4800 3175
+	4650 2875 4650 2725
+Wire Wire Line
+	4800 2725 4800 3175
 Wire Wire Line
 	4800 3175 4575 3175
@@
 Text HLabel 5575 4575 2    40   Input ~ 0
 SCL
+Wire Wire Line
+	4650 2250 4800 2250
+Wire Wire Line
+	4625 3675 4625 4125
+Wire Wire Line
+	4625 3575 4625 3675
+Wire Wire Line
+	4625 3475 4625 3575
+Wire Wire Line
+	4625 3375 4625 3475
+Wire Wire Line
+	2000 2875 2000 2975
+Wire Wire Line
+	2000 3500 2000 4125
+Wire Wire Line
+	2000 2425 2000 2875
+Wire Wire Line
+	3675 4125 3875 4125
+Wire Wire Line
+	3675 4125 3675 4200
+Wire Wire Line
+	3875 4125 3975 4125
+Wire Wire Line
+	3975 4125 4075 4125
+Wire Wire Line
+	4075 4125 4625 4125
+Wire Wire Line
+	2675 3175 2675 4450
+Wire Wire Line
+	2525 3325 2525 4575
+Wire Wire Line
+	2675 2250 3675 2250
+Wire Wire Line
+	3675 2250 4650 2250
+Wire Wire Line
+	4800 2250 5575 2250
+Wire Wire Line
+	4625 4125 5575 4125
+$Comp
+L chromogram:C_NP C22
+U 1 1 5A613CC0
+P 2200 3200
+F 0 "C22" H 2303 3238 40  0000 L CNN
+F 1 "100nF" H 2303 3163 40  0000 L CNN
+F 2 "" H 2200 3200 60  0000 C CNN
+F 3 "" H 2200 3200 60  0000 C CNN
+	1    2200 3200
+	1    0    0    -1
+$EndComp
 $EndSCHEMATC

Commit message: making progress on schematic
Parts:
- C22: footprint (none) -> chromogram_libs:c_0805
Connections:
- wire segments 54 -> 35
Changed lines of the file:
@@
-EESchema Schematic File Version 4
+EESchema Schematic File Version 2
+LIBS:chromogram
+LIBS:wyolum_kicad_symbols
 LIBS:chromogram-cache
-EELAYER 26 0
+EELAYER 25 0
 EELAYER END
 $Descr A4 11693 8268
@@
 	4650 2250 4650 2425
 Wire Wire Line
-	2525 2250 2675 2250
+	2525 2250 5575 2250
 Wire Wire Line
 	4800 2250 4800 2425
 Wire Wire Line
-	2000 2350 2000 2425
+	2000 2350 2000 2975
 Wire Wire Line
 	4575 3025 5575 3025
 Wire Wire Line
-	4625 3275 4625 3375
+	4625 3275 4625 4125
 Wire Wire Line
 	4625 3675 4575 3675
@@
 	2000 2425 3425 2425
 Wire Wire Line
-	2000 3425 2000 3500
+	2000 3425 2000 4125
 Wire Wire Line
 	2200 2875 2200 3050
@@
 Connection ~ 2000 2425
 Wire Wire Line
-	2000 4125 3675 4125
-Wire Wire Line
-	3675 4075 3675 4125
+	2000 4125 5575 4125
+Wire Wire Line
+	3675 4075 3675 4200
 Wire Wire Line
 	3875 4125 3875 4075
@@
 	2675 2250 2675 2625
 Wire Wire Line
-	2675 2925 2675 3175
+	2675 2925 2675 4450
 Wire Wire Line
 	2675 3175 2775 3175
 Wire Wire Line
-	2525 2925 2525 3325
+	2525 2925 2525 4575
 Wire Wire Line
 	2525 3325 2775 3325
@@
 Text HLabel 5575 4575 2    40   Input ~ 0
 SCL
-Wire Wire Line
-	4650 2250 4800 2250
-Wire Wire Line
-	4625 3675 4625 4125
-Wire Wire Line
-	4625 3575 4625 3675
-Wire Wire Line
-	4625 3475 4625 3575
-Wire Wire Line
-	4625 3375 4625 3475
-Wire Wire Line
-	2000 2875 2000 2975
-Wire Wire Line
-	2000 3500 2000 4125
-Wire Wire Line
-	2000 2425 2000 2875
-Wire Wire Line
-	3675 4125 3875 4125
-Wire Wire Line
-	3675 4125 3675 4200
-Wire Wire Line
-	3875 4125 3975 4125
-Wire Wire Line
-	3975 4125 4075 4125
-Wire Wire Line
-	4075 4125 4625 4125
-Wire Wire Line
-	2675 3175 2675 4450
-Wire Wire Line
-	2525 3325 2525 4575
-Wire Wire Line
-	2675 2250 3675 2250
-Wire Wire Line
-	3675 2250 4650 2250
-Wire Wire Line
-	4800 2250 5575 2250
-Wire Wire Line
-	4625 4125 5575 4125
 $Comp
 L chromogram:C_NP C22
@@
 F 0 "C22" H 2303 3238 40  0000 L CNN
 F 1 "100nF" H 2303 3163 40  0000 L CNN
-F 2 "" H 2200 3200 60  0000 C CNN
+F 2 "chromogram_libs:c_0805" H 2200 3200 60  0001 C CNN
 F 3 "" H 2200 3200 60  0000 C CNN
 	1    2200 3200

Commit message: WIP schematic
Connections:
- wire segments 35 -> 54
Changed lines of the file:
@@
-EESchema Schematic File Version 2
+EESchema Schematic File Version 4
 LIBS:chromogram
-LIBS:wyolum_kicad_symbols
 LIBS:chromogram-cache
-EELAYER 25 0
+EELAYER 26 0
 EELAYER END
 $Descr A4 11693 8268
@@
 	4650 2250 4650 2425
 Wire Wire Line
-	2525 2250 5575 2250
+	2525 2250 2675 2250
 Wire Wire Line
 	4800 2250 4800 2425
 Wire Wire Line
-	2000 2350 2000 2975
+	2000 2350 2000 2425
 Wire Wire Line
 	4575 3025 5575 3025
 Wire Wire Line
-	4625 3275 4625 4125
+	4625 3275 4625 3375
 Wire Wire Line
 	4625 3675 4575 3675
@@
 	2000 2425 3425 2425
 Wire Wire Line
-	2000 3425 2000 4125
+	2000 3425 2000 3500
 Wire Wire Line
 	2200 2875 2200 3050
@@
 Connection ~ 2000 2425
 Wire Wire Line
-	2000 4125 5575 4125
-Wire Wire Line
-	3675 4075 3675 4200
+	2000 4125 3675 4125
+Wire Wire Line
+	3675 4075 3675 4125
 Wire Wire Line
 	3875 4125 3875 4075
@@
 	2675 2250 2675 2625
 Wire Wire Line
-	2675 2925 2675 4450
+	2675 2925 2675 3175
 Wire Wire Line
 	2675 3175 2775 3175
 Wire Wire Line
-	2525 2925 2525 4575
+	2525 2925 2525 3325
 Wire Wire Line
 	2525 3325 2775 3325
@@
 	1    0    0    -1
 $EndComp
+Wire Wire Line
+	4650 2250 4800 2250
+Wire Wire Line
+	4625 3675 4625 4125
+Wire Wire Line
+	4625 3575 4625 3675
+Wire Wire Line
+	4625 3475 4625 3575
+Wire Wire Line
+	4625 3375 4625 3475
+Wire Wire Line
+	2000 2875 2000 2975
+Wire Wire Line
+	2000 3500 2000 4125
+Wire Wire Line
+	2000 2425 2000 2875
+Wire Wire Line
+	3675 4125 3875 4125
+Wire Wire Line
+	3675 4125 3675 4200
+Wire Wire Line
+	3875 4125 3975 4125
+Wire Wire Line
+	3975 4125 4075 4125
+Wire Wire Line
+	4075 4125 4625 4125
+Wire Wire Line
+	2675 3175 2675 4450
+Wire Wire Line
+	2525 3325 2525 4575
+Wire Wire Line
+	2675 2250 3675 2250
+Wire Wire Line
+	3675 2250 4650 2250
+Wire Wire Line
+	4800 2250 5575 2250
+Wire Wire Line
+	4625 4125 5575 4125
 $EndSCHEMATC

Commit message: making progress on PCB
Connections:
- wire segments 54 -> 35
Changed lines of the file:
@@
-EESchema Schematic File Version 4
+EESchema Schematic File Version 2
 LIBS:chromogram
+LIBS:wyolum_kicad_symbols
 LIBS:chromogram-cache
-EELAYER 26 0
+EELAYER 25 0
 EELAYER END
 $Descr A4 11693 8268
@@
 	4650 2250 4650 2425
 Wire Wire Line
-	2525 2250 2675 2250
+	2525 2250 5575 2250
 Wire Wire Line
 	4800 2250 4800 2425
 Wire Wire Line
-	2000 2350 2000 2425
+	2000 2350 2000 2975
 Wire Wire Line
 	4575 3025 5575 3025
 Wire Wire Line
-	4625 3275 4625 3375
+	4625 3275 4625 4125
 Wire Wire Line
 	4625 3675 4575 3675
@@
 	2000 2425 3425 2425
 Wire Wire Line
-	2000 3425 2000 3500
+	2000 3425 2000 4125
 Wire Wire Line
 	2200 2875 2200 3050
@@
 Connection ~ 2000 2425
 Wire Wire Line
-	2000 4125 3675 4125
-Wire Wire Line
-	3675 4075 3675 4125
+	2000 4125 5575 4125
+Wire Wire Line
+	3675 4075 3675 4200
 Wire Wire Line
 	3875 4125 3875 4075
@@
 	2675 2250 2675 2625
 Wire Wire Line
-	2675 2925 2675 3175
+	2675 2925 2675 4450
 Wire Wire Line
 	2675 3175 2775 3175
 Wire Wire Line
-	2525 2925 2525 3325
+	2525 2925 2525 4575
 Wire Wire Line
 	2525 3325 2775 3325
@@
 	1    0    0    -1
 $EndComp
-Wire Wire Line
-	4650 2250 4800 2250
-Wire Wire Line
-	4625 3675 4625 4125
-Wire Wire Line
-	4625 3575 4625 3675
-Wire Wire Line
-	4625 3475 4625 3575
-Wire Wire Line
-	4625 3375 4625 3475
-Wire Wire Line
-	2000 2875 2000 2975
-Wire Wire Line
-	2000 3500 2000 4125
-Wire Wire Line
-	2000 2425 2000 2875
-Wire Wire Line
-	3675 4125 3875 4125
-Wire Wire Line
-	3675 4125 3675 4200
-Wire Wire Line
-	3875 4125 3975 4125
-Wire Wire Line
-	3975 4125 4075 4125
-Wire Wire Line
-	4075 4125 4625 4125
-Wire Wire Line
-	2675 3175 2675 4450
-Wire Wire Line
-	2525 3325 2525 4575
-Wire Wire Line
-	2675 2250 3675 2250
-Wire Wire Line
-	3675 2250 4650 2250
-Wire Wire Line
-	4800 2250 5575 2250
-Wire Wire Line
-	4625 4125 5575 4125
 $EndSCHEMATC

Commit message: WIP PCB layout
Connections:
- wire segments 35 -> 54

Commit message: almost done with PCB
Parts:
- added TP1: ~RST, chromogram_libs:BreakOutPad, symbol chromogram:Conn_01x01
Connections:
- net labels added: 32kHz, SQR
- net labels removed: RST
Changed lines of the file:
@@
 	1    0    0    -1
 $EndComp
-Text Label 5250 4425 0    40   ~ 0
+Text Label 5500 4425 0    40   ~ 0
 SDA
-Text Label 5250 4550 0    40   ~ 0
+Text Label 5500 4550 0    40   ~ 0
 SCL
 $Comp
 L chromogram:R R6
 U 1 1 5A448933
-P 4650 2550
-F 0 "R6" H 4700 2350 40  0000 C CNN
-F 1 "10K" V 4657 2551 40  0000 C CNN
-F 2 "chromogram_libs:r_0805" V 4580 2550 30  0001 C CNN
-F 3 "~" H 4650 2550 30  0000 C CNN
-	1    4650 2550
+P 4900 2550
+F 0 "R6" H 4950 2350 40  0000 C CNN
+F 1 "10K" V 4907 2551 40  0000 C CNN
+F 2 "chromogram_libs:r_0805" V 4830 2550 30  0001 C CNN
+F 3 "~" H 4900 2550 30  0000 C CNN
+	1    4900 2550
 	1    0    0    -1
 $EndComp
@@
 L chromogram:R R7
 U 1 1 5A44893A
-P 4800 2550
-F 0 "R7" H 4850 2350 40  0000 C CNN
-F 1 "10K" V 4807 2551 40  0000 C CNN
-F 2 "chromogram_libs:r_0805" V 4730 2550 30  0001 C CNN
-F 3 "~" H 4800 2550 30  0000 C CNN
-	1    4800 2550
-	1    0    0    -1
-$EndComp
-Text Label 5000 3000 2    40   ~ 0
+P 5050 2550
+F 0 "R7" H 5100 2350 40  0000 C CNN
+F 1 "10K" V 5057 2551 40  0000 C CNN
+F 2 "chromogram_libs:r_0805" V 4980 2550 30  0001 C CNN
+F 3 "~" H 5050 2550 30  0000 C CNN
+	1    5050 2550
+	1    0    0    -1
+$EndComp
+Text Label 4600 3000 0    40   ~ 0
 RESET
 $Comp
@@
 Wire Wire Line
 	3675 2225 3675 2400
-Connection ~ 4650 2225
-Wire Wire Line
-	4650 2225 4650 2400
+Connection ~ 4900 2225
+Wire Wire Line
+	4900 2225 4900 2400
 Wire Wire Line
 	2525 2225 2675 2225
 Wire Wire Line
-	4800 2225 4800 2400
+	5050 2225 5050 2400
 Wire Wire Line
 	2000 2325 2000 2400
 Wire Wire Line
-	4575 3000 5575 3000
+	4575 3000 5600 3000
 Wire Wire Line
 	4625 3250 4625 3350
@@
 	2525 3300 2775 3300
 Wire Wire Line
-	2675 4425 5575 4425
+	2675 4425 5825 4425
 Connection ~ 2675 3150
 Wire Wire Line
-	2525 4550 5575 4550
+	2525 4550 5825 4550
 Connection ~ 2525 3300
 Wire Wire Line
-	4575 2850 4650 2850
-Wire Wire Line
-	4650 2850 4650 2700
-Wire Wire Line
-	4800 2700 4800 3150
-Wire Wire Line
-	4800 3150 4575 3150
+	4575 2850 4900 2850
+Wire Wire Line
+	4900 2850 4900 2700
+Wire Wire Line
+	5050 2700 5050 3150
+Wire Wire Line
+	5050 3150 4575 3150
 Connection ~ 2675 2225
 Connection ~ 3675 2225
-Connection ~ 4800 2225
+Connection ~ 5050 2225
 Connection ~ 4625 4100
-Text HLabel 5575 2225 2    40   Input ~ 0
+Text HLabel 5825 2225 2    40   Input ~ 0
 5V
-Text HLabel 5575 4100 2    40   Input ~ 0
+Text HLabel 5825 4100 2    40   Input ~ 0
 GND
-Text HLabel 5575 3000 2    40   Input ~ 0
-RST
-Text HLabel 5575 4425 2    40   Input ~ 0
+Text HLabel 5825 4425 2    40   Input ~ 0
 SDA
-Text HLabel 5575 4550 2    40   Input ~ 0
+Text HLabel 5825 4550 2    40   Input ~ 0
 SCL
 $Comp
@@
 $EndComp
 Wire Wire Line
-	4650 2225 4800 2225
+	4900 2225 5050 2225
 Wire Wire Line
 	4625 3650 4625 4100
@@
 	2675 2225 3675 2225
 Wire Wire Line
-	3675 2225 4650 2225
-Wire Wire Line
-	4800 2225 5575 2225
-Wire Wire Line
-	4625 4100 5575 4100
+	3675 2225 4900 2225
+Wire Wire Line
+	5050 2225 5825 2225
+Wire Wire Line
+	4625 4100 5825 4100
+$Comp
+L chromogram:Conn_01x01 TP1
+U 1 1 5A48EA43
+P 5800 3000
+F 0 "TP1" H 5925 3100 50  0000 L CNN
+F 1 "~RST" H 5925 2950 50  0000 L CNN
+F 2 "chromogram_libs:BreakOutPad" H 5800 3000 50  0001 C CNN
+F 3 "~" H 5800 3000 50  0001 C CNN
+	1    5800 3000
+	1    0    0    -1
+$EndComp
+Text Label 4600 2850 0    40   ~ 0
+SQR
+Text Label 4600 3150 0    40   ~ 0
+32kHz
 $EndSCHEMATC

Commit message: modified diode footprints
Parts:
- BT1: footprint chromogram_libs:CR2032_SMD -> chromogram_libs:CR2032_SMD2
- R6, R7: value 10K -> 10k
Changed lines of the file:
@@
 P 4900 2550
 F 0 "R6" H 4950 2350 40  0000 C CNN
-F 1 "10K" V 4907 2551 40  0000 C CNN
+F 1 "10k" V 4907 2551 40  0000 C CNN
 F 2 "chromogram_libs:r_0805" V 4830 2550 30  0001 C CNN
 F 3 "~" H 4900 2550 30  0000 C CNN
@@
 P 5050 2550
 F 0 "R7" H 5100 2350 40  0000 C CNN
-F 1 "10K" V 5057 2551 40  0000 C CNN
+F 1 "10k" V 5057 2551 40  0000 C CNN
 F 2 "chromogram_libs:r_0805" V 4980 2550 30  0001 C CNN
 F 3 "~" H 5050 2550 30  0000 C CNN
@@
 F 0 "BT1" V 1900 3125 40  0000 C CNN
 F 1 "Batt_RTC" H 2150 3125 40  0000 C CNN
-F 2 "chromogram_libs:CR2032_SMD" H 2000 3200 60  0001 C CNN
+F 2 "chromogram_libs:CR2032_SMD2" H 2000 3200 60  0001 C CNN
 F 3 "" H 2000 3200 60  0000 C CNN
 F 4 "BU2032SM-HD-GCT-ND " H 2100 3500 60  0001 C CNN "Digikey"
