File: kicad/rtc_ds3231.sch (KiCad schematic (older format))
At the start: 8 parts, among them U130 DS3231N

Commit message: renamed all files, fresh Gerbers
Parts:
- BT1: footprint chromogram_libs:CR2032_SMD2 -> KlokTHREEjr_libs:CR2032_SMD2; symbol chromogram:Batt_RTC -> KlokTHREEjr:Batt_RTC
- C22: footprint chromogram_libs:c_0805 -> KlokTHREEjr_libs:c_0805; symbol chromogram:C_NP -> KlokTHREEjr:C_NP
- R6, R7, R8, R9: footprint chromogram_libs:r_0805 -> KlokTHREEjr_libs:r_0805; symbol chromogram:R -> KlokTHREEjr:R
- TP1: footprint chromogram_libs:BreakOutPad -> KlokTHREEjr_libs:BreakOutPad; symbol chromogram:Conn_01x01 -> KlokTHREEjr:Conn_01x01
- U130: footprint chromogram_libs:DS3231 -> KlokTHREEjr_libs:DS3231; symbol chromogram:DS3231N -> KlokTHREEjr:DS3231N
Changed lines of the file:
@@
 EESchema Schematic File Version 4
-LIBS:chromogram
-LIBS:chromogram-cache
+LIBS:KlokTHREEjr
+LIBS:KlokTHREEjr-cache
 EELAYER 26 0
 EELAYER END
@@
 encoding utf-8
 Sheet 11 12
-Title "Chromogram"
+Title "KlokTHREEjr"
 Date "2017-12-26"
 Rev "rev 1"
-Comp "WyoLum"
-Comment1 "www.wyolum.com"
+Comp "www.wyolum.com"
+Comment1 "https://github.com/wyolum/KlokTHREEjr"
 Comment2 ""
 Comment3 ""
@@
 $EndDescr
 $Comp
-L chromogram:R R8
+L KlokTHREEjr:R R8
 U 1 1 5A448924
 P 2525 2750
 F 0 "R8" H 2575 2550 40  0000 C CNN
 F 1 "4K7" V 2532 2751 40  0000 C CNN
-F 2 "chromogram_libs:r_0805" V 2455 2750 30  0001 C CNN
+F 2 "KlokTHREEjr_libs:r_0805" V 2455 2750 30  0001 C CNN
 F 3 "~" H 2525 2750 30  0000 C CNN
 	1    2525 2750
@@
 $EndComp
 $Comp
-L chromogram:GND #PWR017
+L KlokTHREEjr:GND #PWR017
 U 1 1 5A44892B
 P 3675 4175
@@
 SCL
 $Comp
-L chromogram:R R6
+L KlokTHREEjr:R R6
 U 1 1 5A448933
 P 4900 2550
 F 0 "R6" H 4950 2350 40  0000 C CNN
 F 1 "10k" V 4907 2551 40  0000 C CNN
-F 2 "chromogram_libs:r_0805" V 4830 2550 30  0001 C CNN
+F 2 "KlokTHREEjr_libs:r_0805" V 4830 2550 30  0001 C CNN
 F 3 "~" H 4900 2550 30  0000 C CNN
 	1    4900 2550
@@
 $EndComp
 $Comp
-L chromogram:R R7
+L KlokTHREEjr:R R7
 U 1 1 5A44893A
 P 5050 2550
 F 0 "R7" H 5100 2350 40  0000 C CNN
 F 1 "10k" V 5057 2551 40  0000 C CNN
-F 2 "chromogram_libs:r_0805" V 4980 2550 30  0001 C CNN
+F 2 "KlokTHREEjr_libs:r_0805" V 4980 2550 30  0001 C CNN
 F 3 "~" H 5050 2550 30  0000 C CNN
 	1    5050 2550
@@
 RESET
 $Comp
-L chromogram:PWR_FLAG #FLG018
+L KlokTHREEjr:PWR_FLAG #FLG018
 U 1 1 5A448942
 P 2000 2325
@@
 $EndComp
 $Comp
-L chromogram:DS3231N U130
+L KlokTHREEjr:DS3231N U130
 U 1 1 5A448948
 P 3675 3200
 F 0 "U130" H 3075 3825 40  0000 L CNN
 F 1 "DS3231N" H 3075 3750 40  0000 L CNN
-F 2 "chromogram_libs:DS3231" H 3675 3200 60  0001 C CNN
+F 2 "KlokTHREEjr_libs:DS3231" H 3675 3200 60  0001 C CNN
 F 3 "~" H 3675 3200 60  0000 C CNN
 	1    3675 3200
@@
 $EndComp
 $Comp
-L chromogram:R R9
+L KlokTHREEjr:R R9
 U 1 1 5A44894F
 P 2675 2750
 F 0 "R9" H 2725 2550 40  0000 C CNN
 F 1 "4K7" V 2682 2751 40  0000 C CNN
-F 2 "chromogram_libs:r_0805" V 2605 2750 30  0001 C CNN
+F 2 "KlokTHREEjr_libs:r_0805" V 2605 2750 30  0001 C CNN
 F 3 "~" H 2675 2750 30  0000 C CNN
 	1    2675 2750
@@
 $EndComp
 $Comp
-L chromogram:Batt_RTC BT1
+L KlokTHREEjr:Batt_RTC BT1
 U 1 1 5A448957
 P 2000 3200
 F 0 "BT1" V 1900 3125 40  0000 C CNN
 F 1 "Batt_RTC" H 2150 3125 40  0000 C CNN
-F 2 "chromogram_libs:CR2032_SMD2" H 2000 3200 60  0001 C CNN
+F 2 "KlokTHREEjr_libs:CR2032_SMD2" H 2000 3200 60  0001 C CNN
 F 3 "" H 2000 3200 60  0000 C CNN
 F 4 "BU2032SM-HD-GCT-ND " H 2100 3500 60  0001 C CNN "Digikey"
@@
 SCL
 $Comp
-L chromogram:C_NP C22
+L KlokTHREEjr:C_NP C22
 U 1 1 5A613CC0
 P 2200 3175
 F 0 "C22" H 2303 3213 40  0000 L CNN
 F 1 "100nF" H 2303 3138 40  0000 L CNN
-F 2 "chromogram_libs:c_0805" H 2200 3175 60  0001 C CNN
+F 2 "KlokTHREEjr_libs:c_0805" H 2200 3175 60  0001 C CNN
 F 3 "" H 2200 3175 60  0000 C CNN
 	1    2200 3175
@@
 	4625 4100 5825 4100
 $Comp
-L chromogram:Conn_01x01 TP1
+L KlokTHREEjr:Conn_01x01 TP1
 U 1 1 5A48EA43
 P 5800 3000
 F 0 "TP1" H 5925 3100 50  0000 L CNN
 F 1 "~RST" H 5925 2950 50  0000 L CNN
-F 2 "chromogram_libs:BreakOutPad" H 5800 3000 50  0001 C CNN
+F 2 "KlokTHREEjr_libs:BreakOutPad" H 5800 3000 50  0001 C CNN
 F 3 "~" H 5800 3000 50  0001 C CNN
 	1    5800 3000

Commit message: added voltage translation ckt for I2C 3V3 to 5V
Parts:
- added C29, C30: 100nF, KlokTHREEjr_libs:c_0805, symbol KlokTHREEjr:C_NP
- added R5: 10k, KlokTHREEjr_libs:r_0805, symbol KlokTHREEjr:R
- added U133: TXB0102DCU, KlokTHREEjr_libs:VSSOP-8_2.4x2.1mm_Pitch0.5mm, symbol KlokTHREEjr:TXB0102DCU
Connections:
- net labels added: 3V3, SCL_5V, SDA_5V
- wire segments 54 -> 77
Other:
- note added: "LEVEL TRANSLATOR\nFOR I2C 5V TO 3V3"
Changed lines of the file:
@@
 	1    0    0    -1
 $EndComp
-Text Label 5500 4425 0    40   ~ 0
-SDA
-Text Label 5500 4550 0    40   ~ 0
-SCL
+Text Label 5825 5225 0    40   ~ 0
+SDA_5V
+Text Label 5825 5025 0    40   ~ 0
+SCL_5V
 $Comp
 L KlokTHREEjr:R R6
@@
 	2000 2325 2000 2400
 Wire Wire Line
-	4575 3000 5600 3000
+	4575 3000 7550 3000
 Wire Wire Line
 	4625 3250 4625 3350
@@
 Wire Wire Line
 	2525 3300 2775 3300
-Wire Wire Line
-	2675 4425 5825 4425
 Connection ~ 2675 3150
-Wire Wire Line
-	2525 4550 5825 4550
 Connection ~ 2525 3300
 Wire Wire Line
@@
 Connection ~ 5050 2225
 Connection ~ 4625 4100
-Text HLabel 5825 2225 2    40   Input ~ 0
+Text HLabel 7775 2225 2    40   Input ~ 0
 5V
-Text HLabel 5825 4100 2    40   Input ~ 0
-GND
-Text HLabel 5825 4425 2    40   Input ~ 0
+Text HLabel 7775 4100 2    40   Input ~ 0
+GND
+Text HLabel 7775 5225 2    40   Input ~ 0
 SDA
-Text HLabel 5825 4550 2    40   Input ~ 0
+Text HLabel 7775 5025 2    40   Input ~ 0
 SCL
 $Comp
@@
 	4075 4100 4625 4100
 Wire Wire Line
-	2675 3150 2675 4425
-Wire Wire Line
-	2525 3300 2525 4550
+	2675 3150 2675 5025
+Wire Wire Line
+	2525 3300 2525 5225
 Wire Wire Line
 	2675 2225 3675 2225
@@
 	3675 2225 4900 2225
 Wire Wire Line
-	5050 2225 5825 2225
-Wire Wire Line
-	4625 4100 5825 4100
+	5050 2225 7775 2225
+Wire Wire Line
+	4625 4100 7775 4100
 $Comp
 L KlokTHREEjr:Conn_01x01 TP1
 U 1 1 5A48EA43
-P 5800 3000
-F 0 "TP1" H 5925 3100 50  0000 L CNN
-F 1 "~RST" H 5925 2950 50  0000 L CNN
-F 2 "KlokTHREEjr_libs:BreakOutPad" H 5800 3000 50  0001 C CNN
-F 3 "~" H 5800 3000 50  0001 C CNN
-	1    5800 3000
+P 7750 3000
+F 0 "TP1" H 7875 3100 50  0000 L CNN
+F 1 "~RST" H 7875 2950 50  0000 L CNN
+F 2 "KlokTHREEjr_libs:BreakOutPad" H 7750 3000 50  0001 C CNN
+F 3 "~" H 7750 3000 50  0001 C CNN
+	1    7750 3000
 	1    0    0    -1
 $EndComp
@@
 Text Label 4600 3150 0    40   ~ 0
 32kHz
+$Comp
+L KlokTHREEjr:TXB0102DCU U133
+U 1 1 5A57AF6A
+P 6600 5125
+F 0 "U133" H 6950 4825 50  0000 L CNN
+F 1 "TXB0102DCU" H 6950 4750 50  0000 L CNN
+F 2 "KlokTHREEjr_libs:VSSOP-8_2.4x2.1mm_Pitch0.5mm" H 7600 4525 50  0001 C CNN
+F 3 "http://www.ti.com/lit/ds/symlink/txb0102.pdf" H 6600 5095 50  0001 C CNN
+	1    6600 5125
+	-1   0    0    -1
+$EndComp
+Wire Wire Line
+	7775 5025 7000 5025
+Wire Wire Line
+	7000 5225 7775 5225
+Text Label 7050 5225 0    40   ~ 0
+SDA
+Text Label 7050 5025 0    40   ~ 0
+SCL
+Wire Wire Line
+	6500 4625 6500 4475
+Wire Wire Line
+	6700 4625 6700 4475
+Wire Wire Line
+	6700 4475 7300 4475
+Text Label 6425 4475 0    40   ~ 0
+5V
+Wire Wire Line
+	6600 5625 6600 5925
+Text Label 6600 6100 0    40   ~ 0
+GND
+Text Label 6700 4475 0    40   ~ 0
+3V3
+Text HLabel 7775 4475 2    40   Input ~ 0
+3V3
+Text Notes 6250 5725 2    50   ~ 10
+LEVEL TRANSLATOR\nFOR I2C 5V TO 3V3
+$Comp
+L KlokTHREEjr:R R5
+U 1 1 5A59C780
+P 7300 5675
+F 0 "R5" H 7350 5475 40  0000 C CNN
+F 1 "10k" V 7307 5676 40  0000 C CNN
+F 2 "KlokTHREEjr_libs:r_0805" V 7230 5675 30  0001 C CNN
+F 3 "~" H 7300 5675 30  0000 C CNN
+	1    7300 5675
+	1    0    0    -1
+$EndComp
+Wire Wire Line
+	7000 5425 7300 5425
+Wire Wire Line
+	7300 5425 7300 5525
+Wire Wire Line
+	7300 5825 7300 5925
+Wire Wire Line
+	7300 5925 6600 5925
+Connection ~ 6600 5925
+Wire Wire Line
+	6600 5925 6600 6100
+Wire Wire Line
+	7300 5425 7300 4475
+Connection ~ 7300 5425
+Connection ~ 7300 4475
+Wire Wire Line
+	7300 4475 7500 4475
+$Comp
+L KlokTHREEjr:C_NP C29
+U 1 1 5A5A129F
+P 5725 4650
+F 0 "C29" H 5828 4688 40  0000 L CNN
+F 1 "100nF" H 5828 4613 40  0000 L CNN
+F 2 "KlokTHREEjr_libs:c_0805" H 5725 4650 60  0001 C CNN
+F 3 "" H 5725 4650 60  0000 C CNN
+	1    5725 4650
+	1    0    0    -1
+$EndComp
+$Comp
+L KlokTHREEjr:C_NP C30
+U 1 1 5A5A13BD
+P 7500 4650
+F 0 "C30" H 7603 4688 40  0000 L CNN
+F 1 "100nF" H 7603 4613 40  0000 L CNN
+F 2 "KlokTHREEjr_libs:c_0805" H 7500 4650 60  0001 C CNN
+F 3 "" H 7500 4650 60  0000 C CNN
+	1    7500 4650
+	1    0    0    -1
+$EndComp
+Wire Wire Line
+	7500 4500 7500 4475
+Connection ~ 7500 4475
+Wire Wire Line
+	7500 4475 7775 4475
+Wire Wire Line
+	5725 4475 5725 4500
+Wire Wire Line
+	5725 4475 6500 4475
+Wire Wire Line
+	5725 4800 5725 4900
+Wire Wire Line
+	7500 4900 7500 4800
+Text Label 5725 4900 0    40   ~ 0
+GND
+Text Label 7500 4900 0    40   ~ 0
+GND
+Wire Wire Line
+	6200 5025 5100 5025
+Wire Wire Line
+	5100 5225 6200 5225
+Wire Wire Line
+	5100 5225 4900 5025
+Wire Wire Line
+	4900 5025 2675 5025
+Wire Wire Line
+	5100 5025 4900 5225
+Wire Wire Line
+	4900 5225 2525 5225
 $EndSCHEMATC

Commit message: removed voltage translation ckt for I2C, added I2C header
Parts:
- removed C29, C30: 100nF, KlokTHREEjr_libs:c_0805, symbol KlokTHREEjr:C_NP
- removed R5: 10k, KlokTHREEjr_libs:r_0805, symbol KlokTHREEjr:R
- removed U133: TXB0102DCU, KlokTHREEjr_libs:VSSOP-8_2.4x2.1mm_Pitch0.5mm, symbol KlokTHREEjr:TXB0102DCU
- added TP2: SQR, KlokTHREEjr_libs:BreakOutPad, symbol KlokTHREEjr:Conn_01x01
- added TP3: 32kHz, KlokTHREEjr_libs:BreakOutPad, symbol KlokTHREEjr:Conn_01x01
Connections:
- net labels removed: 5V, SCL_5V, SDA_5V
- wire segments 77 -> 56
Other:
- note removed: "LEVEL TRANSLATOR\nFOR I2C 5V TO 3V3"
Changed lines of the file:
@@
 	1    0    0    -1
 $EndComp
-Text Label 5825 5225 0    40   ~ 0
-SDA_5V
-Text Label 5825 5025 0    40   ~ 0
-SCL_5V
 $Comp
 L KlokTHREEjr:R R6
@@
 Text Label 2075 2400 0    40   ~ 0
 BAT
-Text Label 2525 2225 0    40   ~ 0
-5V
-Text Label 2050 4100 0    40   ~ 0
+Text Label 7225 2225 0    40   ~ 0
+3V3
+Text Label 7225 4100 0    40   ~ 0
 GND
 Wire Wire Line
@@
 Connection ~ 4625 4100
 Text HLabel 7775 2225 2    40   Input ~ 0
-5V
+3V3
 Text HLabel 7775 4100 2    40   Input ~ 0
 GND
+Text HLabel 7775 5025 2    40   Input ~ 0
+SDA
 Text HLabel 7775 5225 2    40   Input ~ 0
-SDA
-Text HLabel 7775 5025 2    40   Input ~ 0
 SCL
 $Comp
@@
 U 1 1 5A48EA43
 P 7750 3000
-F 0 "TP1" H 7875 3100 50  0000 L CNN
-F 1 "~RST" H 7875 2950 50  0000 L CNN
+F 0 "TP1" H 7825 3000 50  0000 L CNN
+F 1 "~RST" H 8000 3000 50  0000 L CNN
 F 2 "KlokTHREEjr_libs:BreakOutPad" H 7750 3000 50  0001 C CNN
 F 3 "~" H 7750 3000 50  0001 C CNN
@@
 Text Label 4600 3150 0    40   ~ 0
 32kHz
-$Comp
-L KlokTHREEjr:TXB0102DCU U133
-U 1 1 5A57AF6A
-P 6600 5125
-F 0 "U133" H 6950 4825 50  0000 L CNN
-F 1 "TXB0102DCU" H 6950 4750 50  0000 L CNN
-F 2 "KlokTHREEjr_libs:VSSOP-8_2.4x2.1mm_Pitch0.5mm" H 7600 4525 50  0001 C CNN
-F 3 "http://www.ti.com/lit/ds/symlink/txb0102.pdf" H 6600 5095 50  0001 C CNN
-	1    6600 5125
-	-1   0    0    -1
-$EndComp
-Wire Wire Line
-	7775 5025 7000 5025
-Wire Wire Line
-	7000 5225 7775 5225
-Text Label 7050 5225 0    40   ~ 0
+Wire Wire Line
+	7775 5025 2675 5025
+Wire Wire Line
+	2525 5225 7775 5225
+Text Label 7225 5025 0    40   ~ 0
 SDA
-Text Label 7050 5025 0    40   ~ 0
+Text Label 7225 5225 0    40   ~ 0
 SCL
-Wire Wire Line
-	6500 4625 6500 4475
-Wire Wire Line
-	6700 4625 6700 4475
-Wire Wire Line
-	6700 4475 7300 4475
-Text Label 6425 4475 0    40   ~ 0
-5V
-Wire Wire Line
-	6600 5625 6600 5925
-Text Label 6600 6100 0    40   ~ 0
-GND
-Text Label 6700 4475 0    40   ~ 0
-3V3
-Text HLabel 7775 4475 2    40   Input ~ 0
-3V3
-Text Notes 6250 5725 2    50   ~ 10
-LEVEL TRANSLATOR\nFOR I2C 5V TO 3V3
-$Comp
-L KlokTHREEjr:R R5
-U 1 1 5A59C780
-P 7300 5675
-F 0 "R5" H 7350 5475 40  0000 C CNN
-F 1 "10k" V 7307 5676 40  0000 C CNN
-F 2 "KlokTHREEjr_libs:r_0805" V 7230 5675 30  0001 C CNN
-F 3 "~" H 7300 5675 30  0000 C CNN
-	1    7300 5675
-	1    0    0    -1
-$EndComp
-Wire Wire Line
-	7000 5425 7300 5425
-Wire Wire Line
-	7300 5425 7300 5525
-Wire Wire Line
-	7300 5825 7300 5925
-Wire Wire Line
-	7300 5925 6600 5925
-Connection ~ 6600 5925
-Wire Wire Line
-	6600 5925 6600 6100
-Wire Wire Line
-	7300 5425 7300 4475
-Connection ~ 7300 5425
-Connection ~ 7300 4475
-Wire Wire Line
-	7300 4475 7500 4475
-$Comp
-L KlokTHREEjr:C_NP C29
-U 1 1 5A5A129F
-P 5725 4650
-F 0 "C29" H 5828 4688 40  0000 L CNN
-F 1 "100nF" H 5828 4613 40  0000 L CNN
-F 2 "KlokTHREEjr_libs:c_0805" H 5725 4650 60  0001 C CNN
-F 3 "" H 5725 4650 60  0000 C CNN
-	1    5725 4650
-	1    0    0    -1
-$EndComp
-$Comp
-L KlokTHREEjr:C_NP C30
-U 1 1 5A5A13BD
-P 7500 4650
-F 0 "C30" H 7603 4688 40  0000 L CNN
-F 1 "100nF" H 7603 4613 40  0000 L CNN
-F 2 "KlokTHREEjr_libs:c_0805" H 7500 4650 60  0001 C CNN
-F 3 "" H 7500 4650 60  0000 C CNN
-	1    7500 4650
-	1    0    0    -1
-$EndComp
-Wire Wire Line
-	7500 4500 7500 4475
-Connection ~ 7500 4475
-Wire Wire Line
-	7500 4475 7775 4475
-Wire Wire Line
-	5725 4475 5725 4500
-Wire Wire Line
-	5725 4475 6500 4475
-Wire Wire Line
-	5725 4800 5725 4900
-Wire Wire Line
-	7500 4900 7500 4800
-Text Label 5725 4900 0    40   ~ 0
-GND
-Text Label 7500 4900 0    40   ~ 0
-GND
-Wire Wire Line
-	6200 5025 5100 5025
-Wire Wire Line
-	5100 5225 6200 5225
-Wire Wire Line
-	5100 5225 4900 5025
-Wire Wire Line
-	4900 5025 2675 5025
-Wire Wire Line
-	5100 5025 4900 5225
-Wire Wire Line
-	4900 5225 2525 5225
+$Comp
+L KlokTHREEjr:Conn_01x01 TP2
+U 1 1 5A95B66E
+P 7750 2850
+F 0 "TP2" H 7825 2850 50  0000 L CNN
+F 1 "SQR" H 8000 2850 50  0000 L CNN
+F 2 "KlokTHREEjr_libs:BreakOutPad" H 7750 2850 50  0001 C CNN
+F 3 "~" H 7750 2850 50  0001 C CNN
+	1    7750 2850
+	1    0    0    -1
+$EndComp
+$Comp
+L KlokTHREEjr:Conn_01x01 TP3
+U 1 1 5A95B721
+P 7750 3150
+F 0 "TP3" H 7825 3150 50  0000 L CNN
+F 1 "32kHz" H 8000 3150 50  0000 L CNN
+F 2 "KlokTHREEjr_libs:BreakOutPad" H 7750 3150 50  0001 C CNN
+F 3 "~" H 7750 3150 50  0001 C CNN
+	1    7750 3150
+	1    0    0    -1
+$EndComp
+Wire Wire Line
+	7550 2850 4900 2850
+Connection ~ 4900 2850
+Wire Wire Line
+	5050 3150 7550 3150
+Connection ~ 5050 3150
 $EndSCHEMATC
