File: k3jr_controller_kicad/k3jr_controller.sch (KiCad schematic (older format))
At the start: 26 parts, among them J17 MISO, J18 3V3, J19 SCK, J20 SPI, J21 MOSI, J22 RST, J23 GND, J24 I2C_ext1, J25 I2C_ext2, U129 ESP-wroom-32

Commit message: changed I2C connections
Connections:
- net labels removed: IO21, IO22
Changed lines of the file:
@@
 EndData
 $EndBitmap
-Text Label 1825 1925 0    40   ~ 0
+Text Label 4025 1625 2    40   ~ 0
 SCL
-Text Label 1825 2025 0    40   ~ 0
+Text Label 4025 1925 2    40   ~ 0
 SDA
 Text Label 1825 2425 0    40   ~ 0
@@
 	1825 2425 2075 2425
 Wire Wire Line
-	2075 1925 1825 1925
-Wire Wire Line
-	1825 2025 2075 2025
-Wire Wire Line
 	4025 1425 3775 1425
 Wire Wire Line
@@
 Wire Notes Line
 	4150 2625 4100 2625
-Wire Notes Line
-	1725 1925 1675 1925
-Wire Notes Line
-	1675 1925 1675 2025
-Wire Notes Line
-	1675 2025 1725 2025
 Text Notes 4150 2175 0    40   ~ 0
 BUTTONS
 Text Notes 4150 2575 0    40   ~ 0
 LED CLK/DAT
-Text Notes 1650 1975 2    40   ~ 0
+Text Notes 4525 1675 2    40   ~ 0
 I2C
 Wire Notes Line
@@
 NoConn ~ 2675 3125
 NoConn ~ 3775 1525
-NoConn ~ 3775 1625
 Wire Wire Line
 	3775 1325 4025 1325
@@
 Text Label 3375 3125 3    40   ~ 0
 IO2
-Text Label 3775 1625 0    40   ~ 0
-IO22
 Text Label 3775 1525 0    40   ~ 0
 IO23
-NoConn ~ 3775 1925
-Text Label 3775 1925 0    40   ~ 0
-IO21
 Text Label 3775 2025 0    40   ~ 0
 NC
@@
 	1    0    0    -1
 $EndComp
+Text Label 2425 5900 0    40   ~ 0
+SDA
 Text Label 2425 5800 0    40   ~ 0
-SDA
-Text Label 2425 5900 0    40   ~ 0
 SCL
 Text Label 2425 6000 0    40   ~ 0
@@
 	1    0    0    -1
 $EndComp
+Text Label 3475 5900 0    40   ~ 0
+SDA
 Text Label 3475 5800 0    40   ~ 0
-SDA
-Text Label 3475 5900 0    40   ~ 0
 SCL
 Text Label 3475 6000 0    40   ~ 0
@@
 Wire Wire Line
 	3400 4350 3625 4350
+Wire Wire Line
+	4025 1925 3775 1925
+Wire Wire Line
+	4025 1625 3775 1625
+NoConn ~ 2075 1925
+NoConn ~ 2075 2025
+Wire Notes Line
+	4100 1625 4400 1625
+Wire Notes Line
+	4400 1625 4400 1925
+Wire Notes Line
+	4400 1925 4100 1925
 $EndSCHEMATC

Commit message: kontroller layout modified. Old layout archived as rev _v1
Connections:
- net labels added: IO34, IO35
Changed lines of the file:
@@
 Wire Notes Line
 	4400 1925 4100 1925
+Text Label 2075 1925 2    40   ~ 0
+IO34
+Text Label 2075 2025 2    40   ~ 0
+IO35
 $EndSCHEMATC
