File: k3jr_controller_kicad/esp_pwr_uart.sch (KiCad schematic (older format))
At the start: 29 parts, among them P1 USB_micro, Q1 DDC114TU, U131 1117-33, U132 CP2102N-A01-GQFN28

Commit message: corrected I2C silk legend
Parts:
- U131: symbol KlokTHREEjr:AP1117-15 -> KlokTHREEjr:AP1117-33
Changed lines of the file:
@@
 $EndComp
 $Comp
-L KlokTHREEjr:AP1117-15 U131
+L KlokTHREEjr:AP1117-33 U131
 U 1 1 5A4518D4
 P 2175 1300

Commit message: Kontroller layout/Gerber final
Parts:
- P1: footprint k3jr_controller_libs:USB_Micro-B_Molex-105017-0001_round -> k3jr_controller_libs:USB_Micro-B_Molex-105017-0001
Changed lines of the file:
@@
 F 0 "P1" H 1527 4148 40  0000 C CNB
 F 1 "USB_micro" H 1527 4073 40  0000 C CNB
-F 2 "k3jr_controller_libs:USB_Micro-B_Molex-105017-0001_round" H 1475 4000 60  0001 C CNN
+F 2 "k3jr_controller_libs:USB_Micro-B_Molex-105017-0001" H 1475 4000 60  0001 C CNN
 F 3 "" H 1475 4050 60  0000 C CNN
 	1    1475 4000
